Commit message: hector_sensors_description: added macro kinect_camera with kinect sensor plugin for gazebo hector_quadrotor: added urdf and launch file quadrotor_with_kinect

File: hector_sensors_description/urdf/kinect_camera.urdf.xacro (robot description, xacro)
@@ -28,24 +28,62 @@
         </collision>
       </link>
-<!--    <gazebo reference="${name}_link">
-      <sensor:camera name="${name}_camera_sensor">
-        <imageSize>320 240</imageSize>
-        <imageFormat>R8G8B8</imageFormat>
-        <hfov>90</hfov>
-        <nearClip>0.01</nearClip>
-        <farClip>100</farClip>
-        <updateRate>${update_rate}</updateRate>
-        <controller:gazebo_ros_camera name="${name}_camera_controller" plugin="libgazebo_ros_camera.so">
-          <alwaysOn>true</alwaysOn>
-          <updateRate>${update_rate}</updateRate>
-          <imageTopicName>${ros_topic}</imageTopicName>
-          <cameraInfoTopicName>${cam_info_topic}</cameraInfoTopicName>
-          <frameName>${name}_optical_frame</frameName>
-          <interface:camera name="${name}_camera_iface" />
-        </controller:gazebo_ros_camera>
-      </sensor:camera>
-      <turnGravityOff>true</turnGravityOff>
-      <material>PR2/Blue</material>
-    </gazebo>-->
+    </xacro:macro>
+    <xacro:macro name="kinect_camera" params="name parent *origin">
+      <kinect_camera_model name="${name}" parent="${parent}">
+        <insert_block name="origin" />
+      </kinect_camera_model>
+      <!-- ASUS Xtion PRO camera for simulation -->
+      <!-- gazebo_ros_wge100 plugin is in kt2_gazebo_plugins package -->
+      <!-- <gazebo reference="${name}_link" >
+        <sensor:camera name="${name}" >
+          <imageSize>640 480</imageSize>
+          <imageFormat>R8G8B8</imageFormat>
+          <hfov>62.8</hfov>
+          <nearClip>0.1</nearClip>
+          <farClip>10</farClip>
+          <updateRate>2.0</updateRate>
+          <controller:gazebo_ros_wge100 name="${name}_camera_controller" plugin="libgazebo_ros_wge100.so">
+	    <alwaysOn>true</alwaysOn>
+	    <updateRate>5000.0</updateRate>
+	    <cameraName>${name}/rgb</cameraName>
+	    <frameName>${name}_rgb_optical_frame</frameName>
+	    <hackBaseline>0.0</hackBaseline>
+	    <CxPrime>320.5</CxPrime>
+	    <Cx>320.5</Cx>
+	    <Cy>240.5</Cy>
+	    <baseline>0.09</baseline>
+	    <focal_length>525</focal_length>
+	    <cameraNamespace>camera/rgb</cameraNamespace>
+	    <depthData>true</depthData>
+	    <interface:camera name="camera_iface" />
+          </controller:gazebo_ros_wge100>
+        </sensor:camera>
+      </gazebo> -->
+      <gazebo reference="${name}_link">
+        <sensor:camera name="${name}">
+          <imageFormat>R8G8B8</imageFormat>
+          <imageSize>640 480</imageSize>
+          <hfov>60</hfov>
+          <nearClip>0.05</nearClip>
+          <farClip>3</farClip>
+          <updateRate>20</updateRate>
+          <baseline>0.1</baseline>
+          <controller:gazebo_ros_openni_kinect name="${name}_camera_controller" plugin="libgazebo_ros_openni_kinect.so">
+            <alwaysOn>true</alwaysOn>
+            <updateRate>20</updateRate>
+            <imageTopicName>${name}/rgb/image_raw</imageTopicName>
+            <cameraInfoTopicName>${name}/rgb/camera_info</cameraInfoTopicName>
+            <depthImageTopicName>${name}/depth/image_raw</depthImageTopicName>
+            <depthImageCameraInfoTopicName>${name}/depth/camera_info</depthImageCameraInfoTopicName>
+            <pointCloudTopicName>${name}/depth/points</pointCloudTopicName>
+            <frameName>${name}_depth_optical_frame</frameName>
+            <distortion_k1>0.0</distortion_k1>
+            <distortion_k2>0.0</distortion_k2>
+            <distortion_k3>0.0</distortion_k3>
+            <distortion_t1>0.0</distortion_t1>
+            <distortion_t2>0.0</distortion_t2>
+          </controller:gazebo_ros_openni_kinect>
+        </sensor:camera>
+      </gazebo>
     </xacro:macro>
   </robot>

Commit message: [hector_sensor_description] -calibrate camera sensor head x-coordinate

File: hector_sensors_description/urdf/kinect_camera.urdf.xacro (robot description, xacro)
@@ -37,5 +37,5 @@
       <link name="${name}_depth_optical_frame"/>
       <joint name="${name}_rgb_joint" type="fixed">
-        <origin xyz="0.0 -0.045 0.0" rpy="0 0 0" />
+        <origin xyz="0.0 -0.0125 0.0" rpy="0 0 0" />
         <parent link="${name}_link" />
         <child link="${name}_rgb_frame"/>

Commit message: [hector_sensor_description] -calibrate camera sensor head x-coordinate

File: hector_sensors_description/urdf/kinect_camera.urdf.xacro (robot description, xacro)
@@ -41,5 +41,5 @@
       <link name="${name}_depth_optical_frame"/>
       <joint name="${name}_rgb_joint" type="fixed">
-        <origin xyz="0.0 -0.045 0.0" rpy="0 0 0" />
+        <origin xyz="0.0 -0.0125 0.0" rpy="0 0 0" />
         <parent link="${name}_link" />
         <child link="${name}_rgb_frame"/>
