Commit message: hector_sensors_description: updated plugin code to use new sdf format

File: hector_sensors_description/urdf/asus_camera.urdf.xacro (robot description, xacro)
@@ -1,8 +1,4 @@
 <?xml version="1.0"?>
-<robot xmlns:sensor="http://playerstage.sourceforge.net/gazebo/xmlschema/#sensor"
-xmlns:controller="http://playerstage.sourceforge.net/gazebo/xmlschema/#controller"
-xmlns:interface="http://playerstage.sourceforge.net/gazebo/xmlschema/#interface"
-  xmlns:xacro="http://ros.org/wiki/xacro"
-  >
+<robot xmlns:xacro="http://ros.org/wiki/xacro">
     <include filename="$(find hector_xacro_tools)/urdf/sensor_macros.urdf.xacro" />
     <property name="M_PI" value="3.1415926535897931" />
@@ -63,13 +59,19 @@
       <!-- ASUS Xtion PRO camera for simulation -->
       <gazebo reference="${name}_depth_frame">
-        <sensor:camera name="${name}">
-          <imageFormat>R8G8B8</imageFormat>
-          <imageSize>640 480</imageSize>
-          <hfov>62.8</hfov>
-          <nearClip>0.5</nearClip>
-          <farClip>9</farClip>
-          <updateRate>20</updateRate>
-          <baseline>0.1</baseline>
-          <controller:gazebo_ros_openni_kinect name="${name}_camera_controller" plugin="libgazebo_ros_openni_kinect.so">
+        <sensor type="depth" name="${name}">
+          <update_rate>20</update_rate>
+          <camera>
+            <horizontal_fov>${62.8 * M_PI/180.0}</horizontal_fov>
+            <image>
+              <format>R8G8B8</format>
+              <width>640</width>
+              <height>480</height>
+            </image>
+            <clip>
+              <near>0.5</near>
+              <far>9</far>
+            </clip>
+          </camera>
+          <plugin name="${name}_camera_controller" filename="libgazebo_ros_openni_kinect.so">
             <alwaysOn>true</alwaysOn>
             <updateRate>20</updateRate>
@@ -85,6 +87,6 @@
             <distortion_t1>0.0</distortion_t1>
             <distortion_t2>0.0</distortion_t2>
-          </controller:gazebo_ros_openni_kinect>
-        </sensor:camera>
+          </plugin>
+        </sensor>
       </gazebo>
     </xacro:macro>

File: hector_sensors_description/urdf/generic_camera.urdf.xacro (robot description, xacro)
@@ -1,8 +1,4 @@
 <?xml version="1.0"?>
-<robot xmlns:sensor="http://playerstage.sourceforge.net/gazebo/xmlschema/#sensor"
-xmlns:controller="http://playerstage.sourceforge.net/gazebo/xmlschema/#controller"
-xmlns:interface="http://playerstage.sourceforge.net/gazebo/xmlschema/#interface"
-  xmlns:xacro="http://ros.org/wiki/xacro"
-  >
+<robot xmlns:xacro="http://ros.org/wiki/xacro">
     <property name="M_PI" value="3.1415926535897931" />
     <xacro:macro name="generic_camera" params="name parent *origin ros_topic cam_info_topic update_rate res_x res_y image_format hfov">
@@ -41,12 +37,19 @@
     <link name="${name}_optical_frame"/>
     <gazebo reference="${name}_link">
-      <sensor:camera name="${name}_camera_sensor">
-        <imageSize>${res_x} ${res_y}</imageSize>
-        <imageFormat>${image_format}</imageFormat>
-        <hfov>${hfov}</hfov>
-        <nearClip>0.01</nearClip>
-        <farClip>100</farClip>
-        <updateRate>${update_rate}</updateRate>
-        <controller:gazebo_ros_depth_camera name="${name}_camera_controller" plugin="libgazebo_ros_depth_camera.so">
+      <sensor type="camera" name="${name}_camera_sensor">
+        <update_rate>${update_rate}</update_rate>
+        <camera>
+          <horizontal_fov>${${hfov} * M_PI/180.0}</horizontal_fov>
+          <image>
+            <format>${image_format}</format>
+            <width>${res_x}</width>
+            <height>${res_y}</height>
+          </image>
+          <clip>
+            <near>0.01</near>
+            <far>100</far>
+          </clip>
+        </camera>
+        <plugin name="${name}_camera_controller" filename="libgazebo_ros_depth_camera.so">
 	  <cameraName>${name}</cameraName>
           <alwaysOn>true</alwaysOn>
@@ -55,8 +58,6 @@
           <cameraInfoTopicName>${cam_info_topic}</cameraInfoTopicName>
           <frameName>${name}_optical_frame</frameName>
-          <interface:camera name="${name}_camera_iface" />
         </controller:gazebo_ros_depth_camera>
-      </sensor:camera>
-      <turnGravityOff>true</turnGravityOff>
+      </sensor>
       <material>PR2/Blue</material>
     </gazebo>

File: hector_sensors_description/urdf/hokuyo_utm30lx.urdf.xacro (robot description, xacro)
@@ -1,8 +1,4 @@
 <?xml version="1.0"?>
-<robot xmlns:sensor="http://playerstage.sourceforge.net/gazebo/xmlschema/#sensor"
-xmlns:controller="http://playerstage.sourceforge.net/gazebo/xmlschema/#controller"
-xmlns:interface="http://playerstage.sourceforge.net/gazebo/xmlschema/#interface"
-  xmlns:xacro="http://ros.org/wiki/xacro"
-  >
+<robot xmlns:xacro="http://ros.org/wiki/xacro">
     <xacro:macro name="hokuyo_utm30lx" params="name parent *origin ros_topic update_rate ray_count min_angle max_angle">
       <joint name="${name}_joint" type="fixed">
@@ -32,17 +28,25 @@
       </link>
       <gazebo reference="${name}_frame">
-        <sensor:ray name="${name}">
-          <rayCount>${ray_count}</rayCount>
-          <rangeCount>${ray_count}</rangeCount>
-          <laserCount>1</laserCount>
-          <origin>0.0 0.0 0.0</origin>
-          <displayRays>false</displayRays>
-          <minAngle>${min_angle}</minAngle>
-          <maxAngle>${max_angle}</maxAngle>
-          <minRange>0.08</minRange>
-          <maxRange>30.0</maxRange>
-          <resRange>0.01</resRange>
-          <updateRate>${update_rate}</updateRate>
-          <controller:gazebo_ros_laser name="gazebo_ros_${name}_controller" plugin="libgazebo_ros_laser.so">
+        <sensor type="ray" name="${name}">
+          <always_on>true</always_on>
+          <update_rate>${update_rate}</update_rate>
+          <pose>0 0 0 0 0 0</pose>
+          <visualize>false</visualize>
+          <ray>
+            <scan>
+              <horizontal>
+                <samples>${ray_count}</samples>
+                <resolution>1</resolution>
+                <min_angle>${min_angle}</min_angle>
+                <max_angle>${max_angle}</max_angle>
+              </horizontal>
+            </scan>
+            <range>
+              <min>0.08</min>
+              <max>30.0</max>
+              <resolution>0.01</resolution>
+            </range>
+          </ray>
+          <plugin name="gazebo_ros_${name}_controller" filename="libgazebo_ros_laser.so">
             <gaussianNoise>0.005</gaussianNoise>
             <alwaysOn>true</alwaysOn>
@@ -50,7 +54,6 @@
             <topicName>${ros_topic}</topicName>
             <frameName>${name}_frame</frameName>
-            <interface:laser name="gazebo_ros_${name}_iface" />
-          </controller:gazebo_ros_laser>
-        </sensor:ray>
+          </plugin>
+        </sensor>
       </gazebo>
     </xacro:macro>

File: hector_sensors_description/urdf/kinect_camera.urdf.xacro (robot description, xacro)
@@ -1,8 +1,4 @@
 <?xml version="1.0"?>
-<robot xmlns:sensor="http://playerstage.sourceforge.net/gazebo/xmlschema/#sensor"
-xmlns:controller="http://playerstage.sourceforge.net/gazebo/xmlschema/#controller"
-xmlns:interface="http://playerstage.sourceforge.net/gazebo/xmlschema/#interface"
-  xmlns:xacro="http://ros.org/wiki/xacro"
-  >
+<robot xmlns:xacro="http://ros.org/wiki/xacro">
     <include filename="$(find hector_xacro_tools)/urdf/sensor_macros.urdf.xacro" />
     <property name="M_PI" value="3.1415926535897931" />
@@ -58,13 +54,19 @@
       </kinect_camera_model>
       <gazebo reference="${name}_depth_frame">
-        <sensor:camera name="${name}">
-          <imageFormat>R8G8B8</imageFormat>
-          <imageSize>640 480</imageSize>
-          <hfov>60</hfov>
-          <nearClip>0.05</nearClip>
-          <farClip>3</farClip>
-          <updateRate>20</updateRate>
-          <baseline>0.1</baseline>
-          <controller:gazebo_ros_openni_kinect name="${name}_camera_controller" plugin="libgazebo_ros_openni_kinect.so">
+        <sensor type="depth" name="${name}">
+          <update_rate>20</update_rate>
+          <camera>
+            <horizontal_fov>${60 * M_PI/180.0}</horizontal_fov>
+            <image>
+              <format>R8G8B8</format>
+              <width>640</width>
+              <height>480</height>
+            </image>
+            <clip>
+              <near>0.05</near>
+              <far>3</far>
+            </clip>
+          </camera>
+          <plugin name="${name}_camera_controller" filename="libgazebo_ros_openni_kinect.so">
             <alwaysOn>true</alwaysOn>
             <updateRate>20</updateRate>
@@ -80,6 +82,6 @@
             <distortion_t1>0.0</distortion_t1>
             <distortion_t2>0.0</distortion_t2>
-          </controller:gazebo_ros_openni_kinect>
-        </sensor:camera>
+          </plugin>
+        </sensor>
       </gazebo>
     </xacro:macro>

File: hector_sensors_description/urdf/sonar_sensor.urdf.xacro (robot description, xacro)
@@ -1,8 +1,4 @@
 <?xml version="1.0"?>
-<robot xmlns:sensor="http://playerstage.sourceforge.net/gazebo/xmlschema/#sensor"
-xmlns:controller="http://playerstage.sourceforge.net/gazebo/xmlschema/#controller"
-xmlns:interface="http://playerstage.sourceforge.net/gazebo/xmlschema/#interface"
-xmlns:xacro="http://ros.org/wiki/xacro"
->
+<robot xmlns:xacro="http://ros.org/wiki/xacro">
   <xacro:macro name="sonar_sensor" params="name parent *origin ros_topic update_rate min_range max_range field_of_view ray_count">
     <joint name="${name}_joint" type="fixed">
@@ -32,23 +28,36 @@
     </link>
     <gazebo reference="${name}_link">
-      <sensor:ray name="${name}">
-        <rayCount>${ray_count}</rayCount>
-        <rangeCount>${ray_count}</rangeCount>
-        <verticalRayCount>${ray_count}</verticalRayCount>
-        <verticalRangeCount>${ray_count}</verticalRangeCount>
-        <minAngle>-${field_of_view/2}</minAngle>
-        <verticalMinAngle>-${field_of_view/2}</verticalMinAngle>
-        <maxAngle>${field_of_view/2}</maxAngle>
-        <verticalMaxAngle>${field_of_view/2}</verticalMaxAngle>
-        <minRange>${min_range}</minRange>
-        <maxRange>${max_range}</maxRange>
-        <resRange>0.01</resRange>
-        <updateRate>${update_rate}</updateRate>
-        <controller:hector_gazebo_ros_sonar name="gazebo_ros_${name}_controller" plugin="libhector_gazebo_ros_sonar.so">
+      <sensor type="ray" name="${name}">
+        <always_on>true</always_on>
+        <update_rate>${update_rate}</update_rate>
+        <pose>0 0 0 0 0 0</pose>
+        <visualize>false</visualize>
+        <ray>
+          <scan>
+            <horizontal>
+              <samples>${ray_count}</samples>
+              <resolution>1</resolution>
+              <min_angle>-${field_of_view/2}</min_angle>
+              <max_angle> ${field_of_view/2}</max_angle>
+            </horizontal>
+            <vertical>
+              <samples>${ray_count}</samples>
+              <resolution>1</resolution>
+              <min_angle>-${field_of_view/2}</min_angle>
+              <max_angle> ${field_of_view/2}</max_angle>
+            </vertical>
+          </scan>
+          <range>
+            <min>${min_range}</min>
+            <max>${max_range}</max>
+            <resolution>0.01</resolution>
+          </range>
+        </ray>
+        <plugin name="gazebo_ros_${name}_controller" filename="libhector_gazebo_ros_sonar.so">
           <gaussianNoise>0.005</gaussianNoise>
           <topicName>${ros_topic}</topicName>
           <frameId>${name}_link</frameId>
-        </controller:hector_gazebo_ros_sonar>
-      </sensor:ray>
+        </plugin>
+      </sensor>
     </gazebo>
   </xacro:macro>

File: hector_sensors_description/urdf/thermaleye_camera.urdf.xacro (robot description, xacro)
@@ -1,8 +1,4 @@
 <?xml version="1.0"?>
-<robot xmlns:sensor="http://playerstage.sourceforge.net/gazebo/xmlschema/#sensor"
-xmlns:controller="http://playerstage.sourceforge.net/gazebo/xmlschema/#controller"
-xmlns:interface="http://playerstage.sourceforge.net/gazebo/xmlschema/#interface"
-  xmlns:xacro="http://ros.org/wiki/xacro"
-  >
+<robot xmlns:xacro="http://ros.org/wiki/xacro">
     <include filename="$(find hector_xacro_tools)/urdf/sensor_macros.urdf.xacro" />
     <property name="M_PI" value="3.1415926535897931" />
@@ -29,24 +25,4 @@
       </link>
       <add_optical_frame name="${name}" />
-<!--    <gazebo reference="${name}_link">
-      <sensor:camera name="${name}_camera_sensor">
-        <imageSize>320 240</imageSize>
-        <imageFormat>R8G8B8</imageFormat>
-        <hfov>90</hfov>
-        <nearClip>0.01</nearClip>
-        <farClip>100</farClip>
-        <updateRate>${update_rate}</updateRate>
-        <controller:gazebo_ros_camera name="${name}_camera_controller" plugin="libgazebo_ros_camera.so">
-          <alwaysOn>true</alwaysOn>
-          <updateRate>${update_rate}</updateRate>
-          <imageTopicName>${ros_topic}</imageTopicName>
-          <cameraInfoTopicName>${cam_info_topic}</cameraInfoTopicName>
-          <frameName>${name}_optical_frame</frameName>
-          <interface:camera name="${name}_camera_iface" />
-        </controller:gazebo_ros_camera>
-      </sensor:camera>
-      <turnGravityOff>true</turnGravityOff>
-      <material>PR2/Blue</material>
-    </gazebo>-->
     </xacro:macro>
   </robot>

Commit message: cleaned up urdf descriptions and fixed horizontal_fov tag in generic_camera.urdf.xacro

File: hector_sensors_description/urdf/asus_camera.urdf.xacro (robot description, xacro)
@@ -2,5 +2,5 @@
 <robot xmlns:xacro="http://ros.org/wiki/xacro">
     <include filename="$(find hector_xacro_tools)/urdf/sensor_macros.urdf.xacro" />
-    <property name="M_PI" value="3.1415926535897931" />
+    <xacro:property name="M_PI" value="3.1415926535897931" />
     <xacro:macro name="asus_camera_model" params="name parent *origin">
       <joint name="${name}_joint" type="fixed">

File: hector_sensors_description/urdf/generic_camera.urdf.xacro (robot description, xacro)
@@ -1,33 +1,33 @@
 <?xml version="1.0"?>
 <robot xmlns:xacro="http://ros.org/wiki/xacro">
-    <property name="M_PI" value="3.1415926535897931" />
-    <xacro:macro name="generic_camera" params="name parent *origin ros_topic cam_info_topic update_rate res_x res_y image_format hfov">
-      <joint name="${name}_joint" type="fixed">
-        <insert_block name="origin" />
-        <parent link="${parent}"/>
-        <child link="${name}_link"/>
-      </joint>
-      <link name="${name}_link">
-        <inertial>
-          <mass value="0.001" />
-          <origin xyz="0 0 0" rpy="0 0 0" />
-          <inertia ixx="0.0001" ixy="0" ixz="0" iyy="0.0001" iyz="0" izz="0.0001" />
-        </inertial>
-        <visual>
-          <origin xyz="0 0 0" rpy="0 0 0" />
-          <geometry>
-            <box size="0.01 0.01 0.01" />
-          </geometry>
-	  <material name="Blue">
-      <color rgba="0.0 0.0 0.8 1"/>
-    </material>
-        </visual>
-        <collision>
-          <origin xyz="0 0 0" rpy="0 0 0" />
-          <geometry>
-            <box size="0.01 0.01 0.01" />
-          </geometry>
-        </collision>
-      </link>
+  <xacro:property name="M_PI" value="3.1415926535897931" />
+  <xacro:macro name="generic_camera" params="name parent *origin ros_topic cam_info_topic update_rate res_x res_y image_format hfov">
+    <joint name="${name}_joint" type="fixed">
+      <insert_block name="origin" />
+      <parent link="${parent}"/>
+      <child link="${name}_link"/>
+    </joint>
+    <link name="${name}_link">
+      <inertial>
+        <mass value="0.001" />
+        <origin xyz="0 0 0" rpy="0 0 0" />
+        <inertia ixx="0.0001" ixy="0" ixz="0" iyy="0.0001" iyz="0" izz="0.0001" />
+      </inertial>
+      <visual>
+        <origin xyz="0 0 0" rpy="0 0 0" />
+        <geometry>
+          <box size="0.01 0.01 0.01" />
+        </geometry>
+        <material name="Blue">
+          <color rgba="0.0 0.0 0.8 1"/>
+        </material>
+      </visual>
+      <collision>
+        <origin xyz="0 0 0" rpy="0 0 0" />
+        <geometry>
+          <box size="0.01 0.01 0.01" />
+        </geometry>
+      </collision>
+    </link>
     <joint name="${name}_optical_joint" type="fixed">
       <origin xyz="0 0 0" rpy="${-M_PI/2} 0.0 ${-M_PI/2}" />
@@ -40,5 +40,5 @@
         <update_rate>${update_rate}</update_rate>
         <camera>
-          <horizontal_fov>${${hfov} * M_PI/180.0}</horizontal_fov>
+          <horizontal_fov>${hfov * M_PI/180.0}</horizontal_fov>
           <image>
             <format>${image_format}</format>
@@ -52,5 +52,5 @@
         </camera>
         <plugin name="${name}_camera_controller" filename="libgazebo_ros_depth_camera.so">
-	  <cameraName>${name}</cameraName>
+          <cameraName>${name}</cameraName>
           <alwaysOn>true</alwaysOn>
           <updateRate>${update_rate}</updateRate>
@@ -58,8 +58,8 @@
           <cameraInfoTopicName>${cam_info_topic}</cameraInfoTopicName>
           <frameName>${name}_optical_frame</frameName>
-        </controller:gazebo_ros_depth_camera>
+        </plugin>
       </sensor>
       <material>PR2/Blue</material>
     </gazebo>
-    </xacro:macro>
-  </robot>
+  </xacro:macro>
+</robot>

File: hector_sensors_description/urdf/kinect_camera.urdf.xacro (robot description, xacro)
@@ -2,5 +2,5 @@
 <robot xmlns:xacro="http://ros.org/wiki/xacro">
     <include filename="$(find hector_xacro_tools)/urdf/sensor_macros.urdf.xacro" />
-    <property name="M_PI" value="3.1415926535897931" />
+    <xacro:property name="M_PI" value="3.1415926535897931" />
     <xacro:macro name="kinect_camera_model" params="name parent *origin">
       <joint name="${name}_joint" type="fixed">

File: hector_sensors_description/urdf/thermaleye_camera.urdf.xacro (robot description, xacro)
@@ -2,5 +2,5 @@
 <robot xmlns:xacro="http://ros.org/wiki/xacro">
     <include filename="$(find hector_xacro_tools)/urdf/sensor_macros.urdf.xacro" />
-    <property name="M_PI" value="3.1415926535897931" />
+    <xacro:property name="M_PI" value="3.1415926535897931" />
     <xacro:macro name="thermaleye_camera_model" params="name parent *origin">
       <joint name="${name}_joint" type="fixed">

File: hector_xacro_tools/urdf/inertia_tensors.urdf.xacro (robot description, xacro)
@@ -1,24 +1,21 @@
 <?xml version="1.0"?>
-<robot xmlns:controller="http://playerstage.sourceforge.net/gazebo/xmlschema/#controller"
-  xmlns:interface="http://playerstage.sourceforge.net/gazebo/xmlschema/#interface"
-  xmlns:sensor="http://playerstage.sourceforge.net/gazebo/xmlschema/#sensor"
-  xmlns:xacro="http://ros.org/wiki/xacro">
-<macro name="inertial_cuboid" params="mass x_length y_length z_length">
-  <inertial>
-    <mass value="${mass}" />
-    <origin xyz="0 0 0" />
-    <inertia ixx="${(1/12) * mass* (y_length*y_length+ z_length*z_length)}" ixy="0.0" ixz="0.0"
-             iyy="${(1/12) * mass* (x_length*x_length+ z_length*z_length)}" iyz="0.0"
-             izz="${(1/12) * mass* (x_length*x_length+ y_length*y_length)}" />
-  </inertial>
-</macro>
-<macro name="inertial_sphere" params="mass diameter">
-  <inertial>
-    <mass value="${mass}" />
-    <origin xyz="0 0 0" />
-    <inertia ixx="${(2/5) * mass* ( (diameter*0.5)) * (diameter*0.5))}" ixy="0.0" ixz="0.0"
-             iyy="${(2/5) * mass* ( (diameter*0.5)) * (diameter*0.5))}" iyz="0.0"
-             izz="${(2/5) * mass* ( (diameter*0.5)) * (diameter*0.5))}" />
-  </inertial>
-</macro>
+<robot xmlns:xacro="http://ros.org/wiki/xacro">
+  <xacro:macro name="inertial_cuboid" params="mass x_length y_length z_length">
+    <inertial>
+      <mass value="${mass}" />
+      <origin xyz="0 0 0" />
+      <inertia ixx="${(1/12) * mass* (y_length*y_length+ z_length*z_length)}" ixy="0.0" ixz="0.0"
+               iyy="${(1/12) * mass* (x_length*x_length+ z_length*z_length)}" iyz="0.0"
+               izz="${(1/12) * mass* (x_length*x_length+ y_length*y_length)}" />
+    </inertial>
+  </xacro:macro>
+  <xacro:macro name="inertial_sphere" params="mass diameter">
+    <inertial>
+      <mass value="${mass}" />
+      <origin xyz="0 0 0" />
+      <inertia ixx="${(2/5) * mass* ( (diameter*0.5)) * (diameter*0.5))}" ixy="0.0" ixz="0.0"
+               iyy="${(2/5) * mass* ( (diameter*0.5)) * (diameter*0.5))}" iyz="0.0"
+               izz="${(2/5) * mass* ( (diameter*0.5)) * (diameter*0.5))}" />
+    </inertial>
+  </xacro:macro>
 </robot>

File: hector_xacro_tools/urdf/sensor_macros.urdf.xacro (robot description, xacro)
@@ -1,8 +1,5 @@
 <?xml version="1.0"?>
-<robot xmlns:controller="http://playerstage.sourceforge.net/gazebo/xmlschema/#controller"
-  xmlns:interface="http://playerstage.sourceforge.net/gazebo/xmlschema/#interface"
-  xmlns:sensor="http://playerstage.sourceforge.net/gazebo/xmlschema/#sensor"
-  xmlns:xacro="http://ros.org/wiki/xacro">
-<macro name="add_optical_frame" params="name">
+<robot xmlns:xacro="http://ros.org/wiki/xacro">
+  <xacro:macro name="add_optical_frame" params="name">
     <joint name="${name}_optical_joint" type="fixed">
       <origin xyz="0 0 0" rpy="${-M_PI/2} 0.0 ${-M_PI/2}" />
@@ -10,25 +7,5 @@
       <child link="${name}_optical_frame"/>
     </joint>
-    <link name="${name}_optical_frame">
-<!--      <inertial>
-        <mass value="0.01" />
-        <origin xyz="0 0 0" />
-        <inertia ixx="0.001"  ixy="0.0"  ixz="0.0"
-                 iyy="0.001"  iyz="0.0"
-                 izz="0.001" />
-      </inertial>
-      <visual>
-        <origin xyz="0 0 0" rpy="0 0 0"/>
-        <geometry>
-          <box size="0.001 0.001 0.001" />
-        </geometry>
-      </visual>
-      <collision>
-        <origin xyz="0 0 0" rpy="0 0 0"/>
-        <geometry>
-          <box size="0.001 0.001 0.001" />
-        </geometry>
-      </collision>-->
-    </link>
-</macro>
+    <link name="${name}_optical_frame" />
+  </xacro:macro>
 </robot>

Commit message: -Use cylinder collision geom as box gives spurious errors in LIDAR scans in some URDFs

File: hector_sensors_description/urdf/asus_camera.urdf.xacro (robot description, xacro)
@@ -20,8 +20,16 @@
           </geometry>
         </visual>
-        <collision>
+       <!--
+       <collision>
           <origin xyz="0 0 0" rpy="0 0 0" />
           <geometry>
             <box size="0.035 0.185 0.025"/>
+          </geometry>
+        </collision>
+        -->
+        <collision>
+          <origin xyz="-0.017 0 0" rpy="${M_PI*0.5} 0 0" />
+          <geometry>
+            <cylinder length="0.185" radius="0.02"/>
           </geometry>
         </collision>

Commit message: changed asus description, collision geometry needs to match visual geometry for 3d self filter to work.

File: hector_sensors_description/urdf/asus_camera.urdf.xacro (robot description, xacro)
@@ -29,7 +29,7 @@
         -->
         <collision>
-          <origin xyz="-0.017 0 0" rpy="${M_PI*0.5} 0 0" />
+          <origin xyz="0 0 0" rpy="0 0 0" />
           <geometry>
-            <cylinder length="0.185" radius="0.02"/>
+            <mesh filename="package://hector_sensors_description/meshes/asus_camera/asus_camera_simple.dae"/>
           </geometry>
         </collision>
