Commit message: Move depth frame backward based on testing

File: hector_sensors_description/urdf/asus_camera.urdf.xacro (robot description, xacro)
@@ -36,5 +36,5 @@
       </link>
       <joint name="${name}_depth_joint" type="fixed">
-        <origin xyz="0.0 0.049 0.0" rpy="0 0 0" />
+        <origin xyz="-0.03 0.049 0.0" rpy="0 0 0" />
         <parent link="${name}_link" />
         <child link="${name}_depth_frame"/>
