Commit message: [hector_ugv] -current state of fuerte migration (laser scanner and kinect geometry, textureless top box etc.)

File: hector_sensors_description/urdf/hokuyo_utm30lx.urdf.xacro (robot description, xacro)
@@ -11,5 +11,5 @@
 	<child link="${name}_frame"/>
       </joint>
-      <link name="${name}_frame">
+<link name="${name}_frame">
 	<inertial>
 	  <mass value="0.001" />
@@ -30,26 +30,28 @@
         </geometry>
 	</collision>
-      </link>
-      <gazebo reference="${name}_frame">
-	<sensor:ray name="${name}">
-		<rayCount>${ray_count}</rayCount>
-		<rangeCount>${ray_count}</rangeCount>
-		<displayRays>false</displayRays>
-	  <minAngle>${min_angle}</minAngle>
-	  <maxAngle>${max_angle}</maxAngle>
-	  <minRange>0.05</minRange>
-	  <maxRange>30.0</maxRange>
-	  <resRange>0.01</resRange>
-	  <updateRate>${update_rate}</updateRate>
-	  <controller:gazebo_ros_laser name="gazebo_ros_${name}_controller" plugin="libgazebo_ros_laser.so">
-	    <gaussianNoise>0.005</gaussianNoise>
-	    <alwaysOn>true</alwaysOn>
-	    <updateRate>${update_rate}</updateRate>
-	    <topicName>${ros_topic}</topicName>
-	    <frameName>/${name}_frame</frameName>
-	    <interface:laser name="gazebo_ros_${name}_iface" />
-	  </controller:gazebo_ros_laser>
-	</sensor:ray>
-      </gazebo>
+</link>
+  <gazebo reference="${name}_frame">
+    <sensor:ray name="${name}">
+    <rayCount>${ray_count}</rayCount>
+    <rangeCount>${ray_count}</rangeCount>
+        <laserCount>1</laserCount>
+        <origin>0.0 0.0 0.0</origin>
+        <displayRays>false</displayRays>
+        <minAngle>${min_angle}</minAngle>
+        <maxAngle>${max_angle}</maxAngle>
+        <minRange>0.08</minRange>
+        <maxRange>30.0</maxRange>
+        <resRange>0.01</resRange>
+        <updateRate>${update_rate}</updateRate>
+        <controller:gazebo_ros_laser name="gazebo_ros_${name}_controller" plugin="libgazebo_ros_laser.so">
+          <gaussianNoise>0.005</gaussianNoise>
+          <alwaysOn>true</alwaysOn>
+          <updateRate>${update_rate}</updateRate>
+          <topicName>${ros_topic}</topicName>
+          <frameName>${name}_frame</frameName>
+          <interface:laser name="gazebo_ros_${name}_iface" />
+        </controller:gazebo_ros_laser>
+      </sensor:ray>
+    </gazebo>
     </xacro:macro>
   </robot>

Commit message: [hector_sensors_description] - added asus xiton live pro sensor model ( mesh is  still missing - using kinect mesh) - added mass/inertia for hokoyo laser scanner
[hector_quadrotor_urdf/hector_quadrotor_gazebo]
- added asus xiton quadrotor model/launch file
- added asus with laser scanner quadrotor model/launch file
- updated ultrasonic sensor position

File: hector_sensors_description/urdf/hokuyo_utm30lx.urdf.xacro (robot description, xacro)
@@ -13,7 +13,7 @@
 <link name="${name}_frame">
 	<inertial>
-	  <mass value="0.001" />
+	  <mass value="0.270" />
 	  <origin xyz="0 0 0" rpy="0 0 0" />
-		<inertia ixx="0.0001" ixy="0" ixz="0" iyy="0.0001" iyz="0" izz="0.0001" />
+		<inertia ixx="2.632e-4" ixy="0" ixz="0" iyy="2.632e-4" iyz="0" izz="1.62e-4" />
 	</inertial>
 	<visual>

Commit message: hector_sensors_description: use degrees for min_angle/max_angle parameters of hokuyo_utm30lx macro

File: hector_sensors_description/urdf/hokuyo_utm30lx.urdf.xacro (robot description, xacro)
@@ -1,4 +1,5 @@
 <?xml version="1.0"?>
 <robot xmlns:xacro="http://ros.org/wiki/xacro">
+    <xacro:property name="M_PI" value="3.1415926535897931" />
     <xacro:macro name="hokuyo_utm30lx" params="name parent *origin ros_topic update_rate ray_count min_angle max_angle">
       <joint name="${name}_joint" type="fixed">
@@ -38,6 +39,6 @@
                 <samples>${ray_count}</samples>
                 <resolution>1</resolution>
-                <min_angle>${min_angle}</min_angle>
-                <max_angle>${max_angle}</max_angle>
+                <min_angle>${min_angle * M_PI/180}</min_angle>
+                <max_angle>${max_angle * M_PI/180}</max_angle>
               </horizontal>
             </scan>

Commit message: hector_sensors_description: added hokuyo_utm30lx_model and hokuyo_utm30lx_gpu macros and disabled gpu laser in default hokuyo_utm30lx macro

File: hector_sensors_description/urdf/hokuyo_utm30lx.urdf.xacro (robot description, xacro)
@@ -2,5 +2,5 @@
 <robot xmlns:xacro="http://ros.org/wiki/xacro">
     <xacro:property name="M_PI" value="3.1415926535897931" />
-    <xacro:macro name="hokuyo_utm30lx" params="name parent *origin ros_topic update_rate ray_count min_angle max_angle">
+    <xacro:macro name="hokuyo_utm30lx_model" params="name parent *origin">
       <joint name="${name}_joint" type="fixed">
         <xacro:insert_block name="origin" />
@@ -28,4 +28,44 @@
         </collision>
       </link>
+    </xacro:macro>
+    <xacro:macro name="hokuyo_utm30lx" params="name parent *origin ros_topic update_rate ray_count min_angle max_angle">
+      <xacro:hokuyo_utm30lx_model name="${name}" parent="${parent}">
+        <xacro:insert_block name="origin" />
+      </xacro:hokuyo_utm30lx_model>
+      <gazebo reference="${name}_frame">
+        <sensor type="ray" name="${name}">
+          <always_on>true</always_on>
+          <update_rate>${update_rate}</update_rate>
+          <pose>0 0 0 0 0 0</pose>
+          <visualize>false</visualize>
+          <ray>
+            <scan>
+              <horizontal>
+                <samples>${ray_count}</samples>
+                <resolution>1</resolution>
+                <min_angle>${min_angle * M_PI/180}</min_angle>
+                <max_angle>${max_angle * M_PI/180}</max_angle>
+              </horizontal>
+            </scan>
+            <range>
+              <min>0.08</min>
+              <max>30.0</max>
+              <resolution>0.01</resolution>
+            </range>
+          </ray>
+          <plugin name="gazebo_ros_${name}_controller" filename="libgazebo_ros_laser.so">
+            <gaussianNoise>0.005</gaussianNoise>
+            <alwaysOn>true</alwaysOn>
+            <updateRate>${update_rate}</updateRate>
+            <topicName>${ros_topic}</topicName>
+            <frameName>${name}_frame</frameName>
+          </plugin>
+        </sensor>
+      </gazebo>
+    </xacro:macro>
+    <xacro:macro name="hokuyo_utm30lx_gpu" params="name parent *origin ros_topic update_rate ray_count min_angle max_angle">
+      <xacro:hokuyo_utm30lx_model name="${name}" parent="${parent}">
+        <xacro:insert_block name="origin" />
+      </xacro:hokuyo_utm30lx_model>
       <gazebo reference="${name}_frame">
         <sensor type="gpu_ray" name="${name}">
@@ -59,3 +99,3 @@
       </gazebo>
     </xacro:macro>
-  </robot>
+</robot>

Commit message: collison model of lidar considers now rotation

File: hector_sensors_description/urdf/hokuyo_utm30lx.urdf.xacro (robot description, xacro)
@@ -21,7 +21,7 @@
         </visual>
         <collision>
-          <origin xyz="0 0 -0.0115" rpy="0 0 0" />
+          <origin xyz="0.00 0 0.0" rpy="0 ${0.5 * M_PI} 0" />
           <geometry>
-          <box size="0.058 0.058 0.087" />
+	    <cylinder length="0.079" radius="0.0735"/>
           <!--<mesh filename="package://hector_sensors_description/meshes/hokuyo_utm30lx/hokuyo_utm_30lx.stl"/>-->
         </geometry>
