Commit message: Corrected realsense frames and measures

File: hector_sensors_description/urdf/realsense_camera.urdf.xacro (robot description, xacro)
@@ -45,5 +45,5 @@
       </link>
       <joint name="${name}_depth_joint" type="fixed">
-        <origin xyz="0.0 0.049 0.0" rpy="0 0 0" />
+        <origin xyz="0 -0.051 0.004" rpy="0 0 0" />
         <parent link="${name}_link" />
         <child link="${name}_depth_frame"/>
@@ -56,6 +56,18 @@
       </joint>
       <link name="${name}_depth_optical_frame"/>
+      <joint name="${name}_depth_joint_aux" type="fixed">
+        <origin xyz="0 0.032 0.004" rpy="0 0 0" />
+        <parent link="${name}_link" />
+        <child link="${name}_depth_frame_aux"/>
+      </joint>
+      <link name="${name}_depth_frame_aux"/>
+      <joint name="${name}_depth_optical_joint_aux" type="fixed">
+        <origin xyz="0 0 0" rpy="${-M_PI/2} 0.0 ${-M_PI/2}" />
+        <parent link="${name}_depth_frame_aux" />
+        <child link="${name}_depth_optical_frame_aux"/>
+      </joint>
+      <link name="${name}_depth_optical_frame_aux"/>
       <joint name="${name}_rgb_joint" type="fixed">
-        <origin xyz="0.0 0.022 0.0" rpy="0 0 0" />
+        <origin xyz="0 -0.045 0.004" rpy="0 0 0" />
         <parent link="${name}_link" />
         <child link="${name}_rgb_frame"/>

Commit message: Remove frames as part of model as they are published based on internal intrinsics on real sensor

File: hector_sensors_description/urdf/realsense_camera.urdf.xacro (robot description, xacro)
@@ -1,3 +1,11 @@
 <?xml version="1.0"?>
+<!--
+Note:
+ The real sensor publshes tf data based on internally stored intrinsics. To support this, only the mounting link is
+ used in this macro. The corresponding frames can be added by running static_transform_publishers like so in the
+ Gazebo startup somewhere:
+  <node pkg="tf" type="static_transform_publisher" name="kinect_base_link" args="0 0 0 0 0 0  /arm_rgbd_cam_link /arm_rgbd_cam_depth_frame 100" />
+  <node pkg="tf" type="static_transform_publisher" name="kinect_base_link2" args="0 0 0 -1.57 0 -1.57 /arm_rgbd_cam_depth_frame /arm_rgbd_cam_depth_optical_frame  100" />
+-->
 <robot xmlns:xacro="http://www.ros.org/wiki/xacro">
     <xacro:property name="M_PI" value="3.1415926535897931" />
@@ -44,5 +52,5 @@
         </collision>
       </link>
-      <joint name="${name}_depth_joint" type="fixed">
+<!--      <joint name="${name}_depth_joint" type="fixed">
         <origin xyz="0 -0.051 0.004" rpy="0 0 0" />
         <parent link="${name}_link" />
@@ -73,5 +81,5 @@
         <child link="${name}_rgb_frame"/>
       </joint>
-      <link name="${name}_rgb_frame"/>
+      <link name="${name}_rgbd_cam_link"/>
       <joint name="${name}_rgb_optical_joint" type="fixed">
         <origin xyz="0 0 0" rpy="${-M_PI/2} 0.0 ${-M_PI/2}" />
@@ -79,5 +87,5 @@
         <child link="${name}_rgb_optical_frame"/>
       </joint>
-      <link name="${name}_rgb_optical_frame"/>
+      <link name="${name}_rgb_optical_frame"/>-->
       <gazebo reference="${name}_link">
         <material>Gazebo/Grey</material>
@@ -93,5 +101,5 @@
       </xacro:realsense_camera_model>
       <!-- ASUS Xtion PRO camera for simulation -->
-      <gazebo reference="${name}_depth_frame">
+      <gazebo reference="${name}_link">
         <sensor type="depth" name="${name}">
           <update_rate>20</update_rate>

Commit message: Move cam link to where real realsense driver expects it (rgb cam frame)

File: hector_sensors_description/urdf/realsense_camera.urdf.xacro (robot description, xacro)
@@ -27,5 +27,5 @@
         </inertial>
         <visual>
-          <origin xyz="0 0 0" rpy="0 0 0" />
+          <origin xyz="0 0.051 0" rpy="0 0 0" />
           <geometry>
             <!--Dimensions taken from https://software.intel.com/en-us/realsense/devkit-->
@@ -45,5 +45,5 @@
         -->
         <collision>
-          <origin xyz="0 0 0" rpy="0 0 0" />
+          <origin xyz="0 0.051 0" rpy="0 0 0" />
           <geometry>
             <!--Dimensions taken from https://software.intel.com/en-us/realsense/devkit-->

Commit message: Modify realsense r200 macro to also make version without geometry available

File: hector_sensors_description/urdf/realsense_camera.urdf.xacro (robot description, xacro)
@@ -11,5 +11,5 @@
     <xacro:property name="M_PI" value="3.1415926535897931" />
     <!--
-     The asus_camera_model macro only adds the model, it does not also add
+     This macro only adds the model, it does not also add
      the openni gazebo plugin. See the 'asus_camera' macro below for that
     -->
@@ -36,12 +36,4 @@
           </material>
         </visual>
-       <!--
-       <collision>
-          <origin xyz="0 0 0" rpy="0 0 0" />
-          <geometry>
-            <box size="0.035 0.185 0.025"/>
-          </geometry>
-        </collision>
-        -->
         <collision>
           <origin xyz="0 0.051 0" rpy="0 0 0" />
@@ -52,5 +44,6 @@
         </collision>
       </link>
-<!--      <joint name="${name}_depth_joint" type="fixed">
+      <!--
+      <joint name="${name}_depth_joint" type="fixed">
         <origin xyz="0 -0.051 0.004" rpy="0 0 0" />
         <parent link="${name}_link" />
@@ -87,18 +80,20 @@
         <child link="${name}_rgb_optical_frame"/>
       </joint>
-      <link name="${name}_rgb_optical_frame"/>-->
+      <link name="${name}_rgb_optical_frame"/>
+      -->
       <gazebo reference="${name}_link">
         <material>Gazebo/Grey</material>
       </gazebo>
     </xacro:macro>
-    <!--
-     The asus_camera macro only adds the model, and also adds
-     the openni gazebo plugin.
-    -->
-    <xacro:macro name="realsense_camera" params="name parent *origin">
-      <xacro:realsense_camera_model name="${name}" parent="${parent}">
+    <xacro:macro name="realsense_camera_model_no_geom" params="name parent *origin">
+      <joint name="${name}_joint" type="fixed">
         <xacro:insert_block name="origin" />
-      </xacro:realsense_camera_model>
-      <!-- ASUS Xtion PRO camera for simulation -->
+        <parent link="${parent}"/>
+        <child link="${name}_link"/>
+      </joint>
+      <link name="${name}_link">
+      </link>
+    </xacro:macro>
+    <xacro:macro name="realsense_camera_gazebo_plugin_macro" params="name parent">
       <gazebo reference="${name}_link">
         <sensor type="depth" name="${name}">
@@ -127,3 +122,22 @@
       </gazebo>
     </xacro:macro>
+    <!--
+      Use the macro below for adding the realsense model with link geometry
+    -->
+    <xacro:macro name="realsense_camera" params="name parent *origin">
+      <xacro:realsense_camera_model name="${name}" parent="${parent}">
+        <xacro:insert_block name="origin" />
+      </xacro:realsense_camera_model>
+      <xacro:realsense_camera_gazebo_plugin_macro name="${name}" parent="${parent}"/>
+    </xacro:macro>
+    <!--
+      Use the macro below for adding the realsense model without link geometry,
+      e.g. if the sensor is added into preexisting geometry
+    -->
+    <xacro:macro name="realsense_camera_no_geom" params="name parent *origin">
+      <xacro:realsense_camera_model_no_geom name="${name}" parent="${parent}">
+        <xacro:insert_block name="origin" />
+      </xacro:realsense_camera_model_no_geom>
+      <xacro:realsense_camera_gazebo_plugin_macro name="${name}" parent="${parent}"/>
+    </xacro:macro>
   </robot>

Commit message: explicitly added realsense optical link to urdf so it can be used for calibration (normally the link is only published in tf by the driver)

File: hector_sensors_description/urdf/realsense_camera.urdf.xacro (robot description, xacro)
@@ -69,17 +69,17 @@
       </joint>
       <link name="${name}_depth_optical_frame_aux"/>
+-->
       <joint name="${name}_rgb_joint" type="fixed">
-        <origin xyz="0 -0.045 0.004" rpy="0 0 0" />
+        <origin xyz="0 0 0" rpy="0 0 0" />
         <parent link="${name}_link" />
         <child link="${name}_rgb_frame"/>
       </joint>
-      <link name="${name}_rgbd_cam_link"/>
+      <link name="${name}_rgb_frame"/>
       <joint name="${name}_rgb_optical_joint" type="fixed">
-        <origin xyz="0 0 0" rpy="${-M_PI/2} 0.0 ${-M_PI/2}" />
+        <origin xyz="0 0 0" rpy="-1.571, 0.000, -1.571" />
         <parent link="${name}_rgb_frame" />
         <child link="${name}_rgb_optical_frame"/>
       </joint>
       <link name="${name}_rgb_optical_frame"/>
-      -->
       <gazebo reference="${name}_link">
         <material>Gazebo/Grey</material>
@@ -94,4 +94,16 @@
       <link name="${name}_link">
       </link>
+            <joint name="${name}_rgb_joint" type="fixed">
+        <origin xyz="0 0 0" rpy="0 0 0" />
+        <parent link="${name}_link" />
+        <child link="${name}_rgb_frame"/>
+      </joint>
+      <link name="${name}_rgb_frame"/>
+      <joint name="${name}_rgb_optical_joint" type="fixed">
+        <origin xyz="0 0 0" rpy="-1.571 0.000 -1.571" />
+        <parent link="${name}_rgb_frame" />
+        <child link="${name}_rgb_optical_frame"/>
+      </joint>
+      <link name="${name}_rgb_optical_frame"/>
     </xacro:macro>
     <xacro:macro name="realsense_camera_gazebo_plugin_macro" params="name parent">
@@ -107,5 +119,5 @@
             </image>
             <clip>
-              <near>0.5</near>
+              <near>0.1</near>
               <far>9</far>
             </clip>
@@ -117,5 +129,5 @@
             <depthImageCameraInfoTopicName>${name}/depth/camera_info</depthImageCameraInfoTopicName>
             <pointCloudTopicName>${name}/depth/points</pointCloudTopicName>
-            <frameName>${name}_depth_optical_frame</frameName>
+            <frameName>${name}_rgb_optical_frame</frameName>
           </plugin>
         </sensor>

Commit message: added missing frames to realsense macro

File: hector_sensors_description/urdf/realsense_camera.urdf.xacro (robot description, xacro)
@@ -94,4 +94,16 @@
       <link name="${name}_link">
       </link>
+      <joint name="${name}_rgb_joint" type="fixed">
+        <origin xyz="0 0 0" rpy="0 0 0" />
+        <parent link="${name}_link" />
+        <child link="${name}_rgb_frame"/>
+      </joint>
+      <link name="${name}_rgb_frame"/>
+      <joint name="${name}_rgb_optical_joint" type="fixed">
+        <origin xyz="0 0 0" rpy="${-M_PI/2} 0.0 ${-M_PI/2}" />
+        <parent link="${name}_rgb_frame" />
+        <child link="${name}_rgb_optical_frame"/>
+      </joint>
+      <link name="${name}_rgb_optical_frame"/>
     </xacro:macro>
     <xacro:macro name="realsense_camera_gazebo_plugin_macro" params="name parent">

Commit message: added missing depth links

File: hector_sensors_description/urdf/realsense_camera.urdf.xacro (robot description, xacro)
@@ -106,4 +106,16 @@
       </joint>
       <link name="${name}_rgb_optical_frame"/>
+      <joint name="${name}_depth_joint" type="fixed">
+        <origin xyz="0 0 0" rpy="0 0 0" />
+        <parent link="${name}_link" />
+        <child link="${name}_depth_frame"/>
+      </joint>
+      <link name="${name}_depth_frame"/>
+      <joint name="${name}_depth_optical_joint" type="fixed">
+        <origin xyz="0 0 0" rpy="${-M_PI/2} 0.0 ${-M_PI/2}" />
+        <parent link="${name}_depth_frame" />
+        <child link="${name}_depth_optical_frame"/>
+      </joint>
+      <link name="${name}_depth_optical_frame"/>
     </xacro:macro>
     <xacro:macro name="realsense_camera_gazebo_plugin_macro" params="name parent">

Commit message: Add optional macro for setting realsense topics

File: hector_sensors_description/urdf/realsense_camera.urdf.xacro (robot description, xacro)
@@ -95,8 +95,8 @@
       </link>
     </xacro:macro>
-    <xacro:macro name="realsense_camera_gazebo_plugin_macro" params="name parent">
+    <xacro:macro name="realsense_camera_gazebo_plugin_macro" params="name parent image_topic depth_points_topic min_range max_range update_rate">
       <gazebo reference="${name}_link">
         <sensor type="depth" name="${name}">
-          <update_rate>20</update_rate>
+          <update_rate>${update_rate}</update_rate>
           <camera>
             <horizontal_fov>${53.35 * M_PI/180.0}</horizontal_fov>
@@ -107,14 +107,14 @@
             </image>
             <clip>
-              <near>0.1</near>
-              <far>9</far>
+              <near>${min_range}</near>
+              <far>${max_range}</far>
             </clip>
           </camera>
           <plugin name="${name}_camera_controller" filename="libgazebo_ros_openni_kinect.so">
-            <imageTopicName>${name}/rgb/image_raw</imageTopicName>
+            <imageTopicName>${name}/${image_topic}</imageTopicName>
             <cameraInfoTopicName>${name}/rgb/camera_info</cameraInfoTopicName>
             <depthImageTopicName>${name}/depth/image_raw</depthImageTopicName>
             <depthImageCameraInfoTopicName>${name}/depth/camera_info</depthImageCameraInfoTopicName>
-            <pointCloudTopicName>${name}/depth/points</pointCloudTopicName>
+            <pointCloudTopicName>${name}/${depth_points_topic}</pointCloudTopicName>
             <frameName>${name}_depth_optical_frame</frameName>
           </plugin>
@@ -129,5 +129,5 @@
         <xacro:insert_block name="origin" />
       </xacro:realsense_camera_model>
-      <xacro:realsense_camera_gazebo_plugin_macro name="${name}" parent="${parent}"/>
+      <xacro:realsense_camera_gazebo_plugin_macro name="${name}" parent="${parent}" image_topic="rgb/image_raw" depth_points_topic="depth/points" min_range="0.3" max_range="9.0" update_rate="20"/>
     </xacro:macro>
     <!--
@@ -139,5 +139,11 @@
         <xacro:insert_block name="origin" />
       </xacro:realsense_camera_model_no_geom>
-      <xacro:realsense_camera_gazebo_plugin_macro name="${name}" parent="${parent}"/>
+      <xacro:realsense_camera_gazebo_plugin_macro name="${name}" parent="${parent}" image_topic="rgb/image_raw" depth_points_topic="depth/points" min_range="0.3" max_range="9.0" update_rate="20"/>
+    </xacro:macro>
+    <xacro:macro name="realsense_camera_no_geom_comprehensive_params" params="name parent *origin image_topic depth_points_topic min_range max_range update_rate">
+      <xacro:realsense_camera_model_no_geom name="${name}" parent="${parent}">
+        <xacro:insert_block name="origin" />
+      </xacro:realsense_camera_model_no_geom>
+      <xacro:realsense_camera_gazebo_plugin_macro name="${name}" parent="${parent}" image_topic="${image_topic}" depth_points_topic="${depth_points_topic}" min_range="${min_range}" max_range="${max_range}" update_rate="${update_rate}"/>
     </xacro:macro>
   </robot>

Commit message: making realsense blue

File: hector_sensors_description/urdf/realsense_camera.urdf.xacro (robot description, xacro)
@@ -89,5 +89,5 @@
       <link name="${name}_rgb_optical_frame"/>-->
       <gazebo reference="${name}_link">
-        <material>Gazebo/Grey</material>
+        <material>Gazebo/Blue</material>
       </gazebo>
     </xacro:macro>

Commit message: adding seperate color camera for realsense to stream high res color image

File: hector_sensors_description/urdf/realsense_camera.urdf.xacro (robot description, xacro)
@@ -9,5 +9,4 @@
 -->
 <robot xmlns:xacro="http://ros.org/wiki/xacro">
-    <xacro:property name="M_PI" value="3.1415926535897931" />
     <!--
      The asus_camera_model macro only adds the model, it does not also add
@@ -59,5 +58,5 @@
       <link name="${name}_depth_frame"/>
       <joint name="${name}_depth_optical_joint" type="fixed">
-        <origin xyz="0 0 0" rpy="${-M_PI/2} 0.0 ${-M_PI/2}" />
+        <origin xyz="0 0 0" rpy="${-pi/2} 0.0 ${-pi/2}" />
         <parent link="${name}_depth_frame" />
         <child link="${name}_depth_optical_frame"/>
@@ -71,5 +70,5 @@
       <link name="${name}_depth_frame_aux"/>
       <joint name="${name}_depth_optical_joint_aux" type="fixed">
-        <origin xyz="0 0 0" rpy="${-M_PI/2} 0.0 ${-M_PI/2}" />
+        <origin xyz="0 0 0" rpy="${-pi/2} 0.0 ${-pi/2}" />
         <parent link="${name}_depth_frame_aux" />
         <child link="${name}_depth_optical_frame_aux"/>
@@ -83,5 +82,5 @@
       <link name="${name}_rgbd_cam_link"/>
       <joint name="${name}_rgb_optical_joint" type="fixed">
-        <origin xyz="0 0 0" rpy="${-M_PI/2} 0.0 ${-M_PI/2}" />
+        <origin xyz="0 0 0" rpy="${-pi/2} 0.0 ${-pi/2}" />
         <parent link="${name}_rgb_frame" />
         <child link="${name}_rgb_optical_frame"/>
@@ -96,35 +95,65 @@
      the openni gazebo plugin.
     -->
-    <xacro:macro name="realsense_camera" params="name parent *origin">
-      <xacro:realsense_camera_model name="${name}" parent="${parent}">
-        <xacro:insert_block name="origin" />
-      </xacro:realsense_camera_model>
-      <!-- ASUS Xtion PRO camera for simulation -->
-      <gazebo reference="${name}_link">
-        <sensor type="depth" name="${name}">
-          <update_rate>20</update_rate>
-          <camera>
-            <horizontal_fov>${62.8 * M_PI/180.0}</horizontal_fov>
-            <image>
-              <format>R8G8B8</format>
-              <width>640</width>
-              <height>480</height>
-            </image>
-            <clip>
-              <near>0.5</near>
-              <far>9</far>
-            </clip>
-          </camera>
-          <plugin name="${name}_camera_controller" filename="libgazebo_ros_openni_kinect.so">
-            <robotNamespace>$(arg robot_name)/sensor/</robotNamespace>
-            <imageTopicName>${name}/rgb/image_raw</imageTopicName>
-            <cameraInfoTopicName>${name}/rgb/camera_info</cameraInfoTopicName>
-            <depthImageTopicName>${name}/depth/image_raw</depthImageTopicName>
-            <depthImageCameraInfoTopicName>${name}/depth/camera_info</depthImageCameraInfoTopicName>
-            <pointCloudTopicName>${name}/depth/points</pointCloudTopicName>
-            <frameName>${name}_depth_optical_frame</frameName>
-          </plugin>
-        </sensor>
-      </gazebo>
-    </xacro:macro>
-  </robot>
+  <xacro:macro name="realsense_camera" params="name parent *origin">
+    <xacro:realsense_camera_model name="${name}" parent="${parent}">
+      <xacro:insert_block name="origin" />
+    </xacro:realsense_camera_model>
+    <gazebo reference="${name}_link">
+      <sensor type="camera" name="${name}_color">
+        <always_on>1</always_on>
+        <update_rate>30</update_rate>
+        <visualize>true</visualize>
+        <camera>
+          <horizontal_fov>${70.0 * pi/180.0}</horizontal_fov>
+          <image>
+            <format>B8G8R8</format>
+            <width>1920</width>
+            <height>1080</height>
+          </image>
+          <clip>
+            <near>0.1</near>
+            <far>100</far>
+          </clip>
+          <distortion>
+            <k1>0.0</k1>
+            <k2>0.0</k2>
+            <k3>0.0</k3>
+            <p1>-0.0</p1>
+            <p2>-0.00</p2>
+            <center>0.5 0.5</center>
+          </distortion>
+        </camera>
+        <plugin name="${name}_camera_depth_controller" filename="libgazebo_ros_camera.so">
+          <robotNamespace>$(arg robot_name)/sensor/${name}/color</robotNamespace>
+          <imageTopicName>image_raw</imageTopicName>
+          <cameraInfoTopicName>camera_info</cameraInfoTopicName>
+          <frameName>${name}_color_optical_frame</frameName>
+        </plugin>
+      </sensor>
+      <sensor type="depth" name="${name}_depth">
+        <update_rate>20</update_rate>
+        <camera>
+          <horizontal_fov>${59.0 * pi/180.0}</horizontal_fov>
+          <image>
+            <format>B8G8R8</format>
+            <width>640</width>
+            <height>480</height>
+          </image>
+          <clip>
+            <near>0.5</near>
+            <far>10.0</far>
+          </clip>
+        </camera>
+        <plugin name="${name}_camera_rgb_controller" filename="libgazebo_ros_openni_kinect.so">
+          <robotNamespace>$(arg robot_name)/sensor/${name}</robotNamespace>
+          <imageTopicName>ir/image_raw</imageTopicName>
+          <cameraInfoTopicName>ir/camera_info</cameraInfoTopicName>
+          <depthImageTopicName>depth/image_raw</depthImageTopicName>
+          <depthImageCameraInfoTopicName>depth/camera_info</depthImageCameraInfoTopicName>
+          <pointCloudTopicName>depth/points</pointCloudTopicName>
+          <frameName>${name}_depth_optical_frame</frameName>
+        </plugin>
+      </sensor>
+    </gazebo>
+  </xacro:macro>
+</robot>

Commit message: Add macro for being able to set realsense params in more detail

File: hector_sensors_description/urdf/realsense_camera.urdf.xacro (robot description, xacro)
@@ -148,3 +148,9 @@
       <xacro:realsense_camera_gazebo_plugin_macro name="${name}" parent="${parent}" image_topic="${image_topic}" depth_points_topic="${depth_points_topic}" min_range="${min_range}" max_range="${max_range}" update_rate="${update_rate}"/>
     </xacro:macro>
+    <xacro:macro name="realsense_camera_comprehensive_params" params="name parent *origin image_topic depth_points_topic min_range max_range update_rate">
+      <xacro:realsense_camera_model name="${name}" parent="${parent}">
+        <xacro:insert_block name="origin" />
+      </xacro:realsense_camera_model>
+      <xacro:realsense_camera_gazebo_plugin_macro name="${name}" parent="${parent}" image_topic="${image_topic}" depth_points_topic="${depth_points_topic}" min_range="${min_range}" max_range="${max_range}" update_rate="${update_rate}"/>
+    </xacro:macro>
   </robot>
