Commit message: Make resolution params and set defaults for thermal cam

File: hector_sensors_description/urdf/generic_thermal_camera.urdf.xacro (robot description, xacro)
@@ -2,5 +2,5 @@
 <robot xmlns:xacro="http://ros.org/wiki/xacro">
   <xacro:include filename="$(find hector_xacro_tools)/urdf/sensor_macros.urdf.xacro" />
-  <xacro:macro name="generic_thermal_camera" params="name parent *origin">
+  <xacro:macro name="generic_thermal_camera" params="name parent resolution_x:=320 resolution_y:=256 *origin">
     <joint name="${name}_joint" type="fixed">
       <xacro:insert_block name="origin" />
@@ -9,17 +9,4 @@
     </joint>
     <link name="${name}_frame">
-      <!--        <xacro:inertial_sphere mass="0.01" diameter="0.07" />
-      <visual>
-      <origin xyz="0 0 0" rpy="0 0 0" />
-      <geometry>
-      <mesh filename="package://hector_sensors_description/meshes/thermaleye_camera/thermaleye_camera_hector_v2.dae"/>
-      </geometry>
-      </visual>
-      <collision>
-      <origin xyz="0 0 0" rpy="0 0 0" />
-      <geometry>
-      <mesh filename="package://hector_sensors_description/meshes/thermaleye_camera/thermaleye_camera_hector_v2.stl"/>
-      </geometry>
-      </collision>-->
     </link>
     <xacro:add_optical_frame name="${name}" />
@@ -31,6 +18,6 @@
           <image>
             <format>R8G8B8</format>
-            <width>320</width>
-            <height>256</height>
+            <width>${resolution_x}</width>
+            <height>${resolution_y}</height>
           </image>
           <clip>
