Commit message: renamed realsense t265 macros

File: hector_sensors_description/urdf/realsense_t265.urdf.xacro (robot description, xacro)
@@ -5,5 +5,5 @@
     <xacro:property name="realsense_t265_height" value="0.0245"/>
     <xacro:property name="realsense_t265_depth"  value="0.0125"/>
-    <xacro:macro name="realsense_t265_tracking_camera_housing" params="name parent *origin">
+    <xacro:macro name="realsense_t265_tracking_camera" params="name parent *origin">
       <joint name="${name}_housing_joint" type="fixed">
         <xacro:insert_block name="origin" />
@@ -53,9 +53,9 @@
         </visual>
       </link>
-      <xacro:realsense_t265_tracking_camera name="${name}" parent="${name}_housing_link">
+      <xacro:realsense_t265_tracking_camera_no_geom name="${name}" parent="${name}_housing_link">
         <origin xyz="-0.0003 0.0091 0" rpy="0 0 0" />
-      </xacro:realsense_t265_tracking_camera>
+      </xacro:realsense_t265_tracking_camera_no_geom>
     </xacro:macro>
-    <xacro:macro name="realsense_t265_tracking_camera" params="name parent *origin">
+    <xacro:macro name="realsense_t265_tracking_camera_no_geom" params="name parent *origin">
       <joint name="${name}_joint" type="fixed">
         <xacro:insert_block name="origin" />

Commit message: added t265 pose frame

File: hector_sensors_description/urdf/realsense_t265.urdf.xacro (robot description, xacro)
@@ -64,4 +64,10 @@
       </joint>
       <link name="${name}_link"/>
+      <joint name="${name}_pose_joint" type="fixed">
+        <xacro:insert_block name="origin" />
+        <parent link="${name}_link"/>
+        <child link="${name}_pose_frame"/>
+      </joint>
+      <link name="${name}_pose_frame"/>
     </xacro:macro>
   </robot>

Commit message: Revert "added t265 pose frame". Pose frame is published by driver in tf.
This reverts commit e11f9f1f9932411b386e5cf1d749a6e92a17d46c.

File: hector_sensors_description/urdf/realsense_t265.urdf.xacro (robot description, xacro)
@@ -64,10 +64,4 @@
       </joint>
       <link name="${name}_link"/>
-      <joint name="${name}_pose_joint" type="fixed">
-        <xacro:insert_block name="origin" />
-        <parent link="${name}_link"/>
-        <child link="${name}_pose_frame"/>
-      </joint>
-      <link name="${name}_pose_frame"/>
     </xacro:macro>
   </robot>

Commit message: renamed camera link to camera pose frame to match rs driver names

File: hector_sensors_description/urdf/realsense_t265.urdf.xacro (robot description, xacro)
@@ -58,10 +58,10 @@
     </xacro:macro>
     <xacro:macro name="realsense_t265_tracking_camera_no_geom" params="name parent *origin">
-      <joint name="${name}_joint" type="fixed">
+      <joint name="${name}_pose_joint" type="fixed">
         <xacro:insert_block name="origin" />
         <parent link="${parent}"/>
-        <child link="${name}_link"/>
+        <child link="${name}_pose_frame"/>
       </joint>
-      <link name="${name}_link"/>
+      <link name="${name}_pose_frame"/>
     </xacro:macro>
   </robot>

Commit message: added second tracking frame with the convention of the datasheet

File: hector_sensors_description/urdf/realsense_t265.urdf.xacro (robot description, xacro)
@@ -64,4 +64,10 @@
       </joint>
       <link name="${name}_pose_frame"/>
+      <joint name="${name}_pose_joint2" type="fixed">
+        <origin rpy="${M_PI/2} 0 ${-M_PI/2}"/>
+        <parent link="${name}_pose_frame"/>
+        <child link="${name}_pose_frame_alt"/>
+      </joint>
+      <link name="${name}_pose_frame_alt"/>
     </xacro:macro>
   </robot>
