Commit message: zoom cam mesh

File: hector_sensors_description/urdf/tis_zoom_cam.urdf.xacro (robot description, xacro)
@@ -18,5 +18,5 @@
       <visual>
         <geometry>
-          <box size="${tis_zoom_cam_housing_length} ${tis_zoom_cam_housing_width} ${tis_zoom_cam_housing_height}" />
+          <mesh filename="package://hector_sensors_description/meshes/tis_zoom_cam/zoom_cam_housing.stl" scale="1.0 1.0 1.0"/>
         </geometry>
         <material name="DarkGrey">
