Commit message: Changed tracker simulation topic and color

File: hector_sensors_description/urdf/vive_tracker.urdf.xacro (robot description, xacro)
@@ -19,6 +19,6 @@
           <mesh filename="package://hector_sensors_description/meshes/vive_tracker/tracker.stl"/>
         </geometry>
-        <material name="Blue">
-          <color rgba="0.0 0.0 0.8 1"/>
+        <material name="LightGray">
+          <color rgba="0.2 0.2 0.2 1"/>
         </material>
       </visual>
@@ -34,5 +34,5 @@
         <frameName>world</frameName>
         <bodyName>base_link</bodyName>
-        <topicName>/gazebo/$(arg robot_name)/tracker_odom</topicName>
+        <topicName>/tracker/odometry</topicName>
 	<updateRate>100.0</updateRate>
 	<!--gaussianNoise>0.0001</gaussianNoise-->

Commit message: Replaced vive tracker collision with bounding box and added color

File: hector_sensors_description/urdf/vive_tracker.urdf.xacro (robot description, xacro)
@@ -24,10 +24,13 @@
       </visual>
       <collision>
-        <origin xyz="0 0 0" rpy="0 0 0" />
+        <origin xyz="0 0.021144 -0.003673" rpy="0 0 0" />
         <geometry>
-          <mesh filename="package://hector_sensors_description/meshes/vive_tracker/tracker.stl"/>
+          <box size="0.0944 0.0423 0.0921"/> <!-- Bounding box extracted from STL -->
         </geometry>
       </collision>
     </link>
+    <gazebo reference="${name}_link">
+      <material>Gazebo/DarkGrey</material>
+    </gazebo>
     <gazebo>
       <plugin name="tracker_odom" filename="libgazebo_ros_p3d.so">
@@ -35,5 +38,5 @@
         <bodyName>base_link</bodyName>
         <topicName>/tracker/odometry</topicName>
-	<updateRate>100.0</updateRate>
+        <updateRate>100.0</updateRate>
 	<!--gaussianNoise>0.0001</gaussianNoise-->
       </plugin>

Commit message: Matching vive tracker color to gazebo color

File: hector_sensors_description/urdf/vive_tracker.urdf.xacro (robot description, xacro)
@@ -19,6 +19,6 @@
           <mesh filename="package://hector_sensors_description/meshes/vive_tracker/tracker.stl"/>
         </geometry>
-        <material name="LightGray">
-          <color rgba="0.2 0.2 0.2 1"/>
+        <material name="DarkGrey">
+          <color rgba="0.175 0.175 0.175 1"/>
         </material>
       </visual>
