Commit message: added sensor head collision geometry

File: hector_sensors_description/urdf/seek_thermal_compact.urdf.xacro (robot description, xacro)
@@ -33,4 +33,10 @@
         <material name="DarkGrey" />
       </visual>
+      <collision>
+        <origin xyz="0.0055 0 -0.013375" rpy="0 0 0" />
+        <geometry>
+          <box size="0.031 0.034 0.06075" />
+        </geometry>
+      </collision>
     </link>
     <xacro:add_optical_frame name="${name}" />

Commit message: removed collision size prop

File: hector_sensors_description/urdf/seek_thermal_compact.urdf.xacro (robot description, xacro)
@@ -39,10 +39,9 @@
         </geometry>
       </collision>
-      <xacro:property name="collision_size_factor" value="1"/>
       <xacro:if value="$(arg add_raycast_self_filter_geom)">
         <collision>
           <origin xyz="0.0055 0 -0.013375" rpy="0 0 0" />
           <geometry>
-            <cylinder length="${0.06075 * collision_size_factor}" radius="${0.023 * collision_size_factor}"/>
+            <cylinder length="0.06075" radius="0.023"/>
           </geometry>
         </collision>

Commit message: added a seek thermal macro without geometry

File: hector_sensors_description/urdf/seek_thermal_compact.urdf.xacro (robot description, xacro)
@@ -2,5 +2,5 @@
 <robot xmlns:xacro="http://ros.org/wiki/xacro">
   <xacro:include filename="$(find hector_xacro_tools)/urdf/sensor_macros.urdf.xacro" />
-  <xacro:macro name="seek_thermal_compact_camera_model" params="name parent *origin">
+  <xacro:macro name="seek_thermal_compact_camera_model" params="name parent *origin add_geometry">
     <joint name="${name}_joint" type="fixed">
       <xacro:insert_block name="origin" />
@@ -10,40 +10,42 @@
     <link name="${name}_frame">
       <xacro:inertial_sphere mass="0.03" diameter="0.02" />
-      <visual>
-        <origin xyz="0 0.0 -0.025" rpy="0 0 0" />
-        <geometry>
-          <box size="0.02 0.03 0.0375" />
-        </geometry>
-        <material name="DarkGrey">
-          <color rgba="0.3 0.3 0.3 1" />
-        </material>
-      </visual>
-      <visual>
-        <origin xyz="0 0 0" rpy="0 ${M_PI/2} 0" />
-        <geometry>
-          <cylinder length="0.02" radius="0.017" />
-        </geometry>
-        <material name="DarkGrey" />
-      </visual>
-      <visual>
-        <origin xyz="0.01 0 0" rpy="0 ${M_PI/2} 0" />
-        <geometry>
-          <cylinder length="0.018" radius="0.011" />
-        </geometry>
-        <material name="DarkGrey" />
-      </visual>
-      <collision>
-        <origin xyz="0.0055 0 -0.013375" rpy="0 0 0" />
-        <geometry>
-          <box size="0.031 0.034 0.06075" />
-        </geometry>
-      </collision>
-      <xacro:if value="$(arg add_raycast_self_filter_geom)">
+      <xacro:if value="${add_geometry}">
+        <visual>
+            <origin xyz="0 0.0 -0.025" rpy="0 0 0" />
+            <geometry>
+            <box size="0.02 0.03 0.0375" />
+            </geometry>
+            <material name="DarkGrey">
+            <color rgba="0.3 0.3 0.3 1" />
+            </material>
+        </visual>
+        <visual>
+            <origin xyz="0 0 0" rpy="0 ${M_PI/2} 0" />
+            <geometry>
+            <cylinder length="0.02" radius="0.017" />
+            </geometry>
+            <material name="DarkGrey" />
+        </visual>
+        <visual>
+            <origin xyz="0.01 0 0" rpy="0 ${M_PI/2} 0" />
+            <geometry>
+            <cylinder length="0.018" radius="0.011" />
+            </geometry>
+            <material name="DarkGrey" />
+        </visual>
         <collision>
-          <origin xyz="0.0055 0 -0.013375" rpy="0 0 0" />
-          <geometry>
-            <cylinder length="0.06075" radius="0.023"/>
-          </geometry>
+            <origin xyz="0.0055 0 -0.013375" rpy="0 0 0" />
+            <geometry>
+            <box size="0.031 0.034 0.06075" />
+            </geometry>
         </collision>
+        <xacro:if value="$(arg add_raycast_self_filter_geom)">
+            <collision>
+            <origin xyz="0.0055 0 -0.013375" rpy="0 0 0" />
+            <geometry>
+                <cylinder length="0.06075" radius="0.023"/>
+            </geometry>
+            </collision>
+        </xacro:if>
       </xacro:if>
     </link>
@@ -53,8 +55,5 @@
     </gazebo>
   </xacro:macro>
-  <xacro:macro name="seek_thermal_compact_camera" params="name parent *origin">
-    <xacro:seek_thermal_compact_camera_model name="${name}" parent="${parent}">
-      <xacro:insert_block name="origin" />
-    </xacro:seek_thermal_compact_camera_model>
+  <xacro:macro name="seek_thermal_compact_gazebo_plugin_macro" params="name parent *origin">
     <gazebo reference="${name}_frame">
       <sensor type="camera" name="thermal_camera_sensor">
@@ -83,3 +82,25 @@
     </gazebo>
   </xacro:macro>
+  <xacro:macro name="seek_thermal_compact_camera" params="name parent *origin">
+    <xacro:seek_thermal_compact_camera_model name="${name}" parent="${parent}" add_geometry="true">
+      <xacro:insert_block name="origin" />
+    </xacro:seek_thermal_compact_camera_model>
+    <xacro:seek_thermal_compact_gazebo_plugin_macro name="${name}" parent="${parent}">
+      <xacro:insert_block name="origin" />
+    </xacro:seek_thermal_compact_gazebo_plugin_macro>
+  </xacro:macro>
+  <xacro:macro name="seek_thermal_compact_camera_no_geom" params="name parent *origin">
+    <xacro:seek_thermal_compact_camera_model name="${name}" parent="${parent}" add_geometry="false">
+      <xacro:insert_block name="origin" />
+    </xacro:seek_thermal_compact_camera_model>
+    <xacro:seek_thermal_compact_gazebo_plugin_macro name="${name}" parent="${parent}">
+      <xacro:insert_block name="origin" />
+    </xacro:seek_thermal_compact_gazebo_plugin_macro>
+  </xacro:macro>
+  <xacro:macro name="realsense_camera_no_geom" params="name parent *origin">
+    <xacro:realsense_d435_camera_model_no_geom name="${name}" parent="${parent}">
+      <xacro:insert_block name="origin" />
+    </xacro:realsense_d435_camera_model_no_geom>
+    <xacro:seek_thermal_compact_gazebo_plugin_macro name="${name}" parent="${parent}" image_topic="image_raw" depth_points_topic="depth/points" min_range="0.3" max_range="9.0" update_rate="20"/>
+    </xacro:macro>
 </robot>

Commit message: cleanup

File: hector_sensors_description/urdf/seek_thermal_compact.urdf.xacro (robot description, xacro)
@@ -98,9 +98,3 @@
     </xacro:seek_thermal_compact_gazebo_plugin_macro>
   </xacro:macro>
-  <xacro:macro name="realsense_camera_no_geom" params="name parent *origin">
-    <xacro:realsense_d435_camera_model_no_geom name="${name}" parent="${parent}">
-      <xacro:insert_block name="origin" />
-    </xacro:realsense_d435_camera_model_no_geom>
-    <xacro:seek_thermal_compact_gazebo_plugin_macro name="${name}" parent="${parent}" image_topic="image_raw" depth_points_topic="depth/points" min_range="0.3" max_range="9.0" update_rate="20"/>
-    </xacro:macro>
 </robot>

Commit message: optimized the XM430 sensor head urdf

File: hector_sensors_description/urdf/seek_thermal_compact.urdf.xacro (robot description, xacro)
@@ -52,5 +52,5 @@
     <xacro:add_optical_frame name="${name}" />
     <gazebo reference="${name}_frame">
-      <material>Gazebo/Grey</material>
+      <material>Gazebo/DarkGrey</material>
     </gazebo>
   </xacro:macro>
