Commit message: Added collision geometries for the automess geiger counter

File: hector_sensors_description/urdf/automess_geiger_counter.urdf.xacro (robot description, xacro)
@@ -1,20 +1,25 @@
 <?xml version="1.0" encoding="UTF-8"?>
 <robot xmlns:xacro="http://www.ros.org/wiki/xacro">
+  <xacro:property name="automess_geometry">
+    <geometry>
+      <box size="0.1385 0.0885 0.037"/>
+    </geometry>
+  </xacro:property>
   <xacro:macro name="automess_geiger_counter" params="name parent *origin">
     <joint name="${name}_joint" type="fixed">
-      <xacro:insert_block name="origin" />
-      <parent link="${parent}" />
-      <child link="${name}_frame" />
+      <xacro:insert_block name="origin"/>
+      <parent link="${parent}"/>
+      <child link="${name}_frame"/>
     </joint>
     <link name="${name}_frame">
-        <visual>
-            <origin xyz="0 0 0" rpy="0 0 0" />
-            <geometry>
-            <box size="0.1385 0.0885 0.037" />
-            </geometry>
-            <material name="DarkGrey">
-            <color rgba="0.3 0.3 0.3 1" />
-            </material>
-        </visual>
+      <visual>
+        <xacro:insert_block name="automess_geometry"/>
+        <material name="DarkGrey">
+          <color rgba="0.3 0.3 0.3 1"/>
+        </material>
+      </visual>
+      <collision>
+        <xacro:insert_block name="automess_geometry"/>
+      </collision>
     </link>
   </xacro:macro>

Commit message: replaced the appended frame by link for the automess sensor

File: hector_sensors_description/urdf/automess_geiger_counter.urdf.xacro (robot description, xacro)
@@ -10,7 +10,7 @@
       <xacro:insert_block name="origin"/>
       <parent link="${parent}"/>
-      <child link="${name}_frame"/>
+      <child link="${name}_link"/>
     </joint>
-    <link name="${name}_frame">
+    <link name="${name}_link">
       <visual>
         <xacro:insert_block name="automess_geometry"/>
