Commit message: Add gazebo material for flir and realsense models

File: hector_sensors_description/urdf/flir_a35_camera.urdf.xacro (robot description, xacro)
@@ -29,4 +29,7 @@
     </link>
     <xacro:add_optical_frame name="${name}" />
+    <gazebo reference="${name}_frame">
+      <material>Gazebo/Grey</material>
+    </gazebo>
   </xacro:macro>
 </robot>

File: hector_sensors_description/urdf/realsense_camera.urdf.xacro (robot description, xacro)
@@ -68,4 +68,7 @@
       </joint>
       <link name="${name}_rgb_optical_frame"/>
+      <gazebo reference="${name}_link">
+        <material>Gazebo/Grey</material>
+      </gazebo>
     </xacro:macro>
     <!--

Commit message: Update flir a35 camera macro

File: hector_sensors_description/urdf/flir_a35_camera.urdf.xacro (robot description, xacro)
@@ -33,3 +33,32 @@
     </gazebo>
   </xacro:macro>
+  <xacro:macro name="flir_a35_camera" params="name parent *origin">
+    <xacro:flir_a35_camera_model name="${name}" parent="${parent}">
+      <xacro:insert_block name="origin" />
+    </xacro:flir_a35_camera_model>
+    <gazebo reference="${name}_frame">
+      <sensor type="camera" name="thermal_camera_sensor">
+        <update_rate>10</update_rate>
+        <camera>
+          <horizontal_fov>${90.0*M_PI/180.0}</horizontal_fov>
+          <image>
+            <format>R8G8B8</format>
+            <width>320</width>
+            <height>240</height>
+          </image>
+          <clip>
+            <near>0.01</near>
+            <far>10</far>
+          </clip>
+        </camera>
+        <plugin name="thermal_camera_controller" filename="libgazebo_ros_thermal_camera.so">
+          <alwaysOn>true</alwaysOn>
+          <updateRate>10</updateRate>
+          <imageTopicName>/${name}/image</imageTopicName>
+          <cameraInfoTopicName>/${name}/camera_info</cameraInfoTopicName>
+          <frameName>${name}_optical_frame</frameName>
+        </plugin>
+      </sensor>
+    </gazebo>
+  </xacro:macro>
 </robot>

Commit message: flir housing mesh

File: hector_sensors_description/urdf/flir_a35_camera.urdf.xacro (robot description, xacro)
@@ -2,4 +2,5 @@
 <robot xmlns:xacro="http://www.ros.org/wiki/xacro">
   <xacro:include filename="$(find hector_xacro_tools)/urdf/sensor_macros.urdf.xacro" />
+  <!--Dimensions taken from http://www.flir.com/automation/display/?id=56341-->
   <xacro:macro name="flir_a35_camera_model" params="name parent *origin">
     <joint name="${name}_joint" type="fixed">
@@ -11,8 +12,8 @@
       <xacro:inertial_sphere mass="0.01" diameter="0.07" />
       <visual>
-        <origin xyz="${0.106*-0.5} 0 0" rpy="0 0 0" />
+        <origin xyz="${0.072*-0.5 - 0.0184} 0 0" rpy="0 0 0" />
         <geometry>
-          <!--Dimensions taken from http://www.flir.com/automation/display/?id=56341-->
-          <box size="0.106 0.04 0.043" />
+          <!-- Rear cap: 13.7mm, front cap: 18.4, body length: 72mm, body width: 40mm, body height: 43mm -->
+          <mesh filename="package://hector_sensors_description/meshes/flir_a35_camera/flir_a35_housing.stl" scale="1.0 1.0 1.0"/>
         </geometry>
         <material name="DarkGrey">
@@ -21,8 +22,7 @@
       </visual>
       <collision>
-        <origin xyz="${0.106*-0.5} 0 0" rpy="0 0 0" />
+        <origin xyz="${0.1041*-0.5} 0 0" rpy="0 0 0" />
         <geometry>
-          <!--Dimensions taken from http://www.flir.com/automation/display/?id=56341-->
-          <box size="0.106 0.04 0.043" />
+          <box size="0.1041 0.04 0.043" />
         </geometry>
       </collision>

Commit message: Adjust cam macros for A35 and TIS zoom to follow consistent convention (origin is in optical center) Switch tis cam to use z20 dimensions

File: hector_sensors_description/urdf/flir_a35_camera.urdf.xacro (robot description, xacro)
@@ -12,5 +12,5 @@
       <xacro:inertial_sphere mass="0.01" diameter="0.07" />
       <visual>
-        <origin xyz="${0.072*-0.5 - 0.0184} 0 0" rpy="0 0 0" />
+        <origin xyz="${0.072*-0.5 - 0.0184 + 0.025} 0 0" rpy="0 0 0" />
         <geometry>
           <!-- Rear cap: 13.7mm, front cap: 18.4, body length: 72mm, body width: 40mm, body height: 43mm -->
@@ -22,5 +22,5 @@
       </visual>
       <collision>
-        <origin xyz="${0.1041*-0.5} 0 0" rpy="0 0 0" />
+        <origin xyz="${0.1041*-0.5 + 0.025} 0 0" rpy="0 0 0" />
         <geometry>
           <box size="0.1041 0.04 0.043" />

File: hector_sensors_description/urdf/tis_zoom_cam.urdf.xacro (robot description, xacro)
@@ -5,7 +5,7 @@
   <xacro:include filename="$(find hector_sensors_description)/urdf/generic_camera.urdf.xacro" />
   <!-- Dimensions from https://s1-dl.theimagingsource.com/api/2.5/packages/documentation/factsheets-single/fsdfkz30gp031/5e87e13f-c891-50c8-93c1-7bffd94642a1/fsdfkz30gp031.de_DE.pdf -->
-  <xacro:property name="tis_zoom_cam_housing_width" value="0.0606" />
-  <xacro:property name="tis_zoom_cam_housing_height" value="0.0606" />
-  <xacro:property name="tis_zoom_cam_housing_length" value="0.117" />
+  <xacro:property name="tis_zoom_cam_housing_width" value="0.071" />
+  <xacro:property name="tis_zoom_cam_housing_height" value="0.071" />
+  <xacro:property name="tis_zoom_cam_housing_length" value="0.147" />
   <xacro:macro name="tis_zoom_camera_model" params="name parent *origin">
     <joint name="${name}_mount_joint" type="fixed">
@@ -17,6 +17,7 @@
       <xacro:inertial_cuboid mass="0.02" x_length="0.0285" y_length="0.07" z_length="0.034"/>
       <visual>
+        <origin xyz="-0.06 0 0.0" rpy="0 0 0" />
         <geometry>
-          <mesh filename="package://hector_sensors_description/meshes/tis_zoom_cam/zoom_cam_housing.stl" scale="1.0 1.0 1.0"/>
+          <mesh filename="package://hector_sensors_description/meshes/tis_zoom_cam/zoom_cam_housing.stl" scale="1.1716 1.1716 1.2564"/>
         </geometry>
         <material name="DarkGrey">
@@ -25,4 +26,5 @@
       </visual>
       <collision>
+        <origin xyz="-0.06 0 0.0" rpy="0 0 0" />
         <geometry>
           <box size="${tis_zoom_cam_housing_length} ${tis_zoom_cam_housing_width} ${tis_zoom_cam_housing_height}" />
