Commit message: Update VLP16 macro to provide normal and advanced versions

File: hector_sensors_description/urdf/vlp16.urdf.xacro (robot description, xacro)
@@ -24,5 +24,10 @@
       </link>
     </xacro:macro>
-    <xacro:macro name="vlp16" params="name parent *origin ros_topic update_rate ray_count min_angle max_angle">
+    <xacro:macro name="vlp16" params="name parent *origin ros_topic">
+      <xacro:vlp16_advanced_parameters name="${name}" parent="${parent}" ros_topic="${ros_topic}" update_rate="10" horizontal_samples="512" vertical_samples="8" min_range="0.45" max_range="100">
+        <xacro:insert_block name="origin" />
+      </xacro:vlp16_advanced_parameters>
+    </xacro:macro>
+    <xacro:macro name="vlp16_advanced_parameters" params="name parent *origin ros_topic update_rate horizontal_samples vertical_samples min_range max_range">
       <xacro:vlp16_model name="${name}" parent="${parent}">
         <xacro:insert_block name="origin" />
@@ -59,12 +64,12 @@
           </plugin>
         </sensor>-->
-              <sensor type="ray" name="${name}-VLP16">
+      <sensor type="ray" name="${name}-VLP16">
         <pose>0 0 0 0 0 0</pose>
         <visualize>false</visualize>
-        <update_rate>10</update_rate>
+        <update_rate>${update_rate}</update_rate>
         <ray>
           <scan>
             <horizontal>
-              <samples>512</samples>
+              <samples>${horizontal_samples}</samples>
               <resolution>1</resolution>
               <min_angle>-${M_PI}</min_angle>
@@ -72,5 +77,5 @@
             </horizontal>
             <vertical>
-              <samples>8</samples>
+              <samples>${vertical_samples}</samples>
               <resolution>1</resolution>
               <min_angle>-${15.0*M_PI/180.0}</min_angle>
@@ -79,6 +84,6 @@
           </scan>
           <range>
-            <min>0.2</min>
-            <max>140.0</max>
+            <min>${min_range}</min>
+            <max>${max_range}</max>
             <resolution>0.001</resolution>
           </range>
@@ -92,6 +97,6 @@
           <topicName>${ros_topic}</topicName>
           <frameName>${name}_frame</frameName>
-          <min_range>0.45</min_range>
-          <max_range>130.0</max_range>
+          <min_range>${min_range}</min_range>
+          <max_range>${max_range}</max_range>
           <gaussianNoise>0.008</gaussianNoise>
         </plugin>

Commit message: added high res visuals for vlp16

File: hector_sensors_description/urdf/vlp16.urdf.xacro (robot description, xacro)
@@ -9,9 +9,22 @@
       </joint>
       <link name="${name}_frame">
-        <xacro:inertial_sphere mass="0.8" diameter="0.1033" />
-        <visual>        -->
-          <origin rpy="0 0 0" xyz="0 0 0.0018500"/>
+        <xacro:inertial_sphere mass="0.83" diameter="0.1033" />
+        <!-- Visual geometry by velodyne_simulator https://bitbucket.org/DataspeedInc/velodyne_simulator -->
+        <visual>
+          <origin xyz="0 0 -0.0377" />
           <geometry>
-            <cylinder radius="0.0516" length="0.0717"/>
+            <mesh filename="package://hector_sensors_description/meshes/vlp16/VLP16_base_1.dae" />
+          </geometry>
+        </visual>
+        <visual>
+          <origin xyz="0 0 -0.0377" />
+          <geometry>
+            <mesh filename="package://hector_sensors_description/meshes/vlp16/VLP16_base_2.dae" />
+          </geometry>
+        </visual>
+        <visual>
+          <origin xyz="0 0 -0.0377" />
+          <geometry>
+            <mesh filename="package://hector_sensors_description/meshes/vlp16/VLP16_scan.dae" />
           </geometry>
         </visual>

Commit message: unified the GPU and non-GPU VLP16 xacro macro

File: hector_sensors_description/urdf/vlp16.urdf.xacro (robot description, xacro)
@@ -1,80 +1,58 @@
 <?xml version="1.0"?>
 <robot xmlns:xacro="http://www.ros.org/wiki/xacro">
-    <xacro:property name="M_PI" value="3.1415926535897931" />
-    <xacro:macro name="vlp16_model" params="name parent *origin">
-      <joint name="${name}_joint" type="fixed">
-        <xacro:insert_block name="origin" />
-        <parent link="${parent}"/>
-        <child link="${name}_frame"/>
-      </joint>
-      <link name="${name}_frame">
-        <xacro:inertial_sphere mass="0.83" diameter="0.1033" />
-        <visual>
-          <origin xyz="0 0 -0.0378" rpy="${M_PI/2} 0 ${M_PI}" />
-          <geometry>
-            <mesh filename="package://hector_sensors_description/meshes/vlp16/VLP16_base_1.dae" scale="0.001 0.001 0.001"/>
-          </geometry>
-        </visual>
-        <visual>
-          <origin xyz="0 0 -0.0378" rpy="${M_PI/2} 0 ${M_PI}" />
-          <geometry>
-            <mesh filename="package://hector_sensors_description/meshes/vlp16/VLP16_base_2.dae" scale="0.001 0.001 0.001"/>
-          </geometry>
-        </visual>
-        <visual>
-          <origin xyz="0 0 -0.0378" rpy="${M_PI/2} 0 ${M_PI}" />
-          <geometry>
-            <mesh filename="package://hector_sensors_description/meshes/vlp16/VLP16_scan.dae" scale="0.001 0.001 0.001"/>
-          </geometry>
-        </visual>
-        <collision>
-          <origin rpy="0 0 0" xyz="0 0 -0.00225"/>
-          <geometry>
-            <cylinder radius="0.0516" length="0.0717"/>
-          </geometry>
-        </collision>
-      </link>
-    </xacro:macro>
-    <xacro:macro name="vlp16" params="name parent *origin ros_topic">
-      <xacro:vlp16_advanced_parameters name="${name}" parent="${parent}" ros_topic="${ros_topic}" update_rate="10" horizontal_samples="512" vertical_samples="8" min_range="0.45" max_range="100">
-        <xacro:insert_block name="origin" />
-      </xacro:vlp16_advanced_parameters>
-    </xacro:macro>
-    <xacro:macro name="vlp16_advanced_parameters" params="name parent *origin ros_topic update_rate horizontal_samples vertical_samples min_range max_range">
-      <xacro:vlp16_model name="${name}" parent="${parent}">
-        <xacro:insert_block name="origin" />
-      </xacro:vlp16_model>
-      <gazebo reference="${name}_frame">
-<!--        <sensor type="ray" name="${name}">
-          <always_on>true</always_on>
-          <update_rate>${update_rate}</update_rate>
-          <pose>0 0 0 0 0 0</pose>
-          <visualize>false</visualize>
-          <ray>
-            <scan>
-              <horizontal>
-                <samples>${ray_count}</samples>
-                <resolution>1</resolution>
-                <min_angle>${min_angle * M_PI/180}</min_angle>
-                <max_angle>${max_angle * M_PI/180}</max_angle>
-              </horizontal>
-            </scan>
-            <range>
-              <min>0.2</min>
-              <max>30.0</max>
-              <resolution>0.01</resolution>
-            </range>
-            <noise>
-              <type>gaussian</type>
-              <mean>0.0</mean>
-              <stddev>0.004</stddev>
-            </noise>
-          </ray>
-          <plugin name="gazebo_ros_${name}_controller" filename="libgazebo_ros_laser.so">
-            <topicName>${ros_topic}</topicName>
-            <frameName>${name}_frame</frameName>
-          </plugin>
-        </sensor>-->
-      <sensor type="ray" name="${name}-VLP16">
+  <xacro:property name="M_PI" value="3.1415926535897931"/>
+  <xacro:macro name="vlp16_model" params="name parent *origin">
+    <joint name="${name}_joint" type="fixed">
+      <xacro:insert_block name="origin"/>
+      <parent link="${parent}"/>
+      <child link="${name}_frame"/>
+    </joint>
+    <link name="${name}_frame">
+      <xacro:inertial_sphere mass="0.83" diameter="0.1033"/>
+      <visual>
+        <origin xyz="0 0 -0.0378" rpy="${M_PI/2} 0 ${M_PI}"/>
+        <geometry>
+          <mesh filename="package://hector_sensors_description/meshes/vlp16/VLP16_base_1.dae" scale="0.001 0.001 0.001"/>
+        </geometry>
+      </visual>
+      <visual>
+        <origin xyz="0 0 -0.0378" rpy="${M_PI/2} 0 ${M_PI}"/>
+        <geometry>
+          <mesh filename="package://hector_sensors_description/meshes/vlp16/VLP16_base_2.dae" scale="0.001 0.001 0.001"/>
+        </geometry>
+      </visual>
+      <visual>
+        <origin xyz="0 0 -0.0378" rpy="${M_PI/2} 0 ${M_PI}"/>
+        <geometry>
+          <mesh filename="package://hector_sensors_description/meshes/vlp16/VLP16_scan.dae" scale="0.001 0.001 0.001"/>
+        </geometry>
+      </visual>
+      <collision>
+        <origin rpy="0 0 0" xyz="0 0 -0.00225"/>
+        <geometry>
+          <cylinder radius="0.0516" length="0.0717"/>
+        </geometry>
+      </collision>
+    </link>
+  </xacro:macro>
+  <xacro:macro name="vlp16" params="name parent *origin ros_topic">
+    <xacro:vlp16_advanced_parameters name="${name}" parent="${parent}" ros_topic="${ros_topic}" update_rate="10" horizontal_samples="512" vertical_samples="8" min_range="0.45" max_range="100">
+      <xacro:insert_block name="origin"/>
+    </xacro:vlp16_advanced_parameters>
+  </xacro:macro>
+  <xacro:macro name="vlp16_advanced_parameters" params="name parent *origin ros_topic update_rate horizontal_samples vertical_samples min_range max_range use_gpu:='false'">
+    <xacro:vlp16_model name="${name}" parent="${parent}">
+      <xacro:insert_block name="origin"/>
+    </xacro:vlp16_model>
+    <gazebo reference="${name}_frame">
+      <xacro:if value="${use_gpu}">
+        <xacro:property name="sensor_type" value="gpu_ray"/>
+        <xacro:property name="gazebo_plugin_name" value="libgazebo_ros_velodyne_gpu_laser.so"/>
+      </xacro:if >
+      <xacro:unless value="${use_gpu}">
+        <xacro:property name="sensor_type" value="ray"/>
+        <xacro:property name="gazebo_plugin_name" value="libgazebo_ros_velodyne_laser.so"/>
+      </xacro:unless>
+      <sensor type="${sensor_type}" name="${name}-VLP16">
         <pose>0 0 0 0 0 0</pose>
         <visualize>false</visualize>
@@ -86,5 +64,5 @@
               <resolution>1</resolution>
               <min_angle>-${M_PI}</min_angle>
-              <max_angle> ${M_PI}</max_angle>
+              <max_angle>${M_PI}</max_angle>
             </horizontal>
             <vertical>
@@ -92,5 +70,5 @@
               <resolution>1</resolution>
               <min_angle>-${15.0*M_PI/180.0}</min_angle>
-              <max_angle> ${15.0*M_PI/180.0}</max_angle>
+              <max_angle>${15.0*M_PI/180.0}</max_angle>
             </vertical>
           </scan>
@@ -106,5 +84,5 @@
           </noise>
         </ray>
-        <plugin name="gazebo_ros_laser_controller" filename="libgazebo_ros_velodyne_laser.so">
+        <plugin name="gazebo_ros_laser_controller" filename="${gazebo_plugin_name}">
           <topicName>${ros_topic}</topicName>
           <frameName>${name}_frame</frameName>
@@ -114,41 +92,5 @@
         </plugin>
       </sensor>
-      </gazebo>
-    </xacro:macro>
-    <xacro:macro name="vlp16_gpu" params="name parent *origin ros_topic update_rate ray_count min_angle max_angle">
-      <xacro:vlp16_model name="${name}" parent="${parent}">
-        <xacro:insert_block name="origin" />
-      </xacro:vlp16_model>
-      <gazebo reference="${name}_frame">
-        <sensor type="gpu_ray" name="${name}">
-          <update_rate>${update_rate}</update_rate>
-          <pose>0 0 0 0 0 0</pose>
-          <visualize>false</visualize>
-          <ray>
-            <scan>
-              <horizontal>
-                <samples>${ray_count}</samples>
-                <resolution>1</resolution>
-                <min_angle>${min_angle * M_PI/180}</min_angle>
-                <max_angle>${max_angle * M_PI/180}</max_angle>
-              </horizontal>
-            </scan>
-            <range>
-              <min>0.2</min>
-              <max>30.0</max>
-              <resolution>0.01</resolution>
-            </range>
-            <noise>
-              <type>gaussian</type>
-              <mean>0.0</mean>
-              <stddev>0.004</stddev>
-            </noise>
-          </ray>
-          <plugin name="gazebo_ros_${name}_controller" filename="libgazebo_ros_gpu_laser.so">
-            <topicName>${ros_topic}</topicName>
-            <frameName>${name}_frame</frameName>
-          </plugin>
-        </sensor>
-      </gazebo>
-    </xacro:macro>
+    </gazebo>
+  </xacro:macro>
 </robot>

Commit message: Use xacro param defaulting to false to optionally organize vlp16 points

File: hector_sensors_description/urdf/vlp16.urdf.xacro (robot description, xacro)
@@ -43,39 +43,9 @@
       </xacro:vlp16_advanced_parameters>
     </xacro:macro>
-    <xacro:macro name="vlp16_advanced_parameters" params="name parent *origin ros_topic update_rate horizontal_samples vertical_samples min_range max_range">
+    <xacro:macro name="vlp16_advanced_parameters" params="name parent *origin ros_topic update_rate horizontal_samples vertical_samples min_range max_range organize_cloud:=false">
       <xacro:vlp16_model name="${name}" parent="${parent}">
         <xacro:insert_block name="origin" />
       </xacro:vlp16_model>
       <gazebo reference="${name}_frame">
-<!--        <sensor type="ray" name="${name}">
-          <always_on>true</always_on>
-          <update_rate>${update_rate}</update_rate>
-          <pose>0 0 0 0 0 0</pose>
-          <visualize>false</visualize>
-          <ray>
-            <scan>
-              <horizontal>
-                <samples>${ray_count}</samples>
-                <resolution>1</resolution>
-                <min_angle>${min_angle * M_PI/180}</min_angle>
-                <max_angle>${max_angle * M_PI/180}</max_angle>
-              </horizontal>
-            </scan>
-            <range>
-              <min>0.2</min>
-              <max>30.0</max>
-              <resolution>0.01</resolution>
-            </range>
-            <noise>
-              <type>gaussian</type>
-              <mean>0.0</mean>
-              <stddev>0.004</stddev>
-            </noise>
-          </ray>
-          <plugin name="gazebo_ros_${name}_controller" filename="libgazebo_ros_laser.so">
-            <topicName>${ros_topic}</topicName>
-            <frameName>${name}_frame</frameName>
-          </plugin>
-        </sensor>-->
       <sensor type="ray" name="${name}-VLP16">
         <pose>0 0 0 0 0 0</pose>
@@ -111,4 +81,5 @@
           <topicName>${ros_topic}</topicName>
           <frameName>${name}_frame</frameName>
+          <organize_cloud>${organize_cloud}</organize_cloud>
           <min_range>${min_range}</min_range>
           <max_range>${max_range}</max_range>
@@ -118,5 +89,5 @@
       </gazebo>
     </xacro:macro>
-    <xacro:macro name="vlp16_gpu" params="name parent *origin ros_topic update_rate ray_count min_angle max_angle">
+    <xacro:macro name="vlp16_gpu" params="name parent *origin ros_topic update_rate ray_count min_angle max_angle organize_cloud:=false">
       <xacro:vlp16_model name="${name}" parent="${parent}">
         <xacro:insert_block name="origin" />
@@ -150,4 +121,5 @@
             <topicName>${ros_topic}</topicName>
             <frameName>${name}_frame</frameName>
+            <organize_cloud>${organize_cloud}</organize_cloud>
           </plugin>
         </sensor>

Commit message: Added optional parameter for organized clouds to vlp16 macro

File: hector_sensors_description/urdf/vlp16.urdf.xacro (robot description, xacro)
@@ -42,5 +42,5 @@
     </xacro:vlp16_advanced_parameters>
   </xacro:macro>
-  <xacro:macro name="vlp16_advanced_parameters" params="name parent *origin ros_topic update_rate horizontal_samples vertical_samples min_range max_range use_gpu:='false'">
+  <xacro:macro name="vlp16_advanced_parameters" params="name parent *origin ros_topic update_rate horizontal_samples vertical_samples min_range max_range use_gpu:='false' organize_cloud:=false">
     <xacro:vlp16_model name="${name}" parent="${parent}">
       <xacro:insert_block name="origin"/>
@@ -88,4 +88,5 @@
           <topicName>${ros_topic}</topicName>
           <frameName>${name}_frame</frameName>
+          <organize_cloud>${organize_cloud}</organize_cloud>
           <min_range>${min_range}</min_range>
           <max_range>${max_range}</max_range>

Commit message: Revert "Use xacro param defaulting to false to optionally organize vlp16 points"
This reverts commit 1ec1f48b058c96cfc9530ad37820c1e8ca541760.

File: hector_sensors_description/urdf/vlp16.urdf.xacro (robot description, xacro)
@@ -43,9 +43,39 @@
       </xacro:vlp16_advanced_parameters>
     </xacro:macro>
-    <xacro:macro name="vlp16_advanced_parameters" params="name parent *origin ros_topic update_rate horizontal_samples vertical_samples min_range max_range organize_cloud:=false">
+    <xacro:macro name="vlp16_advanced_parameters" params="name parent *origin ros_topic update_rate horizontal_samples vertical_samples min_range max_range">
       <xacro:vlp16_model name="${name}" parent="${parent}">
         <xacro:insert_block name="origin" />
       </xacro:vlp16_model>
       <gazebo reference="${name}_frame">
+<!--        <sensor type="ray" name="${name}">
+          <always_on>true</always_on>
+          <update_rate>${update_rate}</update_rate>
+          <pose>0 0 0 0 0 0</pose>
+          <visualize>false</visualize>
+          <ray>
+            <scan>
+              <horizontal>
+                <samples>${ray_count}</samples>
+                <resolution>1</resolution>
+                <min_angle>${min_angle * M_PI/180}</min_angle>
+                <max_angle>${max_angle * M_PI/180}</max_angle>
+              </horizontal>
+            </scan>
+            <range>
+              <min>0.2</min>
+              <max>30.0</max>
+              <resolution>0.01</resolution>
+            </range>
+            <noise>
+              <type>gaussian</type>
+              <mean>0.0</mean>
+              <stddev>0.004</stddev>
+            </noise>
+          </ray>
+          <plugin name="gazebo_ros_${name}_controller" filename="libgazebo_ros_laser.so">
+            <topicName>${ros_topic}</topicName>
+            <frameName>${name}_frame</frameName>
+          </plugin>
+        </sensor>-->
       <sensor type="ray" name="${name}-VLP16">
         <pose>0 0 0 0 0 0</pose>
@@ -81,5 +111,4 @@
           <topicName>${ros_topic}</topicName>
           <frameName>${name}_frame</frameName>
-          <organize_cloud>${organize_cloud}</organize_cloud>
           <min_range>${min_range}</min_range>
           <max_range>${max_range}</max_range>
@@ -89,5 +118,5 @@
       </gazebo>
     </xacro:macro>
-    <xacro:macro name="vlp16_gpu" params="name parent *origin ros_topic update_rate ray_count min_angle max_angle organize_cloud:=false">
+    <xacro:macro name="vlp16_gpu" params="name parent *origin ros_topic update_rate ray_count min_angle max_angle">
       <xacro:vlp16_model name="${name}" parent="${parent}">
         <xacro:insert_block name="origin" />
@@ -121,5 +150,4 @@
             <topicName>${ros_topic}</topicName>
             <frameName>${name}_frame</frameName>
-            <organize_cloud>${organize_cloud}</organize_cloud>
           </plugin>
         </sensor>

Commit message: ignition adaptions

File: hector_sensors_description/urdf/vlp16.urdf.xacro (robot description, xacro)
@@ -52,5 +52,5 @@
       </xacro:if >
       <xacro:unless value="${use_gpu}">
-	      <xacro:property name="sensor_type" value="gpu_lidar"/><!--currently only gpu possible -->
+	      <xacro:property name="sensor_type" value="lidar"/><!--currently only gpu possible -->
         <xacro:property name="gazebo_plugin_name" value="libgazebo_ros_velodyne_laser.so"/>
       </xacro:unless>
