Commit message: fix D435 macro

File: hector_sensors_description/urdf/realsense_d435_camera.urdf.xacro (robot description, xacro)
@@ -27,5 +27,5 @@
         </inertial>
         <visual>
-          <origin xyz="0 0.0115 0" rpy="0 0 0" />
+          <origin xyz="-0.02 -0.0325 0" rpy="0 0 0" />
           <geometry>
             <!--Dimensions taken from https://click.intel.com/intelr-realsensetm-depth-camera-d435.html-->
@@ -37,9 +37,9 @@
         </visual>
         <collision>
-          <origin xyz="0 0.0115 0" rpy="0 0 0" />
+          <origin xyz="-0.02 -0.0325 0" rpy="0 0 0" />
           <geometry>
             <!--Dimensions taken from https://click.intel.com/intelr-realsensetm-depth-camera-d435.html-->
             <box size="0.025 0.09 0.025" />
-          </geometry>update_rate
+          </geometry>
         </collision>
       </link>
@@ -65,5 +65,5 @@
             <image>
               <format>B8G8R8</format>
-              <width>848</width>
+              <width>640</width>
               <height>480</height>
             </image>

Commit message: added the rgb optical frame

File: hector_sensors_description/urdf/realsense_d435_camera.urdf.xacro (robot description, xacro)
@@ -47,4 +47,10 @@
         <material>Gazebo/Grey</material>
       </gazebo>
+      <joint name="${name}_rgb_optical_joint" type="fixed">
+        <origin xyz="0 0 0" rpy="${-M_PI/2} 0.0 ${-M_PI/2}" />
+        <parent link="${name}_link" />
+        <child link="${name}_rgb_optical_frame"/>
+      </joint>
+      <link name="${name}_rgb_optical_frame"/>
     </xacro:macro>
     <xacro:macro name="realsense_d435_camera_model_no_geom" params="name parent *origin">

Commit message: fix name

File: hector_sensors_description/urdf/realsense_d435_camera.urdf.xacro (robot description, xacro)
@@ -47,10 +47,10 @@
         <material>Gazebo/Grey</material>
       </gazebo>
-      <joint name="${name}_rgb_optical_joint" type="fixed">
+      <joint name="${name}_color_optical_joint" type="fixed">
         <origin xyz="0 0 0" rpy="${-M_PI/2} 0.0 ${-M_PI/2}" />
         <parent link="${name}_link" />
-        <child link="${name}_rgb_optical_frame"/>
+        <child link="${name}_color_optical_frame"/>
       </joint>
-      <link name="${name}_rgb_optical_frame"/>
+      <link name="${name}_color_optical_frame"/>
     </xacro:macro>
     <xacro:macro name="realsense_d435_camera_model_no_geom" params="name parent *origin">

Commit message: d435 macro refactoring

File: hector_sensors_description/urdf/realsense_d435_camera.urdf.xacro (robot description, xacro)
@@ -10,7 +10,10 @@
 <robot xmlns:xacro="http://ros.org/wiki/xacro">
     <xacro:property name="M_PI" value="3.1415926535897931" />
+  <xacro:property name="realsense_d435_width" value="0.09"/>
+  <xacro:property name="realsense_d435_height" value="0.025"/>
+  <xacro:property name="realsense_d435_depth" value="0.025"/>
     <!--
      This macro only adds the model, it does not also add
-     the openni gazebo plugin. See the 'asus_camera' macro below for that
+     the openni gazebo plugin.
     -->
     <xacro:macro name="realsense_d435_camera_model" params="name parent *origin">
@@ -30,5 +33,5 @@
           <geometry>
             <!--Dimensions taken from https://click.intel.com/intelr-realsensetm-depth-camera-d435.html-->
-            <box size="0.025 0.09 0.025" />
+            <box size="${realsense_d435_depth} ${realsense_d435_width} ${realsense_d435_height}" />
           </geometry>
           <material name="DarkGrey">
@@ -40,5 +43,5 @@
           <geometry>
             <!--Dimensions taken from https://click.intel.com/intelr-realsensetm-depth-camera-d435.html-->
-            <box size="0.025 0.09 0.025" />
+            <box size="${realsense_d435_depth} ${realsense_d435_width} ${realsense_d435_height}" />
           </geometry>
         </collision>

Commit message: fixed visual and collision of d435

File: hector_sensors_description/urdf/realsense_d435_camera.urdf.xacro (robot description, xacro)
@@ -9,11 +9,15 @@
 -->
 <robot xmlns:xacro="http://ros.org/wiki/xacro">
-    <xacro:property name="M_PI" value="3.1415926535897931" />
+  <xacro:property name="M_PI" value="3.1415926535897931" />
   <xacro:property name="realsense_d435_width" value="0.09"/>
   <xacro:property name="realsense_d435_height" value="0.025"/>
   <xacro:property name="realsense_d435_depth" value="0.025"/>
+<!--   <xacro:property name="realsense_d435_case_offset_x" value="-0.02"/> -->
+  <xacro:property name="realsense_d435_case_offset_x" value="-0.0083"/>
+  <xacro:property name="realsense_d435_case_offset_y" value="-0.0175"/>
+  <xacro:property name="realsense_d435_case_offset_z" value="0.0"/>
     <!--
-     This macro only adds the model, it does not also add
-     the openni gazebo plugin.
+     This macro only adds the model, it does not also add the openni gazebo plugin.
+     The origin is the left infrared (depth) camera, which is also the origin of the depth image
     -->
     <xacro:macro name="realsense_d435_camera_model" params="name parent *origin">
@@ -30,5 +34,5 @@
         </inertial>
         <visual>
-          <origin xyz="-0.02 -0.0325 0" rpy="0 0 0" />
+          <origin xyz="${realsense_d435_case_offset_x} ${realsense_d435_case_offset_y} ${realsense_d435_case_offset_z}" rpy="0 0 0" />
           <geometry>
             <!--Dimensions taken from https://click.intel.com/intelr-realsensetm-depth-camera-d435.html-->
@@ -40,5 +44,5 @@
         </visual>
         <collision>
-          <origin xyz="-0.02 -0.0325 0" rpy="0 0 0" />
+          <origin xyz="${realsense_d435_case_offset_x} ${realsense_d435_case_offset_y} ${realsense_d435_case_offset_z}" rpy="0 0 0" />
           <geometry>
             <!--Dimensions taken from https://click.intel.com/intelr-realsensetm-depth-camera-d435.html-->

Commit message: more refactoring and added option to use realsense d435 mesh

File: hector_sensors_description/urdf/realsense_d435_camera.urdf.xacro (robot description, xacro)
@@ -13,6 +13,6 @@
   <xacro:property name="realsense_d435_height" value="0.025"/>
   <xacro:property name="realsense_d435_depth" value="0.025"/>
-<!--   <xacro:property name="realsense_d435_case_offset_x" value="-0.02"/> -->
-  <xacro:property name="realsense_d435_case_offset_x" value="-0.0083"/>
+  <xacro:property name="realsense_d435_front_to_depth" value="0.0042" />
+  <xacro:property name="realsense_d435_case_offset_x" value="${realsense_d435_front_to_depth - realsense_d435_depth/2.0}"/>
   <xacro:property name="realsense_d435_case_offset_y" value="-0.0175"/>
   <xacro:property name="realsense_d435_case_offset_z" value="0.0"/>
@@ -36,5 +36,4 @@
           <origin xyz="${realsense_d435_case_offset_x} ${realsense_d435_case_offset_y} ${realsense_d435_case_offset_z}" rpy="0 0 0" />
           <geometry>
-            <!--Dimensions taken from https://click.intel.com/intelr-realsensetm-depth-camera-d435.html-->
             <box size="${realsense_d435_depth} ${realsense_d435_width} ${realsense_d435_height}" />
           </geometry>
@@ -43,4 +42,10 @@
           </material>
         </visual>
+<!--        <visual>
+          <origin xyz="${realsense_d435_front_to_depth} ${realsense_d435_case_offset_y} 0.0" rpy="${M_PI/2} 0 ${M_PI/2}" />
+          <geometry>
+            <mesh filename="package://realsense2_camera/meshes/d435.dae" />
+          </geometry>
+        </visual>-->
         <collision>
           <origin xyz="${realsense_d435_case_offset_x} ${realsense_d435_case_offset_y} ${realsense_d435_case_offset_z}" rpy="0 0 0" />

Commit message: added new d435 macro with origin in mounting hole

File: hector_sensors_description/urdf/realsense_d435_camera.urdf.xacro (robot description, xacro)
@@ -13,7 +13,8 @@
   <xacro:property name="realsense_d435_height" value="0.025"/>
   <xacro:property name="realsense_d435_depth" value="0.025"/>
-  <xacro:property name="realsense_d435_front_to_depth" value="0.0042" />
+  <xacro:property name="realsense_d435_front_to_depth" value="0.0042" /> <!-- Intel_RealSense_D400_Family_Datasheet_Jan2019.pdf, page 64 -->
+  <xacro:property name="realsense_d435_mount_hole_to_front" value="0.0149" /> <!-- Measured from CAD file -->
   <xacro:property name="realsense_d435_case_offset_x" value="${realsense_d435_front_to_depth - realsense_d435_depth/2.0}"/>
-  <xacro:property name="realsense_d435_case_offset_y" value="-0.0175"/>
+  <xacro:property name="realsense_d435_case_offset_y" value="-0.0175"/> <!-- mounting hole to depth frame, Intel_RealSense_D400_Family_Datasheet_Jan2019.pdf, page 66 -->
   <xacro:property name="realsense_d435_case_offset_z" value="0.0"/>
     <!--
@@ -59,4 +60,16 @@
         <material>Gazebo/Grey</material>
       </gazebo>
+    </xacro:macro>
+    <xacro:macro name="realsense_d435_camera_model_with_mount" params="name parent *origin">
+      <joint name="${name}_mount_joint" type="fixed">
+        <xacro:insert_block name="origin" />
+        <parent link="${parent}"/>
+        <child link="${name}_mount_link"/>
+      </joint>
+      <link name="${name}_mount_link">
+      </link>
+      <xacro:realsense_d435_camera_model name="${name}" parent="${name}_mount_link">
+        <origin xyz="${realsense_d435_mount_hole_to_front - realsense_d435_front_to_depth} ${-realsense_d435_case_offset_y} ${realsense_d435_height/2.0}" rpy="0 0 0"/>
+      </xacro:realsense_d435_camera_model>
     </xacro:macro>
     <xacro:macro name="realsense_d435_camera_model_no_geom" params="name parent *origin">
@@ -128,3 +141,9 @@
       <xacro:realsense_d435_camera_gazebo_plugin_macro name="${name}" parent="${parent}" image_topic="${image_topic}" depth_points_topic="${depth_points_topic}" min_range="${min_range}" max_range="${max_range}" update_rate="${update_rate}"/>
     </xacro:macro>
+    <xacro:macro name="realsense_d435_camera_with_mount_comprehensive_params" params="name parent *origin image_topic depth_points_topic min_range max_range update_rate">
+      <xacro:realsense_d435_camera_model_with_mount name="${name}" parent="${parent}">
+        <xacro:insert_block name="origin" />
+      </xacro:realsense_d435_camera_model_with_mount>
+      <xacro:realsense_d435_camera_gazebo_plugin_macro name="${name}" parent="${parent}" image_topic="${image_topic}" depth_points_topic="${depth_points_topic}" min_range="${min_range}" max_range="${max_range}" update_rate="${update_rate}"/>
+    </xacro:macro>
   </robot>

Commit message: added raycast geom

File: hector_sensors_description/urdf/realsense_d435_camera.urdf.xacro (robot description, xacro)
@@ -56,4 +56,12 @@
           </geometry>
         </collision>
+      <xacro:if value="$(arg add_raycast_self_filter_geom)">
+        <collision>
+          <origin xyz="${realsense_d435_case_offset_x} ${realsense_d435_case_offset_y} ${realsense_d435_case_offset_z}" rpy="${M_PI*0.5} 0 0" />
+          <geometry>
+            <cylinder length="0.09" radius="0.0177"/>
+          </geometry>
+        </collision>
+      </xacro:if>
       </link>
       <gazebo reference="${name}_link">

File: hector_sensors_description/urdf/seek_thermal_compact.urdf.xacro (robot description, xacro)
@@ -39,4 +39,13 @@
         </geometry>
       </collision>
+      <xacro:property name="collision_size_factor" value="1"/>
+      <xacro:if value="$(arg add_raycast_self_filter_geom)">
+        <collision>
+          <origin xyz="0.0055 0 -0.013375" rpy="0 0 0" />
+          <geometry>
+            <cylinder length="${0.06075 * collision_size_factor}" radius="${0.023 * collision_size_factor}"/>
+          </geometry>
+        </collision>
+      </xacro:if>
     </link>
     <xacro:add_optical_frame name="${name}" />

Commit message: added macro for realsense with mount

File: hector_sensors_description/urdf/realsense_d435_camera.urdf.xacro (robot description, xacro)
@@ -121,4 +121,5 @@
     <!--
       Use the macro below for adding the realsense model with link geometry
+      The origin is the left infrared (depth) camera, which is also the origin of the depth image
     -->
     <xacro:macro name="realsense_d435_camera" params="name parent *origin">
@@ -126,4 +127,13 @@
         <xacro:insert_block name="origin" />
       </xacro:realsense_d435_camera_model>
+      <xacro:realsense_d435_camera_gazebo_plugin_macro name="${name}" parent="${parent}" image_topic="image_raw" depth_points_topic="depth/points" min_range="0.3" max_range="9.0" update_rate="20"/>
+    </xacro:macro>
+    <!--
+      Insert the realsense with link geometry. Origin is the mounting hole at the back of the camera.
+    -->
+    <xacro:macro name="realsense_d435_camera_with_mount" params="name parent *origin">
+      <xacro:realsense_d435_camera_model_with_mount name="${name}" parent="${parent}">
+        <xacro:insert_block name="origin" />
+      </xacro:realsense_d435_camera_model_with_mount>
       <xacro:realsense_d435_camera_gazebo_plugin_macro name="${name}" parent="${parent}" image_topic="image_raw" depth_points_topic="depth/points" min_range="0.3" max_range="9.0" update_rate="20"/>
     </xacro:macro>

Commit message: use a prettier D435 model

File: hector_sensors_description/urdf/realsense_d435_camera.urdf.xacro (robot description, xacro)
@@ -35,19 +35,10 @@
           <inertia ixx="5.8083e-4" ixy="0" ixz="0" iyy="3.0833e-5" iyz="0" izz="5.9083e-4" />
         </inertial>
-        <visual>
-          <origin xyz="${realsense_d435_case_offset_x} ${realsense_d435_case_offset_y} ${realsense_d435_case_offset_z}" rpy="0 0 0" />
-          <geometry>
-            <box size="${realsense_d435_depth} ${realsense_d435_width} ${realsense_d435_height}" />
-          </geometry>
-          <material name="DarkGrey">
-            <color rgba="0.3 0.3 0.3 1"/>
-          </material>
-        </visual>
-<!--        <visual>
+	<visual>
           <origin xyz="${realsense_d435_front_to_depth} ${realsense_d435_case_offset_y} 0.0" rpy="${M_PI/2} 0 ${M_PI/2}" />
           <geometry>
-            <mesh filename="package://realsense2_camera/meshes/d435.dae" />
+            <mesh filename="package://hector_sensors_description/meshes/intel_realsense_d435/D435.dae" scale="0.001 0.001 0.001" />
           </geometry>
-        </visual>-->
+        </visual>
         <collision>
           <origin xyz="${realsense_d435_case_offset_x} ${realsense_d435_case_offset_y} ${realsense_d435_case_offset_z}" rpy="0 0 0" />

Commit message: ignition changes

File: hector_sensors_description/urdf/realsense_d435_camera.urdf.xacro (robot description, xacro)
@@ -84,5 +84,5 @@
     <xacro:macro name="realsense_d435_camera_gazebo_plugin_macro" params="name parent image_topic depth_topic:=image_raw depth_points_topic frame_name:=color min_range max_range update_rate">
       <gazebo reference="${name}_link">
-        <sensor type="depth" name="${name}">
+        <sensor type="rgbd" name="${name}">
           <update_rate>${update_rate}</update_rate>
           <camera>
@@ -98,5 +98,6 @@
             </clip>
           </camera>
-          <plugin name="${name}_camera_controller" filename="libgazebo_ros_openni_kinect.so">
+	  <topic>${name}</topic>
+          <!--plugin name="${name}_camera_controller" filename="libgazebo_ros_openni_kinect.so">
             <cameraName>${name}</cameraName>
             <imageTopicName>color/${image_topic}</imageTopicName>
@@ -105,10 +106,10 @@
             <depthImageCameraInfoTopicName>depth/camera_info</depthImageCameraInfoTopicName>
             <pointCloudTopicName>${depth_points_topic}</pointCloudTopicName>
-            <frameName>${name}_${frame_name}_optical_frame</frameName>
+            <frameName>${name}_${frame_name}_optical_frame</frameName-->
             <!-- Important information about frames: Currently, this plugin only supports simulation of color image and depth image/cloud from a single frame.
             This frame is given in the <gazebo reference=""> tag above and is set to the ${name}_link which coincides with the depth camera frame. The camera axis is the X-axis. ROS requires an optical frame
             with the Z-axis as camera axis. It is advised to use the depth_optical_frame for this purpose (frame_name="depth"), even though camera images will have the same frame.
             The color_optical_frame does not coincide with the depth_optical_frame, so depth image/cloud will be misaligned! -->
-          </plugin>
+          <!--/plugin-->
         </sensor>
       </gazebo>

File: hector_sensors_description/urdf/seek_thermal_compact.urdf.xacro (robot description, xacro)
@@ -57,5 +57,5 @@
   <xacro:macro name="seek_thermal_compact_gazebo_plugin_macro" params="name parent *origin">
     <gazebo reference="${name}_frame">
-      <sensor type="camera" name="thermal_camera_sensor">
+      <sensor type="thermal" name="thermal_camera_sensor">
         <update_rate>10</update_rate>
         <camera>
@@ -71,5 +71,6 @@
           </clip>
         </camera>
-        <plugin name="thermal_camera_controller" filename="libgazebo_ros_thermal_camera.so">
+	<topic>${name}/image_raw</topic>
+        <!--plugin name="thermal_camera_controller" filename="libgazebo_ros_thermal_camera.so">
           <alwaysOn>true</alwaysOn>
           <updateRate>10</updateRate>
@@ -78,5 +79,5 @@
           <cameraInfoTopicName>camera_info</cameraInfoTopicName>
           <frameName>${name}_optical_frame</frameName>
-        </plugin>
+        </plugin-->
       </sensor>
     </gazebo>

File: hector_sensors_description/urdf/vlp16.urdf.xacro (robot description, xacro)
@@ -48,9 +48,9 @@
     <gazebo reference="${name}_frame">
       <xacro:if value="${use_gpu}">
-        <xacro:property name="sensor_type" value="gpu_ray"/>
+        <xacro:property name="sensor_type" value="gpu_lidar"/>
         <xacro:property name="gazebo_plugin_name" value="libgazebo_ros_velodyne_gpu_laser.so"/>
       </xacro:if >
       <xacro:unless value="${use_gpu}">
-        <xacro:property name="sensor_type" value="ray"/>
+	      <xacro:property name="sensor_type" value="gpu_lidar"/><!--currently only gpu possible -->
         <xacro:property name="gazebo_plugin_name" value="libgazebo_ros_velodyne_laser.so"/>
       </xacro:unless>
@@ -59,5 +59,6 @@
         <visualize>false</visualize>
         <update_rate>${update_rate}</update_rate>
-        <ray>
+        <topic>${ros_topic}</topic>
+        <lidar>
           <scan>
             <horizontal>
@@ -82,8 +83,8 @@
             <type>gaussian</type>
             <mean>0.0</mean>
-            <stddev>0.0</stddev>
+            <stddev>0.008</stddev>
           </noise>
-        </ray>
-        <plugin name="gazebo_ros_laser_controller" filename="${gazebo_plugin_name}">
+        </lidar>
+        <!--plugin name="gazebo_ros_laser_controller" filename="${gazebo_plugin_name}">
           <topicName>${ros_topic}</topicName>
           <frameName>${name}_frame</frameName>
@@ -92,5 +93,5 @@
           <max_range>${max_range}</max_range>
           <gaussianNoise>0.008</gaussianNoise>
-        </plugin>
+        </plugin-->
       </sensor>
     </gazebo>

Commit message: Removed missing parameters

File: hector_sensors_description/urdf/realsense_d435_camera.urdf.xacro (robot description, xacro)
@@ -23,5 +23,4 @@
     -->
     <xacro:macro name="realsense_d435_camera_model" params="name parent *origin">
-      <xacro:arg name="add_raycast_self_filter_geom" default="false"/>
       <joint name="${name}_joint" type="fixed">
         <xacro:insert_block name="origin" />
@@ -48,12 +47,4 @@
           </geometry>
         </collision>
-      <xacro:if value="$(arg add_raycast_self_filter_geom)">
-        <collision>
-          <origin xyz="${realsense_d435_case_offset_x} ${realsense_d435_case_offset_y} ${realsense_d435_case_offset_z}" rpy="${M_PI*0.5} 0 0" />
-          <geometry>
-            <cylinder length="0.09" radius="0.0177"/>
-          </geometry>
-        </collision>
-      </xacro:if>
       </link>
       <gazebo reference="${name}_link">

File: hector_sensors_description/urdf/seek_thermal_compact.urdf.xacro (robot description, xacro)
@@ -40,12 +40,4 @@
             </geometry>
         </collision>
-        <xacro:if value="$(arg add_raycast_self_filter_geom)">
-            <collision>
-            <origin xyz="0.0055 0 -0.013375" rpy="0 0 0" />
-            <geometry>
-                <cylinder length="0.06075" radius="0.023"/>
-            </geometry>
-            </collision>
-        </xacro:if>
       </xacro:if>
     </link>

Commit message: added comprehensive params for camera and mount to have default params

File: hector_sensors_description/urdf/realsense_d435_camera.urdf.xacro (robot description, xacro)
@@ -140,5 +140,5 @@
       <xacro:realsense_camera_gazebo_plugin_macro name="${name}" parent="${parent}" image_topic="${image_topic}" depth_topic="${depth_topic}" depth_points_topic="${depth_points_topic}" frame_name="${frame_name}" min_range="${min_range}" max_range="${max_range}" update_rate="${update_rate}"/>
     </xacro:macro>
-    <xacro:macro name="realsense_d435_camera_comprehensive_params" params="name parent *origin image_topic depth_topic:=image_raw depth_points_topic frame_name:=color min_range max_range update_rate">
+    <xacro:macro name="realsense_d435_camera_comprehensive_params" params="name parent *origin image_topic:=image_raw depth_topic:=image_raw depth_points_topic:=depth/color/points frame_name:=color min_range:=0.3 max_range:=9.0 update_rate:=20">
       <xacro:realsense_d435_camera_model name="${name}" parent="${parent}">
         <xacro:insert_block name="origin" />
@@ -146,5 +146,5 @@
       <xacro:realsense_d435_camera_gazebo_plugin_macro name="${name}" parent="${parent}" image_topic="${image_topic}" depth_topic="${depth_topic}" depth_points_topic="${depth_points_topic}" frame_name="${frame_name}" min_range="${min_range}" max_range="${max_range}" update_rate="${update_rate}"/>
     </xacro:macro>
-    <xacro:macro name="realsense_d435_camera_with_mount_comprehensive_params" params="name parent *origin image_topic depth_topic:=image_raw depth_points_topic frame_name:=color min_range max_range update_rate">
+    <xacro:macro name="realsense_d435_camera_with_mount_comprehensive_params" params="name parent *origin image_topic:=image_raw depth_topic:=image_raw depth_points_topic:=depth/color/points frame_name:=color min_range:=0.3 max_range:=9.0 update_rate:=20">
       <xacro:realsense_d435_camera_model_with_mount name="${name}" parent="${parent}">
         <xacro:insert_block name="origin" />
