Commit message: hector_sensors_description: added camera frames for the kinect camera and removed inertia from optical frame for the generic camera

File: hector_sensors_description/urdf/generic_camera.urdf.xacro (robot description, xacro)
@@ -39,25 +39,5 @@
       <child link="${name}_optical_frame"/>
     </joint>
-    <link name="${name}_optical_frame">
-      <inertial>
-        <mass value="0.01" />
-        <origin xyz="0 0 0" />
-        <inertia ixx="0.001"  ixy="0.0"  ixz="0.0"
-                 iyy="0.001"  iyz="0.0"
-                 izz="0.001" />
-      </inertial>
-      <visual>
-        <origin xyz="0 0 0" rpy="0 0 0"/>
-        <geometry>
-          <box size="0.001 0.001 0.001" />
-        </geometry>
-      </visual>
-      <collision>
-        <origin xyz="0 0 0" rpy="0 0 0"/>
-        <geometry>
-          <box size="0.001 0.001 0.001" />
-        </geometry>
-      </collision>
-    </link>
+    <link name="${name}_optical_frame"/>
     <gazebo reference="${name}_link">
       <sensor:camera name="${name}_camera_sensor">

File: hector_sensors_description/urdf/kinect_camera.urdf.xacro (robot description, xacro)
@@ -28,4 +28,28 @@
         </collision>
       </link>
+      <joint name="${name}_depth_joint" type="fixed">
+        <origin xyz="0.0 -0.02 0.0" rpy="0 0 0" />
+        <parent link="${name}_link" />
+        <child link="${name}_depth_frame"/>
+      </joint>
+      <link name="${name}_depth_frame"/>
+      <joint name="${name}_depth_optical_joint" type="fixed">
+        <origin xyz="0 0 0" rpy="${-M_PI/2} 0.0 ${-M_PI/2}" />
+        <parent link="${name}_depth_frame" />
+        <child link="${name}_depth_optical_frame"/>
+      </joint>
+      <link name="${name}_depth_optical_frame"/>
+      <joint name="${name}_rgb_joint" type="fixed">
+        <origin xyz="0.0 -0.045 0.0" rpy="0 0 0" />
+        <parent link="${name}_link" />
+        <child link="${name}_rgb_frame"/>
+      </joint>
+      <link name="${name}_rgb_frame"/>
+      <joint name="${name}_rgb_optical_joint" type="fixed">
+        <origin xyz="0 0 0" rpy="${-M_PI/2} 0.0 ${-M_PI/2}" />
+        <parent link="${name}_rgb_frame" />
+        <child link="${name}_rgb_optical_frame"/>
+      </joint>
+      <link name="${name}_rgb_optical_frame"/>
     </xacro:macro>
     <xacro:macro name="kinect_camera" params="name parent *origin">
@@ -60,5 +84,5 @@
         </sensor:camera>
       </gazebo> -->
-      <gazebo reference="${name}_link">
+      <gazebo reference="${name}_depth_frame">
         <sensor:camera name="${name}">
           <imageFormat>R8G8B8</imageFormat>

Commit message: hector_sensors_description: use gazebo_ros_camera plugin instead of gazebo_ros_depth_camera for the generic camera
* This was a relict from gazebo for fuerte.

File: hector_sensors_description/urdf/generic_camera.urdf.xacro (robot description, xacro)
@@ -51,5 +51,5 @@
           </clip>
         </camera>
-        <plugin name="${name}_camera_controller" filename="libgazebo_ros_depth_camera.so">
+        <plugin name="${name}_camera_controller" filename="libgazebo_ros_camera.so">
           <cameraName>${name}</cameraName>
           <alwaysOn>true</alwaysOn>
@@ -60,5 +60,4 @@
         </plugin>
       </sensor>
-      <material>PR2/Blue</material>
     </gazebo>
   </xacro:macro>

Commit message: hector_sensors_description: use radians for angle parameters consistently (affects generic_camera.urdf.xacro)

File: hector_sensors_description/urdf/generic_camera.urdf.xacro (robot description, xacro)
@@ -40,5 +40,5 @@
         <update_rate>${update_rate}</update_rate>
         <camera>
-          <horizontal_fov>${hfov * M_PI/180.0}</horizontal_fov>
+          <horizontal_fov>${hfov}</horizontal_fov>
           <image>
             <format>${image_format}</format>

File: hector_sensors_description/urdf/thermaleye_camera.urdf.xacro (robot description, xacro)
@@ -2,5 +2,4 @@
 <robot xmlns:xacro="http://ros.org/wiki/xacro">
     <xacro:include filename="$(find hector_xacro_tools)/urdf/sensor_macros.urdf.xacro" />
-    <xacro:property name="M_PI" value="3.1415926535897931" />
     <xacro:macro name="thermaleye_camera_model" params="name parent *origin">
       <joint name="${name}_joint" type="fixed">

Commit message: Revert "hector_sensors_description: use radians for angle parameters consistently (affects generic_camera.urdf.xacro)"
This reverts commit 89e18055753addd0d669f824755499f48ba75b01.

File: hector_sensors_description/urdf/generic_camera.urdf.xacro (robot description, xacro)
@@ -40,5 +40,5 @@
         <update_rate>${update_rate}</update_rate>
         <camera>
-          <horizontal_fov>${hfov}</horizontal_fov>
+          <horizontal_fov>${hfov * M_PI/180.0}</horizontal_fov>
           <image>
             <format>${image_format}</format>

File: hector_sensors_description/urdf/thermaleye_camera.urdf.xacro (robot description, xacro)
@@ -2,4 +2,5 @@
 <robot xmlns:xacro="http://ros.org/wiki/xacro">
     <xacro:include filename="$(find hector_xacro_tools)/urdf/sensor_macros.urdf.xacro" />
+    <xacro:property name="M_PI" value="3.1415926535897931" />
     <xacro:macro name="thermaleye_camera_model" params="name parent *origin">
       <joint name="${name}_joint" type="fixed">

Commit message: Remove link geometries where not needed Add generic_thermal_camera macro

File: hector_sensors_description/urdf/generic_camera.urdf.xacro (robot description, xacro)
@@ -9,5 +9,5 @@
     </joint>
     <link name="${name}_link">
-      <inertial>
+<!--      <inertial>
         <mass value="0.001" />
         <origin xyz="0 0 0" rpy="0 0 0" />
@@ -28,5 +28,5 @@
           <box size="0.01 0.01 0.01" />
         </geometry>
-      </collision>
+      </collision>-->
     </link>
     <joint name="${name}_optical_joint" type="fixed">

File: hector_sensors_description/urdf/generic_stereo_camera.urdf.xacro (robot description, xacro)
@@ -2,5 +2,5 @@
 <robot xmlns:xacro="http://ros.org/wiki/xacro">
   <xacro:property name="M_PI" value="3.1415926535897931" />
-  <xacro:macro name="generic_stereo_camera" params="name parent *origin ros_topic cam_info_topic update_rate res_x res_y image_format hfov">
+  <xacro:macro name="generic_stereo_camera" params="name parent *origin ros_topic cam_info_topic update_rate res_x res_y image_format hfov baseline">
   <!-- Stereo Camera -->
   <joint name="${name}_left_camera_frame_joint" type="fixed">
@@ -11,10 +11,9 @@
   </joint>
   <link name="${name}_left_camera_frame">
-    <inertial>
+<!--    <inertial>
       <mass value="1e-5" />
-      <!-- collocate with parent link and remove mass from it -->
       <origin xyz="-0.075493 0.035033383 0.02574"/>
       <inertia ixx="1e-6" ixy="0" ixz="0" iyy="1e-6" iyz="0" izz="1e-6" />
-    </inertial>
+    </inertial>-->
   </link>
   <joint name="${name}_left_camera_optical_frame_joint" type="fixed">
@@ -54,5 +53,5 @@
       </camera>
       <camera name="right">
-        <pose>0 -0.07 0 0 0 0</pose>
+        <pose>0 ${-baseline} 0 0 0 0</pose>
         <!-- Spec sheet says 80deg X 45deg @ 1024x544pix.  Based on feedback
              from teams, we're instead doing 80deg X 80deg @ 800x800pix. -->
@@ -87,5 +86,5 @@
         <frameName>${name}_left_camera_optical_frame</frameName>
         <!--<rightFrameName>right_camera_optical_frame</rightFrameName>-->
-        <hackBaseline>0.07</hackBaseline>
+        <hackBaseline>${baseline}</hackBaseline>
         <distortionK1>0.0</distortionK1>
         <distortionK2>0.0</distortionK2>
@@ -97,15 +96,14 @@
   </gazebo>
   <joint name="${name}_right_camera_frame_joint" type="fixed">
-    <origin xyz="0.0 -0.07 -0.0"/>
+    <origin xyz="0.0 ${-baseline} -0.0"/>
     <parent link="${name}_left_camera_frame"/>
     <child link="${name}_right_camera_frame"/>
   </joint>
   <link name="${name}_right_camera_frame">
-    <inertial>
+<!--    <inertial>
       <mass value="1e-5" />
-      <!-- collocate with parent link and remove mass from it -->
       <origin xyz="-0.075493 -0.034966617 0.02574"/>
       <inertia ixx="1e-6" ixy="0" ixz="0" iyy="1e-6" iyz="0" izz="1e-6" />
-    </inertial>
+    </inertial>-->
   </link>
   <joint name="${name}_right_camera_optical_frame_joint" type="fixed">

Commit message: Add params and defaults for near and far clip planes of generic camera macro

File: hector_sensors_description/urdf/generic_camera.urdf.xacro (robot description, xacro)
@@ -2,5 +2,5 @@
 <robot xmlns:xacro="http://www.ros.org/wiki/xacro">
   <xacro:property name="M_PI" value="3.1415926535897931" />
-  <xacro:macro name="generic_camera" params="name parent *origin ros_topic cam_info_topic update_rate res_x res_y image_format hfov">
+  <xacro:macro name="generic_camera" params="name parent *origin ros_topic cam_info_topic update_rate res_x res_y image_format hfov near_clip:=0.1 far_clip:=100.0">
     <joint name="${name}_joint" type="fixed">
       <xacro:insert_block name="origin" />
@@ -47,6 +47,6 @@
           </image>
           <clip>
-            <near>0.01</near>
-            <far>100</far>
+            <near>${near_clip}</near>
+            <far>${far_clip}</far>
           </clip>
         </camera>
