Commit message: added calibration parameter

File: hector_sensors_description/urdf/camera360.urdf.xacro (robot description, xacro)
@@ -2,5 +2,5 @@
 <robot xmlns:xacro="http://ros.org/wiki/xacro">
   <xacro:property name="M_PI" value="3.1415926535897931" />
-  <xacro:property name="dist_between_cameras" value="0.01602869966119076" />
+  <xacro:property name="dist_between_cameras" value="0.03850784" />
   <xacro:macro name="camera360" params="name right_cam_name left_cam_name parent *origin *calibration ros_topic update_rate res_x res_y image_format fov">
     <joint name="${name}_center_joint" type="fixed">
@@ -52,16 +52,16 @@
       </sensor>
     </gazebo>
-    <joint name="${name}_${left_cam_name}_joint" type="fixed">
+    <joint name="${name}_${left_cam_name}_optical_joint" type="fixed">
       <xacro:insert_block name="calibration" />
-      <parent link="${name}_${right_cam_name}_link"/>
-      <child link="${name}_${left_cam_name}_link"/>
-    </joint>
-    <link name="${name}_${left_cam_name}_link"/>
-    <joint name="${name}_${left_cam_name}_optical_joint" type="fixed">
-      <origin xyz="0 0 0" rpy="${-M_PI/2} 0.0 ${-M_PI/2}" />
-      <parent link="${name}_${left_cam_name}_link" />
+      <parent link="${name}_${right_cam_name}_optical_frame"/>
       <child link="${name}_${left_cam_name}_optical_frame"/>
     </joint>
     <link name="${name}_${left_cam_name}_optical_frame"/>
+    <joint name="${name}_${left_cam_name}_joint" type="fixed">
+      <origin xyz="0 0 0" rpy="${M_PI/2} 0.0 ${M_PI/2}" />
+      <parent link="${name}_${left_cam_name}_optical_frame"/>
+      <child link="${name}_${left_cam_name}_link" />
+    </joint>
+    <link name="${name}_${left_cam_name}_link"/>
     <gazebo reference="${name}_${left_cam_name}_link">
       <sensor type="wideanglecamera" name="${name}_${left_cam_name}_camera_sensor">

Commit message: added parameter for dist between cams to camera360 macro

File: hector_sensors_description/urdf/camera360.urdf.xacro (robot description, xacro)
@@ -2,6 +2,5 @@
 <robot xmlns:xacro="http://ros.org/wiki/xacro">
   <xacro:property name="M_PI" value="3.1415926535897931" />
-  <xacro:property name="dist_between_cameras" value="0.03850784" />
-  <xacro:macro name="camera360" params="name right_cam_name left_cam_name parent *origin *calibration ros_topic update_rate res_x res_y image_format fov">
+  <xacro:macro name="camera360" params="name right_cam_name left_cam_name parent *origin *calibration dist_between_cameras ros_topic update_rate res_x res_y image_format fov">
     <joint name="${name}_center_joint" type="fixed">
       <xacro:insert_block name="origin" />
@@ -11,5 +10,5 @@
     <link name="${name}_center_link" />
     <joint name="${name}_${right_cam_name}_joint" type="fixed">
-      <origin xyz="${0} ${dist_between_cameras/2} 0" rpy="${M_PI*0.5} 0 ${-M_PI*0.5}"/>
+      <origin xyz="0 ${dist_between_cameras/2} 0" rpy="${M_PI*0.5} 0 ${-M_PI*0.5}"/>
       <parent link="${name}_center_link"/>
       <child link="${name}_${right_cam_name}_link"/>

Commit message: fixed default collision radius

File: hector_sensors_description/urdf/camera360.urdf.xacro (robot description, xacro)
@@ -2,5 +2,5 @@
 <robot xmlns:xacro="http://ros.org/wiki/xacro">
   <xacro:property name="M_PI" value="3.1415926535897931" />
-  <xacro:property name="default_collision_radius" value="0.25" />
+  <xacro:property name="default_collision_radius" value="0.025" />
   <xacro:property name="visual_radius" value="0.011" />
   <xacro:property name="cable_collision_length" value="0.05" />

Commit message: fixed cam frame orientation

File: hector_sensors_description/urdf/camera360.urdf.xacro (robot description, xacro)
@@ -100,5 +100,5 @@
     <link name="${name}_${left_cam_name}_optical_frame"/>
     <joint name="${name}_${left_cam_name}_joint" type="fixed">
-      <origin xyz="0 0 0" rpy="${M_PI/2} 0.0 ${M_PI/2}" />
+      <origin xyz="0 0 0" rpy="0 ${-M_PI/2} ${M_PI/2}" />
       <parent link="${name}_${left_cam_name}_optical_frame"/>
       <child link="${name}_${left_cam_name}_link" />

Commit message: fixed insta360 cam size

File: hector_sensors_description/urdf/camera360.urdf.xacro (robot description, xacro)
@@ -3,5 +3,5 @@
   <xacro:property name="M_PI" value="3.1415926535897931" />
   <xacro:property name="default_collision_radius" value="0.025" />
-  <xacro:property name="visual_radius" value="0.011" />
+  <xacro:property name="visual_radius" value="0.02" />
   <xacro:property name="cable_collision_length" value="0.05" />
   <xacro:macro name="camera360" params="name right_cam_name left_cam_name parent collision_radius:=${default_collision_radius} *origin *calibration dist_between_cameras ros_topic update_rate res_x res_y image_format fov">

Commit message: adaptions for webots

File: hector_sensors_description/urdf/camera360.urdf.xacro (robot description, xacro)
@@ -63,5 +63,5 @@
     </joint>
     <link name="${name}_${right_cam_name}_optical_frame"/>
-    <gazebo reference="${name}_${right_cam_name}_link">
+    <webots reference="${name}_${right_cam_name}_link">
       <sensor type="wideanglecamera" name="${name}_${right_cam_name}_camera_sensor">
         <update_rate>${update_rate}</update_rate>
@@ -97,12 +97,12 @@
           </lens>
         </camera>
-        <plugin name="${name}_${right_cam_name}_camera_controller" filename="libgazebo_ros_camera.so">
+        <!--plugin name="${name}_${right_cam_name}_camera_controller" filename="libgazebo_ros_camera.so">
           <cameraName>${name}/${right_cam_name}</cameraName>
           <imageTopicName>${ros_topic}</imageTopicName>
           <cameraInfoTopicName>not_used</cameraInfoTopicName>
           <frameName>${name}_${right_cam_name}_optical_frame</frameName>
-        </plugin>
+        </plugin-->
       </sensor>
-    </gazebo>
+    </webots>
     <joint name="${name}_${left_cam_name}_optical_joint" type="fixed">
       <xacro:insert_block name="calibration" />
@@ -117,5 +117,5 @@
     </joint>
     <link name="${name}_${left_cam_name}_link"/>
-    <gazebo reference="${name}_${left_cam_name}_link">
+    <webots reference="${name}_${left_cam_name}_link">
       <sensor type="wideanglecamera" name="${name}_${left_cam_name}_camera_sensor">
         <update_rate>${update_rate}</update_rate>
@@ -151,12 +151,12 @@
           </lens>
         </camera>
-        <plugin name="${name}_${left_cam_name}_camera_controller" filename="libgazebo_ros_camera.so">
+        <!--plugin name="${name}_${left_cam_name}_camera_controller" filename="libgazebo_ros_camera.so">
           <cameraName>${name}/${left_cam_name}</cameraName>
           <imageTopicName>${ros_topic}</imageTopicName>
           <cameraInfoTopicName>not_used</cameraInfoTopicName>
           <frameName>${name}_${left_cam_name}_optical_frame</frameName>
-        </plugin>
+        </plugin-->
       </sensor>
-    </gazebo>
+    </webots>
   </xacro:macro>
 </robot>

File: hector_sensors_description/urdf/generic_camera.urdf.xacro (robot description, xacro)
@@ -36,5 +36,5 @@
     </joint>
     <link name="${name}_optical_frame"/>
-    <gazebo reference="${name}_link">
+    <webots reference="${name}_link">
       <sensor type="camera" name="${name}_camera_sensor">
         <update_rate>${update_rate}</update_rate>
@@ -51,12 +51,6 @@
           </clip>
         </camera>
-        <plugin name="${name}_camera_controller" filename="libgazebo_ros_camera.so">
-          <cameraName>${name}</cameraName>
-          <imageTopicName>${ros_topic}</imageTopicName>
-          <cameraInfoTopicName>${cam_info_topic}</cameraInfoTopicName>
-          <frameName>${name}_optical_frame</frameName>
-        </plugin>
       </sensor>
-    </gazebo>
+    </webots>
   </xacro:macro>
 </robot>

File: hector_sensors_description/urdf/realsense_d435_camera.urdf.xacro (robot description, xacro)
@@ -57,7 +57,7 @@
       </xacro:if>
       </link>
-      <gazebo reference="${name}_link">
+      <webots reference="${name}_link">
         <material>Gazebo/Grey</material>
-      </gazebo>
+      </webots>
     </xacro:macro>
     <xacro:macro name="realsense_d435_camera_model_with_mount" params="name parent *origin">
@@ -83,6 +83,6 @@
     </xacro:macro>
     <xacro:macro name="realsense_d435_camera_gazebo_plugin_macro" params="name parent image_topic depth_topic:=image_raw depth_points_topic frame_name:=color min_range max_range update_rate">
-      <gazebo reference="${name}_link">
-        <sensor type="depth" name="${name}">
+      <webots reference="${name}_link">
+        <sensor type="rgbd" name="${name}">
           <update_rate>${update_rate}</update_rate>
           <camera>
@@ -98,5 +98,5 @@
             </clip>
           </camera>
-          <plugin name="${name}_camera_controller" filename="libgazebo_ros_openni_kinect.so">
+          <!--plugin name="${name}_camera_controller" filename="libgazebo_ros_openni_kinect.so">
             <cameraName>${name}</cameraName>
             <imageTopicName>color/${image_topic}</imageTopicName>
@@ -105,12 +105,12 @@
             <depthImageCameraInfoTopicName>depth/camera_info</depthImageCameraInfoTopicName>
             <pointCloudTopicName>${depth_points_topic}</pointCloudTopicName>
-            <frameName>${name}_${frame_name}_optical_frame</frameName>
+            <frameName>${name}_${frame_name}_optical_frame</frameName-->
             <!-- Important information about frames: Currently, this plugin only supports simulation of color image and depth image/cloud from a single frame.
             This frame is given in the <gazebo reference=""> tag above and is set to the ${name}_link which coincides with the depth camera frame. The camera axis is the X-axis. ROS requires an optical frame
             with the Z-axis as camera axis. It is advised to use the depth_optical_frame for this purpose (frame_name="depth"), even though camera images will have the same frame.
             The color_optical_frame does not coincide with the depth_optical_frame, so depth image/cloud will be misaligned! -->
-          </plugin>
+          <!--/plugin-->
         </sensor>
-      </gazebo>
+      </webots>
     </xacro:macro>
     <!--

File: hector_sensors_description/urdf/vlp16.urdf.xacro (robot description, xacro)
@@ -46,12 +46,12 @@
       <xacro:insert_block name="origin"/>
     </xacro:vlp16_model>
-    <gazebo reference="${name}_frame">
+    <webots reference="${name}_frame">
       <xacro:if value="${use_gpu}">
-        <xacro:property name="sensor_type" value="gpu_ray"/>
-        <xacro:property name="gazebo_plugin_name" value="libgazebo_ros_velodyne_gpu_laser.so"/>
+        <xacro:property name="sensor_type" value="gpu_lidar"/>
+        <xacro:property name="plugin_type" value="lidar"/>
       </xacro:if >
       <xacro:unless value="${use_gpu}">
-        <xacro:property name="sensor_type" value="ray"/>
-        <xacro:property name="gazebo_plugin_name" value="libgazebo_ros_velodyne_laser.so"/>
+        <xacro:property name="sensor_type" value="lidar"/>
+        <xacro:property name="plugin_type" value="lidar"/>
       </xacro:unless>
       <sensor type="${sensor_type}" name="${name}-VLP16">
@@ -85,5 +85,5 @@
           </noise>
         </ray>
-        <plugin name="gazebo_ros_laser_controller" filename="${gazebo_plugin_name}">
+        <plugin name="ros_laser_controller" type="${plugin_type}">
           <topicName>${ros_topic}</topicName>
           <frameName>${name}_frame</frameName>
@@ -94,5 +94,5 @@
         </plugin>
       </sensor>
-    </gazebo>
+    </webots>
   </xacro:macro>
 </robot>
