Commit message: ensuring compatibility with gazebo

File: hector_sensors_description/urdf/camera360.urdf.xacro (robot description, xacro)
@@ -1,4 +1,5 @@
 <?xml version="1.0"?>
 <robot xmlns:xacro="http://www.ros.org/wiki/xacro">
+  <xacro:arg name="simulator" default="gazebo"/>
   <xacro:property name="M_PI" value="3.1415926535897931" />
   <xacro:property name="default_collision_radius" value="0.025" />
@@ -63,5 +64,5 @@
     </joint>
     <link name="${name}_${right_cam_name}_optical_frame"/>
-    <webots reference="${name}_${right_cam_name}_link">
+    <gazebo reference="${name}_${right_cam_name}_link">
       <sensor type="wideanglecamera" name="${name}_${right_cam_name}_camera_sensor">
         <update_rate>${update_rate}</update_rate>
@@ -97,12 +98,14 @@
           </lens>
         </camera>
-        <!--plugin name="${name}_${right_cam_name}_camera_controller" filename="libgazebo_ros_camera.so">
-          <cameraName>${name}/${right_cam_name}</cameraName>
-          <imageTopicName>${ros_topic}</imageTopicName>
-          <cameraInfoTopicName>not_used</cameraInfoTopicName>
-          <frameName>${name}_${right_cam_name}_optical_frame</frameName>
-        </plugin-->
+        <xacro:if value="${simulator == 'gazebo'}">
+          <plugin name="${name}_${right_cam_name}_camera_controller" filename="libgazebo_ros_camera.so">
+            <cameraName>${name}/${right_cam_name}</cameraName>
+            <imageTopicName>${ros_topic}</imageTopicName>
+            <cameraInfoTopicName>not_used</cameraInfoTopicName>
+            <frameName>${name}_${right_cam_name}_optical_frame</frameName>
+          </plugin>
+        </xacro:if>
       </sensor>
-    </webots>
+    </gazebo>
     <joint name="${name}_${left_cam_name}_optical_joint" type="fixed">
       <xacro:insert_block name="calibration" />
@@ -117,5 +120,5 @@
     </joint>
     <link name="${name}_${left_cam_name}_link"/>
-    <webots reference="${name}_${left_cam_name}_link">
+    <gazebo reference="${name}_${left_cam_name}_link">
       <sensor type="wideanglecamera" name="${name}_${left_cam_name}_camera_sensor">
         <update_rate>${update_rate}</update_rate>
@@ -151,12 +154,14 @@
           </lens>
         </camera>
-        <!--plugin name="${name}_${left_cam_name}_camera_controller" filename="libgazebo_ros_camera.so">
-          <cameraName>${name}/${left_cam_name}</cameraName>
-          <imageTopicName>${ros_topic}</imageTopicName>
-          <cameraInfoTopicName>not_used</cameraInfoTopicName>
-          <frameName>${name}_${left_cam_name}_optical_frame</frameName>
-        </plugin-->
+        <xacro:if value="${simulator == 'gazebo'}">
+          <plugin name="${name}_${left_cam_name}_camera_controller" filename="libgazebo_ros_camera.so">
+            <cameraName>${name}/${left_cam_name}</cameraName>
+            <imageTopicName>${ros_topic}</imageTopicName>
+            <cameraInfoTopicName>not_used</cameraInfoTopicName>
+            <frameName>${name}_${left_cam_name}_optical_frame</frameName>
+          </plugin>
+        </xacro:if>
       </sensor>
-    </webots>
+    </gazebo>
   </xacro:macro>
 </robot>

File: hector_sensors_description/urdf/flir_boson_640_8_7_mm.xacro (robot description, xacro)
@@ -1,4 +1,5 @@
 <?xml version="1.0" encoding="UTF-8"?>
 <robot xmlns:xacro="http://www.ros.org/wiki/xacro">
+  <xacro:arg name="simulator" default="gazebo"/>
   <xacro:include filename="$(find hector_xacro_tools)/urdf/sensor_macros.urdf.xacro" />
   <xacro:macro name="flir_boson_640_camera_model" params="name parent *origin add_geometry">
@@ -70,12 +71,14 @@
           </clip>
         </camera>
-        <plugin name="thermal_camera_controller" filename="libgazebo_ros_thermal_camera.so">
-          <alwaysOn>true</alwaysOn>
-          <updateRate>9</updateRate>
-          <cameraName>${name}</cameraName>
-          <imageTopicName>image_raw</imageTopicName>
-          <cameraInfoTopicName>camera_info</cameraInfoTopicName>
-          <frameName>${name}_optical_frame</frameName>
-        </plugin>
+        <xacro:if value="${simulator == 'gazebo'}">
+          <plugin name="thermal_camera_controller" filename="libgazebo_ros_thermal_camera.so">
+            <alwaysOn>true</alwaysOn>
+            <updateRate>9</updateRate>
+            <cameraName>${name}</cameraName>
+            <imageTopicName>image_raw</imageTopicName>
+            <cameraInfoTopicName>camera_info</cameraInfoTopicName>
+            <frameName>${name}_optical_frame</frameName>
+          </plugin>
+        </xacro:if>
       </sensor>
     </gazebo>

File: hector_sensors_description/urdf/generic_camera.urdf.xacro (robot description, xacro)
@@ -1,4 +1,5 @@
 <?xml version="1.0"?>
 <robot xmlns:xacro="http://www.ros.org/wiki/xacro">
+  <xacro:arg name="simulator" default="gazebo"/>
   <xacro:property name="M_PI" value="3.1415926535897931" />
   <xacro:macro name="generic_camera" params="name parent *origin ros_topic cam_info_topic update_rate res_x res_y image_format hfov">
@@ -36,5 +37,5 @@
     </joint>
     <link name="${name}_optical_frame"/>
-    <webots reference="${name}_link">
+    <gazebo reference="${name}_link">
       <sensor type="camera" name="${name}_camera_sensor">
         <update_rate>${update_rate}</update_rate>
@@ -51,6 +52,14 @@
           </clip>
         </camera>
+        <xacro:if value="${simulator == 'gazebo'}">
+          <plugin name="${name}_camera_controller" filename="libgazebo_ros_camera.so">
+            <cameraName>${name}</cameraName>
+            <imageTopicName>${ros_topic}</imageTopicName>
+            <cameraInfoTopicName>${cam_info_topic}</cameraInfoTopicName>
+            <frameName>${name}_optical_frame</frameName>
+          </plugin>
+        </xacro:if>
       </sensor>
-    </webots>
+    </gazebo>
   </xacro:macro>
 </robot>

File: hector_sensors_description/urdf/realsense_d435_camera.urdf.xacro (robot description, xacro)
@@ -9,4 +9,6 @@
 -->
 <robot xmlns:xacro="http://www.ros.org/wiki/xacro">
+  <xacro:arg name="simulator" default="gazebo"/>
+  <xacro:property name="simulator" value="$(arg simulator)"/>
   <xacro:property name="M_PI" value="3.1415926535897931" />
   <xacro:property name="realsense_d435_width" value="0.09"/>
@@ -48,7 +50,7 @@
         </collision>
       </link>
-      <webots reference="${name}_link">
+      <gazebo reference="${name}_link">
         <material>Gazebo/Grey</material>
-      </webots>
+      </gazebo>
     </xacro:macro>
     <xacro:macro name="realsense_d435_camera_model_with_mount" params="name parent *origin">
@@ -74,5 +76,5 @@
     </xacro:macro>
     <xacro:macro name="realsense_d435_camera_gazebo_plugin_macro" params="name parent image_topic depth_topic:=image_raw depth_points_topic frame_name:=color min_range max_range update_rate">
-      <webots reference="${name}_link">
+      <gazebo reference="${name}_link">
         <sensor type="rgbd" name="${name}">
           <update_rate>${update_rate}</update_rate>
@@ -89,19 +91,21 @@
             </clip>
           </camera>
-          <!--plugin name="${name}_camera_controller" filename="libgazebo_ros_openni_kinect.so">
-            <cameraName>${name}</cameraName>
-            <imageTopicName>color/${image_topic}</imageTopicName>
-            <cameraInfoTopicName>color/camera_info</cameraInfoTopicName>
-            <depthImageTopicName>depth/${depth_topic}</depthImageTopicName>
-            <depthImageCameraInfoTopicName>depth/camera_info</depthImageCameraInfoTopicName>
-            <pointCloudTopicName>${depth_points_topic}</pointCloudTopicName>
-            <frameName>${name}_${frame_name}_optical_frame</frameName-->
-            <!-- Important information about frames: Currently, this plugin only supports simulation of color image and depth image/cloud from a single frame.
-            This frame is given in the <gazebo reference=""> tag above and is set to the ${name}_link which coincides with the depth camera frame. The camera axis is the X-axis. ROS requires an optical frame
-            with the Z-axis as camera axis. It is advised to use the depth_optical_frame for this purpose (frame_name="depth"), even though camera images will have the same frame.
-            The color_optical_frame does not coincide with the depth_optical_frame, so depth image/cloud will be misaligned! -->
-          <!--/plugin-->
+          <xacro:if value="${simulator == 'gazebo'}">
+            <plugin name="${name}_camera_controller" filename="libgazebo_ros_openni_kinect.so">
+              <cameraName>${name}</cameraName>
+              <imageTopicName>color/${image_topic}</imageTopicName>
+              <cameraInfoTopicName>color/camera_info</cameraInfoTopicName>
+              <depthImageTopicName>depth/${depth_topic}</depthImageTopicName>
+              <depthImageCameraInfoTopicName>depth/camera_info</depthImageCameraInfoTopicName>
+              <pointCloudTopicName>${depth_points_topic}</pointCloudTopicName>
+              <frameName>${name}_${frame_name}_optical_frame</frameName>
+              <!-- Important information about frames: Currently, this plugin only supports simulation of color image and depth image/cloud from a single frame.
+              This frame is given in the <gazebo reference=""> tag above and is set to the ${name}_link which coincides with the depth camera frame. The camera axis is the X-axis. ROS requires an optical frame
+              with the Z-axis as camera axis. It is advised to use the depth_optical_frame for this purpose (frame_name="depth"), even though camera images will have the same frame.
+              The color_optical_frame does not coincide with the depth_optical_frame, so depth image/cloud will be misaligned! -->
+            </plugin>
+          </xacro:if>
         </sensor>
-      </webots>
+      </gazebo>
     </xacro:macro>
     <!--

File: hector_sensors_description/urdf/vlp16.urdf.xacro (robot description, xacro)
@@ -1,4 +1,6 @@
 <?xml version="1.0"?>
 <robot xmlns:xacro="http://www.ros.org/wiki/xacro">
+  <xacro:arg name="simulator" default="gazebo"/>
+  <xacro:property name="simulator" value="$(arg simulator)"/>
   <xacro:include filename="$(find hector_xacro_tools)/urdf/inertia_tensors.urdf.xacro"/>
   <xacro:property name="M_PI" value="3.1415926535897931"/>
@@ -46,13 +48,25 @@
       <xacro:insert_block name="origin"/>
     </xacro:vlp16_model>
-    <webots reference="${name}_frame">
-      <xacro:if value="${use_gpu}">
-        <xacro:property name="sensor_type" value="gpu_lidar"/>
-        <xacro:property name="plugin_type" value="lidar"/>
-      </xacro:if >
-      <xacro:unless value="${use_gpu}">
-        <xacro:property name="sensor_type" value="lidar"/>
-        <xacro:property name="plugin_type" value="lidar"/>
-      </xacro:unless>
+    <gazebo reference="${name}_frame">
+      <xacro:if value="${simulator == 'webots'}">
+        <xacro:if value="${use_gpu}">
+          <xacro:property name="sensor_type" value="gpu_lidar"/>
+          <!--xacro:property name="plugin_type" value="lidar"/-->
+        </xacro:if >
+        <xacro:unless value="${use_gpu}">
+          <xacro:property name="sensor_type" value="lidar"/>
+          <!--xacro:property name="plugin_type" value="lidar"/-->
+        </xacro:unless>
+      </xacro:if>
+      <xacro:if value="${simulator == 'gazebo'}">
+        <xacro:if value="${use_gpu}">
+          <xacro:property name="sensor_type" value="gpu_ray"/>
+          <xacro:property name="gazebo_plugin_name" value="libgazebo_ros_velodyne_gpu_laser.so"/>
+        </xacro:if >
+        <xacro:unless value="${use_gpu}">
+          <xacro:property name="sensor_type" value="ray"/>
+          <xacro:property name="gazebo_plugin_name" value="libgazebo_ros_velodyne_laser.so"/>
+        </xacro:unless>
+      </xacro:if>
       <sensor type="${sensor_type}" name="${name}-VLP16">
         <pose>0 0 0 0 0 0</pose>
@@ -85,14 +99,16 @@
           </noise>
         </ray>
-        <plugin name="ros_laser_controller" type="${plugin_type}">
-          <topicName>${ros_topic}</topicName>
-          <frameName>${name}_frame</frameName>
-          <organize_cloud>${organize_cloud}</organize_cloud>
-          <min_range>${min_range}</min_range>
-          <max_range>${max_range}</max_range>
-          <gaussianNoise>0.008</gaussianNoise>
-        </plugin>
+        <xacro:if value="${simulator == 'gazebo'}">
+          <plugin name="ros_laser_controller" type="${gazebo_plugin_name}">
+            <topicName>${ros_topic}</topicName>
+            <frameName>${name}_frame</frameName>
+            <organize_cloud>${organize_cloud}</organize_cloud>
+            <min_range>${min_range}</min_range>
+            <max_range>${max_range}</max_range>
+            <gaussianNoise>0.008</gaussianNoise>
+          </plugin>
+        </xacro:if>
       </sensor>
-    </webots>
+    </gazebo>
   </xacro:macro>
 </robot>

Commit message: changed xacro if as it makes problems with different versions

File: hector_sensors_description/urdf/camera360.urdf.xacro (robot description, xacro)
@@ -98,5 +98,5 @@
           </lens>
         </camera>
-        <xacro:if value="${simulator == 'gazebo'}">
+        <xacro:if value="${'$(arg simulator)' == 'gazebo'}">
           <plugin name="${name}_${right_cam_name}_camera_controller" filename="libgazebo_ros_camera.so">
             <cameraName>${name}/${right_cam_name}</cameraName>
@@ -154,5 +154,5 @@
           </lens>
         </camera>
-        <xacro:if value="${simulator == 'gazebo'}">
+        <xacro:if value="${'$(arg simulator)' == 'gazebo'}">
           <plugin name="${name}_${left_cam_name}_camera_controller" filename="libgazebo_ros_camera.so">
             <cameraName>${name}/${left_cam_name}</cameraName>

File: hector_sensors_description/urdf/flir_boson_640_8_7_mm.xacro (robot description, xacro)
@@ -71,5 +71,5 @@
           </clip>
         </camera>
-        <xacro:if value="${simulator == 'gazebo'}">
+        <xacro:if value="${'$(arg simulator)' == 'gazebo'}">
           <plugin name="thermal_camera_controller" filename="libgazebo_ros_thermal_camera.so">
             <alwaysOn>true</alwaysOn>

File: hector_sensors_description/urdf/generic_camera.urdf.xacro (robot description, xacro)
@@ -52,5 +52,5 @@
           </clip>
         </camera>
-        <xacro:if value="${simulator == 'gazebo'}">
+        <xacro:if value="${'$(arg simulator)' == 'gazebo'}">
           <plugin name="${name}_camera_controller" filename="libgazebo_ros_camera.so">
             <cameraName>${name}</cameraName>

File: hector_sensors_description/urdf/realsense_d435_camera.urdf.xacro (robot description, xacro)
@@ -10,5 +10,4 @@
 <robot xmlns:xacro="http://www.ros.org/wiki/xacro">
   <xacro:arg name="simulator" default="gazebo"/>
-  <xacro:property name="simulator" value="$(arg simulator)"/>
   <xacro:property name="M_PI" value="3.1415926535897931" />
   <xacro:property name="realsense_d435_width" value="0.09"/>
@@ -91,5 +90,5 @@
             </clip>
           </camera>
-          <xacro:if value="${simulator == 'gazebo'}">
+          <xacro:if value="${'$(arg simulator)' == 'gazebo'}">
             <plugin name="${name}_camera_controller" filename="libgazebo_ros_openni_kinect.so">
               <cameraName>${name}</cameraName>

File: hector_sensors_description/urdf/vlp16.urdf.xacro (robot description, xacro)
@@ -2,5 +2,4 @@
 <robot xmlns:xacro="http://www.ros.org/wiki/xacro">
   <xacro:arg name="simulator" default="gazebo"/>
-  <xacro:property name="simulator" value="$(arg simulator)"/>
   <xacro:include filename="$(find hector_xacro_tools)/urdf/inertia_tensors.urdf.xacro"/>
   <xacro:property name="M_PI" value="3.1415926535897931"/>
@@ -49,5 +48,5 @@
     </xacro:vlp16_model>
     <gazebo reference="${name}_frame">
-      <xacro:if value="${simulator == 'webots'}">
+      <xacro:if value="${'$(arg simulator)' == 'webots'}">
         <xacro:if value="${use_gpu}">
           <xacro:property name="sensor_type" value="gpu_lidar"/>
@@ -59,5 +58,5 @@
         </xacro:unless>
       </xacro:if>
-      <xacro:if value="${simulator == 'gazebo'}">
+      <xacro:if value="${'$(arg simulator)' == 'gazebo'}">
         <xacro:if value="${use_gpu}">
           <xacro:property name="sensor_type" value="gpu_ray"/>
@@ -99,5 +98,5 @@
           </noise>
         </ray>
-        <xacro:if value="${simulator == 'gazebo'}">
+        <xacro:if value="${'$(arg simulator)' == 'gazebo'}">
           <plugin filename="libgazebo_ros_velodyne_gpu_laser.so" name="gazebo_ros_laser_controller">
             <topicName>${ros_topic}</topicName>
