Commit message: added a seperate points topic to mimic the real sensor

File: hector_sensors_description/urdf/os0-128.urdf.xacro (robot description, xacro)
@@ -37,9 +37,9 @@
   </xacro:macro>
   <xacro:macro name="os0_128" params="name parent *origin ros_topic">
-    <xacro:os0_128_advanced_parameters name="${name}" parent="${parent}" ros_topic="${ros_topic}" update_rate="10" horizontal_samples="512" vertical_samples="8" min_range="0.45" max_range="100">
+    <xacro:os0_128_advanced_parameters name="${name}" parent="${parent}" update_rate="10" horizontal_samples="512" vertical_samples="8" min_range="0.45" max_range="100">
       <xacro:insert_block name="origin"/>
     </xacro:os0_128_advanced_parameters>
   </xacro:macro>
-  <xacro:macro name="os0_128_advanced_parameters" params="name parent *origin ros_topic update_rate horizontal_samples vertical_samples min_range max_range use_gpu:='false'">
+  <xacro:macro name="os0_128_advanced_parameters" params="name parent *origin update_rate horizontal_samples vertical_samples min_range max_range use_gpu:='false'">
     <xacro:os0_128_model name="${name}" parent="${parent}">
       <xacro:insert_block name="origin"/>
@@ -85,5 +85,5 @@
         </ray>
         <plugin name="gazebo_ros_laser_controller" filename="${gazebo_plugin_name}">
-          <topicName>${ros_topic}</topicName>
+          <topicName>${name}/points</topicName>
           <frameName>${name}_frame</frameName>
           <min_range>${min_range}</min_range>

Commit message: added os0

File: hector_sensors_description/urdf/os0-128.urdf.xacro (robot description, xacro)
@@ -11,13 +11,13 @@
       <xacro:inertial_sphere mass="0.992" diameter="0.08082"/>
       <visual>
-        <origin xyz="0 0 -0.000825" rpy="0 0 0" />
+        <origin xyz="0 0 -0.062825" rpy="0 0 0" />
         <geometry>
-          <cylinder radius="0.04041" length="0.0735"/>
+          <mesh filename="package://hector_sensors_description/meshes/ouster_os0/os0_baseplate.dae" scale="0.001 0.001 0.001"/>
         </geometry>
       </visual>
       <visual>
-        <origin xyz="0 0 -0.047825" rpy="0 0 0"/>
+        <origin xyz="0 0 -0.040825" rpy="0 0 0" />
         <geometry>
-          <box size="0.11 0.11 0.0205"/>
+          <mesh filename="package://hector_sensors_description/meshes/ouster_os0/os0.dae" scale="0.001 0.001 0.001"/>
         </geometry>
       </visual>

Commit message: Add missing parameter

File: hector_sensors_description/urdf/os0-128.urdf.xacro (robot description, xacro)
@@ -41,5 +41,5 @@
     </xacro:os0_128_advanced_parameters>
   </xacro:macro>
-  <xacro:macro name="os0_128_advanced_parameters" params="name parent *origin update_rate horizontal_samples vertical_samples min_range max_range use_gpu:='false'">
+  <xacro:macro name="os0_128_advanced_parameters" params="name parent *origin update_rate horizontal_samples vertical_samples min_range max_range use_gpu:='false' organize_cloud">
     <xacro:os0_128_model name="${name}" parent="${parent}">
       <xacro:insert_block name="origin"/>

Commit message: Add point cloud structure parameters

File: hector_sensors_description/urdf/os0-128.urdf.xacro (robot description, xacro)
@@ -41,5 +41,6 @@
     </xacro:os0_128_advanced_parameters>
   </xacro:macro>
-  <xacro:macro name="os0_128_advanced_parameters" params="name parent *origin update_rate horizontal_samples vertical_samples min_range max_range use_gpu:='false' organize_cloud">
+  <xacro:macro name="os0_128_advanced_parameters" params="name parent *origin update_rate horizontal_samples vertical_samples min_range max_range use_gpu:='false'
+  organize_cloud:='true' row_major:='false' rings_top_bottom:='false' columns_left_right='false' zeros_instead_of_nans:='false'">
     <xacro:os0_128_model name="${name}" parent="${parent}">
       <xacro:insert_block name="origin"/>
@@ -90,9 +91,9 @@
           <max_range>${max_range}</max_range>
           <gaussianNoise>0.008</gaussianNoise>
-          <organize_cloud>true</organize_cloud>
-          <row_major>false</row_major>
-          <rings_top_bottom>true</rings_top_bottom>
-          <columns_left_right>false</columns_left_right>
-          <zeros_instead_of_nans>false</zeros_instead_of_nans>
+          <organize_cloud>${organize_cloud}</organize_cloud>
+          <row_major>${row_major}</row_major>
+          <rings_top_bottom>${rings_top_bottom}</rings_top_bottom>
+          <columns_left_right>${columns_left_right}</columns_left_right>
+          <zeros_instead_of_nans>${zeros_instead_of_nans}</zeros_instead_of_nans>
         </plugin>
       </sensor>

Commit message: Add point cloud structure parameters

File: hector_sensors_description/urdf/os0-128.urdf.xacro (robot description, xacro)
@@ -41,5 +41,6 @@
     </xacro:os0_128_advanced_parameters>
   </xacro:macro>
-  <xacro:macro name="os0_128_advanced_parameters" params="name parent *origin update_rate horizontal_samples vertical_samples min_range max_range use_gpu:='false'">
+  <xacro:macro name="os0_128_advanced_parameters" params="name parent *origin update_rate horizontal_samples vertical_samples min_range max_range use_gpu:='false'
+  organize_cloud:='true' row_major:='false' rings_top_bottom:='false' columns_left_right='false' zeros_instead_of_nans:='false'">
     <xacro:os0_128_model name="${name}" parent="${parent}">
       <xacro:insert_block name="origin"/>
@@ -90,4 +91,9 @@
           <max_range>${max_range}</max_range>
           <gaussianNoise>0.008</gaussianNoise>
+          <organize_cloud>${organize_cloud}</organize_cloud>
+          <row_major>${row_major}</row_major>
+          <rings_top_bottom>${rings_top_bottom}</rings_top_bottom>
+          <columns_left_right>${columns_left_right}</columns_left_right>
+          <zeros_instead_of_nans>${zeros_instead_of_nans}</zeros_instead_of_nans>
         </plugin>
       </sensor>
