Commit message: -URDF hardware interface changes for new gazebo ros control style (#185)

File: hector_components_description/urdf/spinning_lidar_mount.urdf.xacro (robot description, xacro)
@@ -65,5 +65,7 @@
     <transmission name="${name}_spinning_lidar_spin_joint_transmssion">
       <type>transmission_interface/SimpleTransmission</type>
-      <joint name="${name}_spinning_lidar_spin_joint"/>
+      <joint name="${name}_spinning_lidar_spin_joint">
+        <hardwareInterface>EffortJointInterface</hardwareInterface>
+      </joint>
       <actuator name="${name}_spinning_lidar_spin_joint_motor">
         <hardwareInterface>EffortJointInterface</hardwareInterface>

Commit message: Update LIDAR mount with reasonable inertia

File: hector_components_description/urdf/spinning_lidar_mount.urdf.xacro (robot description, xacro)
@@ -1,4 +1,5 @@
 <?xml version="1.0"?>
-<robot xmlns:xacro="http://playerstage.sourceforge.net/gazebo/xmlschema/#interface">
+<robot xmlns:xacro="http://ros.org/wiki/xacro">
+  <xacro:include filename="$(find hector_xacro_tools)/urdf/inertia_tensors.urdf.xacro" />
   <property name="M_PI" value="3.14159265359"/>
   <macro name="spinning_lidar_macro" params="parent name angle_deg *origin">
@@ -10,10 +11,7 @@
     </joint>
     <link name="${name}_spinning_lidar_root_link">
-      <origin xyz="0 0 0" rpy="0 0 0"/>
-      <inertial>
-        <mass value="1.0"/>
-        <origin xyz="0.0 0.0 0.5" rpy="0 0 0"/>
-        <inertia ixx="0.005" ixy="0.0" ixz="0.0" iyy="0.005" iyz="0.0" izz="0.005"/>
-      </inertial>
+      <xacro:inertial_sphere_with_pose mass="0.1" diameter="0.03">
+        <origin xyz="0.0 0.0 -0.0" rpy="0 0 0"/>
+      </xacro:inertial_sphere_with_pose>
       <collision name="collision">
         <origin xyz="0.0 0.0 0" rpy="0 0 0"/>
@@ -37,14 +35,11 @@
       <origin xyz="0 0 0.02" rpy="0 ${0 * M_PI/180.0} 0"/>
       <axis xyz="0 0 1" rpy="0 0 0"/>
-      <limit effort="100" velocity="100"/>
+      <limit effort="1000" velocity="100"/>
       <joint_properties damping="0.0" friction="0.0"/>
     </joint>
     <link name="${name}_spinning_lidar_spin_link">
-      <origin xyz="0 0 0" rpy="0 0 0"/>
-      <inertial>
-        <mass value="1.0"/>
-        <origin xyz="0.0 0.0 0.5" rpy="0 0 0"/>
-        <inertia ixx="0.005" ixy="0.0" ixz="0.0" iyy="0.005" iyz="0.0" izz="0.005"/>
-      </inertial>
+      <xacro:inertial_sphere_with_pose mass="0.1" diameter="0.03">
+        <origin xyz="0.0 0.0 -0.0" rpy="0 0 0"/>
+      </xacro:inertial_sphere_with_pose>
       <collision name="collision">
         <origin xyz="0.0 0.0 0" rpy="0 0 0"/>
