Commit message: -Formatting

File: hector_components_description/urdf/spinning_hokuyo_utm30lx.urdf.xacro (robot description, xacro)
@@ -1,15 +1,14 @@
 <?xml version="1.0"?>
-<robot
-  xmlns:xacro="http://playerstage.sourceforge.net/gazebo/xmlschema/#interface">
-  <property name="M_PI" value="3.14159265359" />
-  <xacro:include filename="$(find hector_components_description)/urdf/spinning_lidar_mount.urdf.xacro" />
-  <xacro:include filename="$(find hector_sensors_description)/urdf/hokuyo_utm30lx.urdf.xacro" />
+<robot xmlns:xacro="http://playerstage.sourceforge.net/gazebo/xmlschema/#interface">
+  <property name="M_PI" value="3.14159265359"/>
+  <xacro:include filename="$(find hector_components_description)/urdf/spinning_lidar_mount.urdf.xacro"/>
+  <xacro:include filename="$(find hector_sensors_description)/urdf/hokuyo_utm30lx.urdf.xacro"/>
   <macro name="spinning_hokuyo_utm30lx_macro" params="parent name angle_deg *origin">
     <spinning_lidar_macro parent="base_link" name="mid" angle_deg="45">
       <origin xyz="0 0 0.5" rpy="0 0 0"/>
-    </spinning_lidar_macro >
+    </spinning_lidar_macro>
     <xacro:hokuyo_utm30lx name="hokuyo_laser" parent="mid_spinning_lidar_spin_link" ros_topic="${name}_spinning_lidar}/scan" update_rate="40" ray_count="1040" min_angle="130" max_angle="-130">
-       <origin xyz="0.00 -0.0 0.055" rpy="0 ${angle_deg * M_PI/180.0} 0"/>
-     </xacro:hokuyo_utm30lx>
-    </macro>
+      <origin xyz="0.00 -0.0 0.055" rpy="0 ${angle_deg * M_PI/180.0} 0"/>
+    </xacro:hokuyo_utm30lx>
+  </macro>
 </robot>

File: hector_components_description/urdf/spinning_lidar_mount.urdf.xacro (robot description, xacro)
@@ -1,77 +1,67 @@
 <?xml version="1.0"?>
-<robot
-  xmlns:xacro="http://playerstage.sourceforge.net/gazebo/xmlschema/#interface">
-  <property name="flipper_base_mass" value="2.0"/>
-  <property name="flipper_x" value="0.3"/>
-  <property name="flipper_y" value="0.1"/>
-  <property name="flipper_z" value="0.1"/>
-  <property name="M_PI" value="3.14159265359" />
+<robot xmlns:xacro="http://playerstage.sourceforge.net/gazebo/xmlschema/#interface">
+  <property name="M_PI" value="3.14159265359"/>
   <macro name="spinning_lidar_macro" params="parent name angle_deg *origin">
- <!-- front is either 1 (for front flipper) or -1 (for back flipper) -->
-<joint name="${name}_spinning_lidar_base_joint" type="fixed">
-  <insert_block name="origin"/>
+    <joint name="${name}_spinning_lidar_base_joint" type="fixed">
+      <insert_block name="origin"/>
       <axis xyz="0 1 0"/>
       <parent link="${parent}"/>
       <child link="${name}_spinning_lidar_base_link"/>
     </joint>
-<link name="${name}_spinning_lidar_base_link">
-<origin xyz="0 0 0" rpy="0 0 0" />
-                <inertial>
-                <mass value="1.0" />
-                <origin xyz="0.0 0.0 0.5" rpy="0 0 0" />
-                <inertia ixx="0.005" ixy="0.0" ixz="0.0"
-                         iyy="0.005" iyz="0.0"
-                         izz="0.005" />
-            </inertial>
-            <collision name='collision'>
-             <origin xyz="0.0 0.0 0" rpy="0 0 0" />
-                <geometry>
-                  <box size="0.05 0.05 0.015"/>
-                </geometry>
-            </collision>
-            <visual name='visual'>
-                <origin xyz="0.0 0.0 0" rpy="0 0 0" />
-                <geometry>
-                  <box size="0.05 0.05 0.015"/>
-                </geometry>
-                <material name="DarkGrey" >
-                    <color rgba="0.3 0.3 0.3 1"/>
-                </material>
-            </visual>
-        </link>
+    <link name="${name}_spinning_lidar_base_link">
+      <origin xyz="0 0 0" rpy="0 0 0"/>
+      <inertial>
+        <mass value="1.0"/>
+        <origin xyz="0.0 0.0 0.5" rpy="0 0 0"/>
+        <inertia ixx="0.005" ixy="0.0" ixz="0.0" iyy="0.005" iyz="0.0" izz="0.005"/>
+      </inertial>
+      <collision name="collision">
+        <origin xyz="0.0 0.0 0" rpy="0 0 0"/>
+        <geometry>
+          <box size="0.05 0.05 0.015"/>
+        </geometry>
+      </collision>
+      <visual name="visual">
+        <origin xyz="0.0 0.0 0" rpy="0 0 0"/>
+        <geometry>
+          <box size="0.05 0.05 0.015"/>
+        </geometry>
+        <material name="DarkGrey">
+          <color rgba="0.3 0.3 0.3 1"/>
+        </material>
+      </visual>
+    </link>
     <joint name="${name}_spinning_lidar_spin_joint" type="continuous">
       <parent link="${name}_spinning_lidar_base_link"/>
       <child link="${name}_spinning_lidar_spin_link"/>
-      <origin xyz="0 0 0.02" rpy="0 ${0 * M_PI/180.0} 0" />
-      <axis xyz="0 0 1" rpy="0 0 0" />
+      <origin xyz="0 0 0.02" rpy="0 ${0 * M_PI/180.0} 0"/>
+      <axis xyz="0 0 1" rpy="0 0 0"/>
       <limit effort="100" velocity="100"/>
       <joint_properties damping="0.0" friction="0.0"/>
     </joint>
     <link name="${name}_spinning_lidar_spin_link">
-<origin xyz="0 0 0" rpy="0 0 0" />
-                <inertial>
-                <mass value="1.0" />
-                <origin xyz="0.0 0.0 0.5" rpy="0 0 0" />
-                <inertia ixx="0.005" ixy="0.0" ixz="0.0"
-                         iyy="0.005" iyz="0.0"
-                         izz="0.005" />
-            </inertial>
-            <collision name='collision'>
-             <origin xyz="0.0 0.0 0" rpy="0 0 0" />
-                <geometry>
-                  <box size="0.05 0.05 0.015"/>
-                </geometry>
-            </collision>
-            <visual name='visual'>
-                <origin xyz="0.0 0.0 0" rpy="0 0 0" />
-                <geometry>
-                  <box size="0.05 0.05 0.015"/>
-                </geometry>
-                <material name="DarkGrey" >
-                    <color rgba="0.3 0.3 0.3 1"/>
-                </material>
-            </visual>
-        </link>
-<gazebo reference="${name}_spinning_lidar_base_link">
+      <origin xyz="0 0 0" rpy="0 0 0"/>
+      <inertial>
+        <mass value="1.0"/>
+        <origin xyz="0.0 0.0 0.5" rpy="0 0 0"/>
+        <inertia ixx="0.005" ixy="0.0" ixz="0.0" iyy="0.005" iyz="0.0" izz="0.005"/>
+      </inertial>
+      <collision name="collision">
+        <origin xyz="0.0 0.0 0" rpy="0 0 0"/>
+        <geometry>
+          <box size="0.05 0.05 0.015"/>
+        </geometry>
+      </collision>
+      <visual name="visual">
+        <origin xyz="0.0 0.0 0" rpy="0 0 0"/>
+        <geometry>
+          <box size="0.05 0.05 0.015"/>
+        </geometry>
+        <material name="DarkGrey">
+          <color rgba="0.3 0.3 0.3 1"/>
+        </material>
+      </visual>
+    </link>
+    <gazebo reference="${name}_spinning_lidar_base_link">
       <material>Gazebo/Green</material>
     </gazebo>
@@ -79,4 +69,4 @@
       <material>Gazebo/Green</material>
     </gazebo>
-    </macro>
+  </macro>
 </robot>

Commit message: -Add gazebo_ros_control required tags to spinning lidar macros

File: hector_components_description/urdf/spinning_hokuyo_utm30lx.urdf.xacro (robot description, xacro)
@@ -5,8 +5,8 @@
   <xacro:include filename="$(find hector_sensors_description)/urdf/hokuyo_utm30lx.urdf.xacro"/>
   <macro name="spinning_hokuyo_utm30lx_macro" params="parent name angle_deg *origin">
-    <spinning_lidar_macro parent="base_link" name="mid" angle_deg="45">
+    <spinning_lidar_macro parent="base_link" name="${name}" angle_deg="45">
       <origin xyz="0 0 0.5" rpy="0 0 0"/>
     </spinning_lidar_macro>
-    <xacro:hokuyo_utm30lx name="hokuyo_laser" parent="mid_spinning_lidar_spin_link" ros_topic="${name}_spinning_lidar}/scan" update_rate="40" ray_count="1040" min_angle="130" max_angle="-130">
+    <xacro:hokuyo_utm30lx name="hokuyo_laser" parent="${name}_spinning_lidar_spin_link" ros_topic="${name}_spinning_lidar/scan" update_rate="40" ray_count="1040" min_angle="130" max_angle="-130">
       <origin xyz="0.00 -0.0 0.055" rpy="0 ${angle_deg * M_PI/180.0} 0"/>
     </xacro:hokuyo_utm30lx>

File: hector_components_description/urdf/spinning_lidar_mount.urdf.xacro (robot description, xacro)
@@ -3,11 +3,11 @@
   <property name="M_PI" value="3.14159265359"/>
   <macro name="spinning_lidar_macro" params="parent name angle_deg *origin">
-    <joint name="${name}_spinning_lidar_base_joint" type="fixed">
+    <joint name="${name}_spinning_lidar_root_joint" type="fixed">
       <insert_block name="origin"/>
       <axis xyz="0 1 0"/>
       <parent link="${parent}"/>
-      <child link="${name}_spinning_lidar_base_link"/>
+      <child link="${name}_spinning_lidar_root_link"/>
     </joint>
-    <link name="${name}_spinning_lidar_base_link">
+    <link name="${name}_spinning_lidar_root_link">
       <origin xyz="0 0 0" rpy="0 0 0"/>
       <inertial>
@@ -33,5 +33,5 @@
     </link>
     <joint name="${name}_spinning_lidar_spin_joint" type="continuous">
-      <parent link="${name}_spinning_lidar_base_link"/>
+      <parent link="${name}_spinning_lidar_root_link"/>
       <child link="${name}_spinning_lidar_spin_link"/>
       <origin xyz="0 0 0.02" rpy="0 ${0 * M_PI/180.0} 0"/>
@@ -63,9 +63,17 @@
       </visual>
     </link>
-    <gazebo reference="${name}_spinning_lidar_base_link">
-      <material>Gazebo/Green</material>
+    <transmission name="${name}_spinning_lidar_spin_joint_transmssion">
+      <type>transmission_interface/SimpleTransmission</type>
+      <joint name="${name}_spinning_lidar_spin_joint"/>
+      <actuator name="${name}_spinning_lidar_spin_joint_motor">
+        <hardwareInterface>EffortJointInterface</hardwareInterface>
+        <mechanicalReduction>1</mechanicalReduction>
+      </actuator>
+    </transmission>
+    <gazebo reference="${name}_spinning_lidar_root_link">
+      <material>Gazebo/Grey</material>
     </gazebo>
     <gazebo reference="${name}_spinning_lidar_spin_link">
-      <material>Gazebo/Green</material>
+      <material>Gazebo/Grey</material>
     </gazebo>
   </macro>

Commit message: -Fix origin block not getting used correctly

File: hector_components_description/urdf/spinning_hokuyo_utm30lx.urdf.xacro (robot description, xacro)
@@ -6,5 +6,5 @@
   <macro name="spinning_hokuyo_utm30lx_macro" params="parent name angle_deg *origin">
     <spinning_lidar_macro parent="base_link" name="${name}" angle_deg="45">
-      <origin xyz="0 0 0.5" rpy="0 0 0"/>
+      <insert_block name="origin"/>
     </spinning_lidar_macro>
     <xacro:hokuyo_utm30lx name="hokuyo_laser" parent="${name}_spinning_lidar_spin_link" ros_topic="${name}_spinning_lidar/scan" update_rate="40" ray_count="1040" min_angle="130" max_angle="-130">

Commit message: -Add second spinning hokuyo variant

File: hector_components_description/urdf/spinning_hokuyo_utm30lx.urdf.xacro (robot description, xacro)
@@ -8,7 +8,15 @@
       <insert_block name="origin"/>
     </spinning_lidar_macro>
-    <xacro:hokuyo_utm30lx name="hokuyo_laser" parent="${name}_spinning_lidar_spin_link" ros_topic="${name}_spinning_lidar/scan" update_rate="40" ray_count="1040" min_angle="130" max_angle="-130">
+    <xacro:hokuyo_utm30lx name="${name}_hokuyo_laser" parent="${name}_spinning_lidar_spin_link" ros_topic="${name}_spinning_lidar/scan" update_rate="40" ray_count="1040" min_angle="130" max_angle="-130">
       <origin xyz="0.00 -0.0 0.055" rpy="0 ${angle_deg * M_PI/180.0} 0"/>
     </xacro:hokuyo_utm30lx>
   </macro>
+  <macro name="spinning_hokuyo_utm30lx_lidar_mount_offset_macro" params="parent name angle_deg *origin">
+    <spinning_lidar_macro parent="base_link" name="${name}" angle_deg="45">
+      <insert_block name="origin"/>
+    </spinning_lidar_macro>
+    <xacro:hokuyo_utm30lx name="${name}_hokuyo_laser" parent="${name}_spinning_lidar_spin_link" ros_topic="${name}_spinning_lidar/scan" update_rate="40" ray_count="1040" min_angle="130" max_angle="-130">
+      <origin xyz="0.03 -0.0 0.055" rpy="0 ${angle_deg * M_PI/180.0} 0"/>
+    </xacro:hokuyo_utm30lx>
+  </macro>
 </robot>

Commit message: Refactor spinning lidar mount

File: hector_components_description/urdf/spinning_hokuyo_utm30lx.urdf.xacro (robot description, xacro)
@@ -17,5 +17,5 @@
     </spinning_lidar_macro>
     <xacro:hokuyo_utm30lx name="${name}_hokuyo_laser" parent="${name}_spinning_lidar_spin_link" ros_topic="${name}_spinning_lidar/scan" update_rate="40" ray_count="1040" min_angle="130" max_angle="-130">
-      <origin xyz="0.03 -0.0 0.055" rpy="0 ${angle_deg * M_PI/180.0} 0"/>
+      <origin xyz=" 0.019760 -0.0  0.157466" rpy="0 ${-angle_deg * M_PI/180.0} ${M_PI}"/>
     </xacro:hokuyo_utm30lx>
   </macro>

File: hector_components_description/urdf/spinning_lidar_mount.urdf.xacro (robot description, xacro)
@@ -33,5 +33,5 @@
       <parent link="${name}_spinning_lidar_root_link"/>
       <child link="${name}_spinning_lidar_spin_link"/>
-      <origin xyz="0 0 0.02" rpy="0 ${0 * M_PI/180.0} 0"/>
+      <origin xyz="0 0 0.00" rpy="0 ${0 * M_PI/180.0} 0"/>
       <axis xyz="0 0 1" rpy="0 0 0"/>
       <limit effort="1000" velocity="100"/>

Commit message: Update rotating hokuyo transform

File: hector_components_description/urdf/spinning_hokuyo_utm30lx.urdf.xacro (robot description, xacro)
@@ -17,5 +17,5 @@
     </spinning_lidar_macro>
     <xacro:hokuyo_utm30lx name="${name}_hokuyo_laser" parent="${name}_spinning_lidar_spin_link" ros_topic="${name}_spinning_lidar/scan" update_rate="40" ray_count="1040" min_angle="130" max_angle="-130">
-      <origin xyz=" 0.019760 -0.0  0.157466" rpy="0 ${-angle_deg * M_PI/180.0} ${M_PI}"/>
+      <origin xyz=" 0.0098995 -0.0  0.1583919" rpy="0 ${-angle_deg * M_PI/180.0} ${M_PI}"/>
     </xacro:hokuyo_utm30lx>
   </macro>

Commit message: Update spinning lidar mount properties

File: hector_components_description/urdf/spinning_hokuyo_utm30lx.urdf.xacro (robot description, xacro)
@@ -17,5 +17,5 @@
     </spinning_lidar_macro>
     <xacro:hokuyo_utm30lx_gpu name="${name}_hokuyo_laser" parent="${name}_spinning_lidar_spin_link" ros_topic="${name}_spinning_lidar/scan" update_rate="40" ray_count="1040" min_angle="-130" max_angle="130">
-      <origin xyz=" 0.0098995 -0.0  0.1583919" rpy="0 ${-angle_deg * M_PI/180.0} ${M_PI}"/>
+      <origin xyz="0.021 0.0  -0.0  " rpy="0 ${-angle_deg * M_PI/180.0} ${M_PI}"/>
     </xacro:hokuyo_utm30lx_gpu>
   </macro>

File: hector_components_description/urdf/spinning_lidar_mount.urdf.xacro (robot description, xacro)
@@ -12,7 +12,7 @@
     <link name="${name}_spinning_lidar_root_link">
       <xacro:inertial_sphere_with_pose mass="0.01" diameter="0.03">
-        <origin xyz="0.0 0.0 -0.0" rpy="0 0 0"/>
+        <origin xyz="0.0 0.0 0.0" rpy="0 0 0"/>
       </xacro:inertial_sphere_with_pose>
-      <collision name="collision">
+<!--      <collision name="collision">
         <origin xyz="0.0 0.0 0" rpy="0 0 0"/>
         <geometry>
@@ -28,5 +28,5 @@
           <color rgba="0.3 0.3 0.3 1"/>
         </material>
-      </visual>
+      </visual>-->
     </link>
     <joint name="${name}_spinning_lidar_spin_joint" type="continuous">
@@ -42,5 +42,5 @@
         <origin xyz="0.0 0.0 -0.0" rpy="0 0 0"/>
       </xacro:inertial_sphere_with_pose>
-      <collision name="collision">
+<!--      <collision name="collision">
         <origin xyz="0.0 0.0 0" rpy="0 0 0"/>
         <geometry>
@@ -56,5 +56,5 @@
           <color rgba="0.3 0.3 0.3 1"/>
         </material>
-      </visual>
+      </visual>-->
     </link>
     <transmission name="${name}_spinning_lidar_spin_joint_transmssion">

Commit message: added makro that allows you to define a calibration transformation

File: hector_components_description/urdf/spinning_hokuyo_utm30lx.urdf.xacro (robot description, xacro)
@@ -13,9 +13,15 @@
   </xacro:macro>
   <xacro:macro name="spinning_hokuyo_utm30lx_lidar_mount_offset_macro" params="parent name scan_topic_in_namespace angle_deg *origin">
+    <xacro:spinning_hokuyo_utm30lx_lidar_calibration_offset_macro parent="${parent}" name="${name}" scan_topic_in_namespace="${scan_topic_in_namespace}" angle_deg="${angle_deg}">
+      <xacro:insert_block name="origin"/>
+      <origin xyz="0.021 0 0" rpy="0 ${-angle_deg * M_PI/180.0} ${M_PI}"/>
+    </xacro:spinning_hokuyo_utm30lx_lidar_calibration_offset_macro>
+  </xacro:macro>
+    <xacro:macro name="spinning_hokuyo_utm30lx_lidar_calibration_offset_macro" params="parent name scan_topic_in_namespace angle_deg *origin *calibration">
     <xacro:spinning_lidar_macro parent="${parent}" name="${name}" angle_deg="45">
       <xacro:insert_block name="origin"/>
     </xacro:spinning_lidar_macro>
     <xacro:hokuyo_utm30lx_gpu name="${name}_hokuyo_laser" parent="${name}_spinning_lidar_spin_link" ros_topic="${name}_spinning_lidar/${scan_topic_in_namespace}" update_rate="40" ray_count="1040" min_angle="-130" max_angle="130">
-      <origin xyz="0.021 0.0  -0.0  " rpy="0 ${-angle_deg * M_PI/180.0} ${M_PI}"/>
+      <xacro:insert_block name="calibration"/>
     </xacro:hokuyo_utm30lx_gpu>
   </xacro:macro>

Commit message: xml tag alignment

File: hector_components_description/urdf/spinning_hokuyo_utm30lx.urdf.xacro (robot description, xacro)
@@ -18,5 +18,5 @@
     </xacro:spinning_hokuyo_utm30lx_lidar_calibration_offset_macro>
   </xacro:macro>
-    <xacro:macro name="spinning_hokuyo_utm30lx_lidar_calibration_offset_macro" params="parent name scan_topic_in_namespace angle_deg *origin *calibration">
+  <xacro:macro name="spinning_hokuyo_utm30lx_lidar_calibration_offset_macro" params="parent name scan_topic_in_namespace angle_deg *origin *calibration">
     <xacro:spinning_lidar_macro parent="${parent}" name="${name}" angle_deg="45">
       <xacro:insert_block name="origin"/>

Commit message: Make no gpu laser work with calibration changes merged in

File: hector_components_description/urdf/spinning_hokuyo_utm30lx.urdf.xacro (robot description, xacro)
@@ -13,9 +13,15 @@
   </xacro:macro>
   <xacro:macro name="spinning_hokuyo_utm30lx_lidar_mount_offset_macro" params="parent name scan_topic_in_namespace angle_deg *origin">
+    <xacro:spinning_hokuyo_utm30lx_lidar_calibration_offset_macro parent="${parent}" name="${name}" scan_topic_in_namespace="${scan_topic_in_namespace}" angle_deg="${angle_deg}">
+      <xacro:insert_block name="origin"/>
+      <origin xyz="0.021 0 0" rpy="0 ${-angle_deg * M_PI/180.0} ${M_PI}"/>
+    </xacro:spinning_hokuyo_utm30lx_lidar_calibration_offset_macro>
+  </xacro:macro>
+  <xacro:macro name="spinning_hokuyo_utm30lx_lidar_calibration_offset_macro" params="parent name scan_topic_in_namespace angle_deg *origin *calibration">
     <xacro:spinning_lidar_macro parent="${parent}" name="${name}" angle_deg="45">
       <xacro:insert_block name="origin"/>
     </xacro:spinning_lidar_macro>
     <xacro:hokuyo_utm30lx name="${name}_hokuyo_laser" parent="${name}_spinning_lidar_spin_link" ros_topic="${name}_spinning_lidar/${scan_topic_in_namespace}" update_rate="40" ray_count="1040" min_angle="-130" max_angle="130">
-      <origin xyz="0.021 0.0  -0.0  " rpy="0 ${-angle_deg * M_PI/180.0} ${M_PI}"/>
+      <xacro:insert_block name="calibration"/>
     </xacro:hokuyo_utm30lx>
   </xacro:macro>
