Commit message: - Add UTM-30LX macro to vision box xacro

File: hector_components_description/urdf/vision_box_common.urdf.xacro (robot description, xacro)
@@ -5,4 +5,5 @@
   <xacro:include filename="$(find hector_sensors_description)/urdf/thermaleye_camera.urdf.xacro"/>
   <xacro:include filename="$(find hector_sensors_description)/urdf/kinect_camera.urdf.xacro"/>
+  <xacro:include filename="$(find hector_sensors_description)/urdf/hokuyo_utm30lx.urdf.xacro" />
   <xacro:macro name="vision_box" params="box_type parent *origin">
     <joint name="top_box_joint" type="fixed">
@@ -117,4 +118,7 @@
       <origin xyz="${kinect_x_position} 0 ${kinect_z_position}" rpy="0 0 0"/>
     </xacro:kinect_camera_model>
+    <xacro:hokuyo_utm30lx name="laser1" parent="laser1_link" ros_topic="laser1/scan" update_rate="40" ray_count="1081" min_angle="135" max_angle="-135">
+      <origin xyz="${laser1_center_x_offset} 0 ${laser1_plane_height}" rpy="0 0 0"/>
+    </xacro:hokuyo_utm30lx>
     <!--   <xacro:include filename="$(find monstertruck_urdf)/hector/$(env ROBOT)_addons.urdf.xacro" />-->
   </xacro:macro>

Commit message: hector_components_description: Re-parent LIDAR and camera mount to top_box_link

File: hector_components_description/urdf/vision_box_common.urdf.xacro (robot description, xacro)
@@ -36,5 +36,5 @@
     <joint name="laser1/x" type="revolute">
       <origin xyz="${x_vision_box_front} 0 ${laser1RollServo_height}" rpy="0 0 0"/>
-      <parent link="base_link"/>
+      <parent link="top_box_link"/>
       <child link="laser1RollServo"/>
       <axis xyz="1 0 0"/>
@@ -83,6 +83,6 @@
     </link>
     <joint name="camera/z" type="revolute">
-      <origin xyz="${x_pos_sensor_head_rel_to_base_link} 0 0.215" rpy="0 0 0"/>
-      <parent link="base_link"/>
+      <origin xyz="${x_pos_sensor_head_rel_to_base_link} 0 0.137" rpy="0 0 0"/>
+      <parent link="top_box_link"/>
       <child link="cameraYawServo"/>
       <axis xyz="0 0 1"/>
@@ -124,6 +124,5 @@
       <origin xyz="${laser1_center_x_offset} 0 ${laser1_plane_height}" rpy="0 0 0"/>
     </xacro:hokuyo_utm30lx>
-    <xacro:vision_box_common_gazebo_plugins>
-    </xacro:vision_box_common_gazebo_plugins>
+    <xacro:vision_box_common_gazebo_plugins/>
     <!--   <xacro:include filename="$(find monstertruck_urdf)/hector/$(env ROBOT)_addons.urdf.xacro" />-->
   </xacro:macro>

File: hector_components_description/urdf/vision_box_dimensions_hector1.urdf.xacro (robot description, xacro)
@@ -4,5 +4,5 @@
   <xacro:property name="x_vision_box_front" value="0.084" />
   <xacro:property name="x_pos_sensor_head_rel_to_base_link" value="${x_vision_box_front-0.027}" />
-  <xacro:property name="laser1RollServo_height" value="0.118" /> <!--between base_link and laser1 roll axis-->
+  <xacro:property name="laser1RollServo_height" value="0.04" /> <!--between base_link and laser1 roll axis-->
   <xacro:property name="cameraYawServo_size_z" value="0.082" /> <!--between upper edge of top and camera pitch axis-->
   <xacro:property name="cameraYawServo_x_position" value="-0.027" /> <!--between front edge of top and camera yaw axis-->

File: hector_components_description/urdf/vision_box_dimensions_hector2.urdf.xacro (robot description, xacro)
@@ -4,5 +4,5 @@
   <xacro:property name="x_vision_box_front" value="0.146" />
   <xacro:property name="x_pos_sensor_head_rel_to_base_link" value="${x_vision_box_front-0.052}" />
-  <xacro:property name="laser1RollServo_height" value="0.118" /> <!--between base_link and laser1 roll axis-->
+  <xacro:property name="laser1RollServo_height" value="0.04" /> <!--between base_link and laser1 roll axis-->
   <xacro:property name="cameraYawServo_size_z" value="0.085" /> <!--between upper edge of top and camera pitch axis-->
   <xacro:property name="cameraYawServo_x_position" value="-0.053" /> <!--between front edge of top and camera yaw axis-->

Commit message: [hector_components_description] adapted urdf for asus xtion and added camera variables

File: hector_components_description/urdf/vision_box_common.urdf.xacro (robot description, xacro)
@@ -4,5 +4,5 @@
   <xacro:include filename="$(find hector_xacro_tools)/urdf/sensor_macros.urdf.xacro"/>
   <xacro:include filename="$(find hector_sensors_description)/urdf/thermaleye_camera.urdf.xacro"/>
-  <xacro:include filename="$(find hector_sensors_description)/urdf/kinect_camera.urdf.xacro"/>
+  <xacro:include filename="$(find hector_sensors_description)/urdf/asus_camera.urdf.xacro"/>
   <xacro:include filename="$(find hector_sensors_description)/urdf/hokuyo_utm30lx.urdf.xacro" />
   <xacro:include filename="$(find hector_components_description)/urdf/vision_box_common.gazebo.xacro" />
@@ -118,7 +118,7 @@
       <origin xyz="${infrared_x_position} ${infrared_y_position} ${infrared_z_position}" rpy="0 0 0"/>
     </xacro:thermaleye_camera_model>
-    <xacro:kinect_camera_model name="openni" parent="mounting_link">
-      <origin xyz="${kinect_x_position} 0 ${kinect_z_position}" rpy="0 0 0"/>
-    </xacro:kinect_camera_model>
+    <xacro:asus_camera_model name="openni" parent="mounting_link">
+      <origin xyz="${kinect_x_position} ${kinect_y_position}  ${kinect_z_position}" rpy="${kinect_roll_position} ${kinect_pitch_position} ${kinect_yaw_position}"/>
+    </xacro:asus_camera_model>
     <xacro:hokuyo_utm30lx name="laser1" parent="laser1_link" ros_topic="laser1/scan" update_rate="40" ray_count="1081" min_angle="135" max_angle="-135">
       <origin xyz="${laser1_center_x_offset} 0 ${laser1_plane_height}" rpy="0 0 0"/>

File: hector_components_description/urdf/vision_box_common_dimensions.urdf.xacro (robot description, xacro)
@@ -56,5 +56,8 @@
   <xacro:property name="kinect_size_z" value="0.04" />
   <xacro:property name="kinect_x_position" value="0.055" /> <!--between intersection point of yaw and pitch axis and center of camera lense-->
-  <xacro:property name="kinect_y_position" value="0" />
+  <xacro:property name="kinect_y_position" value="0.0" />
   <xacro:property name="kinect_z_position" value="0.055" />
+  <xacro:property name="kinect_roll_position" value="0" />
+  <xacro:property name="kinect_pitch_position" value="0" />
+<!--   <xacro:property name="kinect_yaw_position" value="0" />/>-->
 </robot>

File: hector_components_description/urdf/vision_box_dimensions_hector1.urdf.xacro (robot description, xacro)
@@ -16,3 +16,4 @@
   <xacro:property name="top_box_size_y" value="0.21" />
   <xacro:property name="top_box_size_z" value="0.133" />
+  <xacro:property name="kinect_yaw_position" value="0.0" />
 </robot>

File: hector_components_description/urdf/vision_box_dimensions_hector2.urdf.xacro (robot description, xacro)
@@ -16,3 +16,4 @@
   <xacro:property name="top_box_size_y" value="0.21" />
   <xacro:property name="top_box_size_z" value="0.133" />
+  <xacro:property name="kinect_yaw_position" value="0.0" />
   </robot>

Commit message: Removed camera from vision box. Added multisensor head.

File: hector_components_description/urdf/vision_box_common.urdf.xacro (robot description, xacro)
@@ -8,4 +8,5 @@
   <xacro:include filename="$(find hector_components_description)/urdf/vision_box_common.gazebo.xacro" />
   <xacro:include filename="$(find hector_components_description)/urdf/vision_box_common_dimensions.urdf.xacro" />
+  <xacro:include filename="$(find hector_components_description)/urdf/hector_multisensor_head.urdf.xacro" />
   <!--<xacro:include filename="$(find hector_components_description)/urdf/vision_box_dimensions_hector2.urdf.xacro" />-->
   <xacro:macro name="vision_box" params="box_type parent *origin">
@@ -34,4 +35,18 @@
       </collision>
     </link>
+    <hector_multisensor_head_macro parent="top_box"  name="head1" scaling="0.001">
+      <origin xyz="0.0 0.0 -0.006" rpy="${M_PI*0.5} 0.0 ${M_PI*0.5}"/>
+      <origin xyz="0.0 0.0 0.0" rpy="0.0 0.0 0.0"/>
+    </hector_multisensor_head_macro>
+    <joint name="multisensor_head1_joint" type="fixed" >
+      <parent link="top_box_link" />
+      <child link="head1_link" />
+      <origin xyz="${x_vision_box_front + 0.097} 0 0.231" rpy="0 ${-M_PI*0.5} 0" />
+    </joint>
+    <gazebo>
+      <plugin name="gazebo_ros_control" filename="libgazebo_ros_control.so">
+        <robotNamespace>sensor_head</robotNamespace>
+      </plugin>
+    </gazebo>
     <joint name="laser1/x" type="revolute">
       <origin xyz="${x_vision_box_front} 0 ${laser1RollServo_height}" rpy="0 0 0"/>
@@ -77,48 +92,8 @@
         <origin xyz="0.0 0.0 ${laser1_size_z/2}" rpy="0 0 0"/>
         <geometry>
-          <!--<box size="${laser1_size_x} ${laser1_size_y} ${laser1_size_z}" />-->
           <box size="${laser1_size_x} ${laser1_size_y} 0.01"/>
         </geometry>
       </collision>
     </link>
-    <joint name="camera/z" type="revolute">
-      <origin xyz="${x_pos_sensor_head_rel_to_base_link} 0 0.137" rpy="0 0 0"/>
-      <parent link="top_box_link"/>
-      <child link="cameraYawServo"/>
-      <axis xyz="0 0 1"/>
-      <limit lower="${-M_PI*3/4}" upper="${M_PI*3/4}" effort="100" velocity="100"/>
-    </joint>
-    <link name="cameraYawServo">
-      <xacro:inertial_sphere mass="0.1" diameter="0.07"/>
-      <visual>
-        <origin xyz="0.0 0.0 ${cameraYawServo_size_z/2}" rpy="0 0 0"/>
-        <geometry>
-          <box size="${cameraYawServo_size_x} ${cameraYawServo_size_y} ${cameraYawServo_size_z}"/>
-        </geometry>
-        <material name="Blue"/>
-      </visual>
-      <collision>
-        <origin xyz="0.0 0.0 ${cameraYawServo_size_z/2}" rpy="0 0 0"/>
-        <geometry>
-          <box size="${cameraYawServo_size_x} ${cameraYawServo_size_y} ${cameraYawServo_size_z}"/>
-        </geometry>
-      </collision>
-    </link>
-    <joint name="camera/y" type="revolute">
-      <origin xyz="0 0 ${cameraYawServo_size_z}" rpy="0 0 0"/>
-      <parent link="cameraYawServo"/>
-      <child link="mounting_link"/>
-      <axis xyz="0 1 0"/>
-      <limit lower="${-M_PI/2}" upper="${M_PI/2}" effort="100" velocity="100"/>
-    </joint>
-    <link name="mounting_link">
-      <xacro:inertial_sphere mass="0.05" diameter="0.07"/>
-    </link>
-    <xacro:thermaleye_camera_model name="infrared" parent="mounting_link">
-      <origin xyz="${infrared_x_position} ${infrared_y_position} ${infrared_z_position}" rpy="0 0 0"/>
-    </xacro:thermaleye_camera_model>
-    <xacro:asus_camera_model name="openni" parent="mounting_link">
-      <origin xyz="${kinect_x_position} ${kinect_y_position}  ${kinect_z_position}" rpy="${kinect_roll_position} ${kinect_pitch_position} ${kinect_yaw_position}"/>
-    </xacro:asus_camera_model>
     <xacro:hokuyo_utm30lx name="laser1" parent="laser1_link" ros_topic="laser1/scan" update_rate="40" ray_count="1081" min_angle="135" max_angle="-135">
       <origin xyz="${laser1_center_x_offset} 0 ${laser1_plane_height}" rpy="0 0 0"/>

Commit message: Fixed naming fix.

File: hector_components_description/urdf/vision_box_common.urdf.xacro (robot description, xacro)
@@ -39,7 +39,7 @@
       <origin xyz="0.0 0.0 0.0" rpy="0.0 0.0 0.0"/>
     </hector_multisensor_head_macro>
-    <joint name="multisensor_head1_joint" type="fixed" >
+    <joint name="multisensor_head_joint" type="fixed" >
       <parent link="top_box_link" />
-      <child link="head1_link" />
+      <child link="head_link" />
       <origin xyz="${x_vision_box_front + 0.097} 0 0.231" rpy="0 ${-M_PI*0.5} 0" />
     </joint>

Commit message: Added calibration.

File: hector_components_description/urdf/vision_box_common.urdf.xacro (robot description, xacro)
@@ -37,5 +37,5 @@
     <hector_multisensor_head_macro parent="top_box"  name="head" scaling="0.001">
       <origin xyz="0.0 0.0 -0.006" rpy="${M_PI*0.5} 0.0 ${M_PI*0.5}"/>
-      <origin xyz="0.0 0.0 0.0" rpy="0.0 0.0 0.0"/>
+      <origin xyz="0 0.000323461 0.0127965" rpy="0 0.021197 -0.00357142"/>
     </hector_multisensor_head_macro>
     <joint name="multisensor_head_joint" type="fixed" >

Commit message: add thermal_camera to demo, however, the thermal image is alway block

File: hector_components_description/urdf/vision_box_common.urdf.xacro (robot description, xacro)
@@ -8,5 +8,5 @@
   <xacro:include filename="$(find hector_components_description)/urdf/vision_box_common.gazebo.xacro" />
   <xacro:include filename="$(find hector_components_description)/urdf/vision_box_common_dimensions.urdf.xacro" />
-  <!--<xacro:include filename="$(find hector_components_description)/urdf/vision_box_dimensions_hector2.urdf.xacro" />-->
+  <xacro:include filename="$(find hector_components_description)/urdf/vision_box_dimensions_hector2.urdf.xacro" />
   <xacro:macro name="vision_box" params="box_type parent *origin">
     <joint name="top_box_joint" type="fixed">

File: hector_sensors_description/urdf/thermaleye_camera.urdf.xacro (robot description, xacro)
@@ -1,12 +1,12 @@
 <?xml version="1.0"?>
 <robot xmlns:xacro="http://www.ros.org/wiki/xacro">
-    <xacro:include filename="$(find hector_xacro_tools)/urdf/sensor_macros.urdf.xacro" />
-    <xacro:macro name="thermaleye_camera_model" params="name parent *origin">
+  <xacro:property name="M_PI" value="3.1415926535897931" />
+    <xacro:macro name="thermaleye_camera" params="name parent *origin ros_topic cam_info_topic update_rate res_x res_y image_format hfov">
       <joint name="${name}_joint" type="fixed">
         <xacro:insert_block name="origin" />
         <parent link="${parent}"/>
-        <child link="${name}_frame"/>
+        <child link="${name}_link"/>
       </joint>
-      <link name="${name}_frame">
+      <link name="${name}_link">
         <xacro:inertial_sphere mass="0.01" diameter="0.07" />
         <visual>
@@ -23,5 +23,33 @@
         </collision>
       </link>
-      <xacro:add_optical_frame name="${name}" />
+      <joint name="${name}_optical_joint" type="fixed">
+        <origin xyz="0 0 0" rpy="${-M_PI/2} 0.0 ${-M_PI/2}" />
+        <parent link="${name}_link" />
+        <child link="${name}_optical_frame"/>
+      </joint>
+      <link name="${name}_optical_frame"/>
+      <gazebo reference="${name}_link">
+        <sensor type="camera" name="${name}_thermal_camera">
+          <update_rate>${update_rate}</update_rate>
+          <camera>
+            <horizontal_fov>${hfov * M_PI/180.0}</horizontal_fov>
+            <image>
+              <format>${image_format}</format>
+              <width>${res_x}</width>
+              <height>${res_y}</height>
+            </image>
+            <clip>
+              <near>0.01</near>
+              <far>100</far>
+            </clip>
+          </camera>
+          <plugin name="${name}_camera_controller" filename="libgazebo_ros_thermal_camera.so">
+            <cameraName>${name}</cameraName>
+            <imageTopicName>${ros_topic}</imageTopicName>
+            <cameraInfoTopicName>${cam_info_topic}</cameraInfoTopicName>
+            <frameName>${name}_optical_frame</frameName>
+          </plugin>
+        </sensor>
+      </gazebo>
     </xacro:macro>
   </robot>
