Commit message: Removing collision for all sensor parts to allow for multiple sensor configurations at once. Addind multisensor heads in different configurations.

File: hector_components_description/urdf/hector_multisensor_head.urdf.xacro (robot description, xacro)
@@ -9,19 +9,19 @@
         <link name="${name}_link">
              <inertial>
-	      <mass value="0.8"/>
+	      <mass value="0.00001"/>
 	      <inertia ixx="0.0025" ixy="0.0" ixz="0.0001" iyy="0.0013" iyz="0.0" izz="0.0026"/>
 	    </inertial>
-            <collision name="collision">
+<!--            <collision name="collision">
                  <xacro:insert_block name="origin"/>
                 <geometry>
                     <mesh filename="package://hector_components_description/meshes/hector_multisensor_head/multisensor_head_collision.stl" scale="${scaling} ${scaling} ${scaling}"/>
                 </geometry>
-            </collision>
-            <visual>
+            </collision>-->
+<!--            <visual>
                 <xacro:insert_block name="origin"/>
                 <geometry>
                     <mesh filename="package://hector_components_description/meshes/hector_multisensor_head/multisensor_head.stl" scale="${scaling} ${scaling} ${scaling}"/>
                 </geometry>
-            </visual>
+            </visual>-->
         </link>
         <joint name="${name}_lidar_spinning_joint" type="continuous">
@@ -34,9 +34,9 @@
         </joint>
         <link name="${name}_lidar_mount_link">
-            <xacro:inertial_sphere_with_pose_macro mass="0.1" diameter="0.03">
+            <xacro:inertial_sphere_with_pose_macro mass="0.00001" diameter="0.03">
                 <origin xyz="0.0 0.0 0.0" rpy="0 0 0"/>
             </xacro:inertial_sphere_with_pose_macro>
         </link>
-        <xacro:hokuyo_utm30lx name="${name}_link_hokuyo_laser" parent="${name}_lidar_mount_link" ros_topic="/head_lidar/scan" update_rate="40" ray_count="1040" min_angle="130" max_angle="-130">
+        <xacro:hokuyo_utm30lx name="${name}_link_hokuyo_laser" parent="${name}_lidar_mount_link" ros_topic="/${name}_lidar/scan" update_rate="40" ray_count="1040" min_angle="130" max_angle="-130">
             <xacro:insert_block name="calibration" />
         </xacro:hokuyo_utm30lx>
@@ -54,7 +54,7 @@
             <implicitSpringDamper>1</implicitSpringDamper>
         </gazebo>
-	<xacro:asus_camera name="${name}_cam" parent="${name}_link">
+<!--	<xacro:asus_camera name="${name}_cam" parent="${name}_link">
 	                <origin xyz="0.065 0.0 0.23" rpy="0 0 0"/>
-	</xacro:asus_camera>
+	</xacro:asus_camera>  -->
         <!-- <gazebo reference="${name}_spinning_lidar_root_link"><material>Gazebo/Grey</material></gazebo><gazebo reference="${name}_spinning_lidar_spin_link"><material>Gazebo/Grey</material></gazebo> -->
     </xacro:macro>

File: hector_components_description/urdf/vision_box_common.urdf.xacro (robot description, xacro)
@@ -35,12 +35,39 @@
       </collision>
     </link>
-    <hector_multisensor_head_macro parent="top_box"  name="head" scaling="0.001">
+    <hector_multisensor_head_macro parent="top_box"  name="head1" scaling="0.001">
       <origin xyz="0.0 0.0 -0.006" rpy="${M_PI*0.5} 0.0 ${M_PI*0.5}"/>
       <origin xyz="0 0.000323461 0.0127965" rpy="0 0.021197 -0.00357142"/>
     </hector_multisensor_head_macro>
-    <joint name="multisensor_head_joint" type="fixed" >
+    <joint name="multisensor_head1_joint" type="fixed" >
       <parent link="top_box_link" />
-      <child link="head_link" />
-      <origin xyz="${x_vision_box_front + 0.097} 0 0.231" rpy="0 ${-M_PI*0.5} 0" />
+      <child link="head1_link" />
+      <origin xyz="${x_vision_box_front + 0.097} 0 ${top_box_size_z/2 + 0.1645}" rpy="0 ${-M_PI*0.5} 0" />
+    </joint>
+    <hector_multisensor_head_macro parent="top_box"  name="head2" scaling="0.001">
+      <origin xyz="0.0 0.0 -0.006" rpy="${M_PI*0.5} 0.0 ${M_PI*0.5}"/>
+      <origin xyz="0.0 0.0 0.01" rpy="0.0 ${M_PI*0.12} 0.0"/>
+    </hector_multisensor_head_macro>
+    <joint name="multisensor_head2_joint" type="fixed" >
+      <parent link="top_box_link" />
+      <child link="head2_link" />
+      <origin xyz="${x_vision_box_front + 0.097} 0 ${top_box_size_z/2 + 0.1645}" rpy="0 ${-M_PI*0.5} 0" />
+    </joint>
+    <hector_multisensor_head_macro parent="top_box"  name="head3" scaling="0.001">
+      <origin xyz="0.0 0.0 -0.006" rpy="${M_PI*0.5} 0.0 ${M_PI*0.5}"/>
+      <origin xyz="0.0 0.0 0.02" rpy="0.0 ${M_PI*0.25} 0.0"/>
+    </hector_multisensor_head_macro>
+    <joint name="multisensor_head3_joint" type="fixed" >
+      <parent link="top_box_link" />
+      <child link="head3_link" />
+      <origin xyz="${x_vision_box_front + 0.097} 0 ${top_box_size_z/2 + 0.1645}" rpy="0 ${-M_PI*0.5} 0" />
+    </joint>
+    <hector_multisensor_head_macro parent="top_box"  name="head4" scaling="0.001">
+      <origin xyz="0.0 0.0 -0.006" rpy="${M_PI*0.5} 0.0 ${M_PI*0.5}"/>
+      <origin xyz="0 0.000323461 0.0127965" rpy="0 0.021197 -0.00357142"/>
+    </hector_multisensor_head_macro>
+    <joint name="multisensor_head4_joint" type="fixed" >
+      <parent link="top_box_link" />
+      <child link="head4_link" />
+      <origin xyz="${x_vision_box_front + 0.03} 0 ${0.02 - top_box_size_z/2}" rpy="0 0 0" />
     </joint>
     <gazebo>
@@ -65,10 +92,10 @@
         <material name="Blue"/>
       </visual>
-      <collision>
+<!--      <collision>
         <origin xyz="${laser1RollServo_size_x/2} 0.0 0.0" rpy="0 0 0"/>
         <geometry>
           <box size="${laser1RollServo_size_x} ${laser1RollServo_size_y} ${laser1RollServo_size_z}"/>
         </geometry>
-      </collision>
+      </collision>-->
     </link>
     <joint name="laser1/y" type="revolute">
@@ -89,11 +116,50 @@
         <material name="Grey"/>
       </visual>
-      <collision>
+<!--      <collision>
         <origin xyz="0.0 0.0 ${laser1_size_z/2}" rpy="0 0 0"/>
         <geometry>
           <box size="${laser1_size_x} ${laser1_size_y} 0.01"/>
         </geometry>
-      </collision>
+      </collision>-->
     </link>
+    <joint name="camera/z" type="revolute">
+      <origin xyz="${x_pos_sensor_head_rel_to_base_link} 0 0.137" rpy="0 0 0"/>
+      <parent link="top_box_link"/>
+      <child link="cameraYawServo"/>
+      <axis xyz="0 0 1"/>
+      <limit lower="${-M_PI*3/4}" upper="${M_PI*3/4}" effort="100" velocity="100"/>
+    </joint>
+    <link name="cameraYawServo">
+      <xacro:inertial_sphere mass="0.1" diameter="0.07"/>
+      <visual>
+        <origin xyz="0.0 0.0 ${cameraYawServo_size_z/2}" rpy="0 0 0"/>
+        <geometry>
+          <box size="${cameraYawServo_size_x} ${cameraYawServo_size_y} ${cameraYawServo_size_z}"/>
+        </geometry>
+        <material name="Blue"/>
+      </visual>
+<!--      <collision>
+        <origin xyz="0.0 0.0 ${cameraYawServo_size_z/2}" rpy="0 0 0"/>
+        <geometry>
+          <box size="${cameraYawServo_size_x} ${cameraYawServo_size_y} ${cameraYawServo_size_z}"/>
+        </geometry>
+      </collision>-->
+    </link>
+    <joint name="camera/y" type="revolute">
+      <origin xyz="0 0 ${cameraYawServo_size_z}" rpy="0 0 0"/>
+      <parent link="cameraYawServo"/>
+      <child link="mounting_link"/>
+      <axis xyz="0 1 0"/>
+      <limit lower="${-M_PI/2}" upper="${M_PI/2}" effort="100" velocity="100"/>
+    </joint>
+    <link name="mounting_link">
+      <xacro:inertial_sphere mass="0.05" diameter="0.07"/>
+    </link>
+    <xacro:thermaleye_camera_model name="infrared" parent="mounting_link">
+      <origin xyz="${infrared_x_position} ${infrared_y_position} ${infrared_z_position}" rpy="0 0 0"/>
+    </xacro:thermaleye_camera_model>
+    <xacro:asus_camera_model name="openni" parent="mounting_link">
+      <origin xyz="${kinect_x_position} ${kinect_y_position}  ${kinect_z_position}" rpy="${kinect_roll_position} ${kinect_pitch_position} ${kinect_yaw_position}"/>
+    </xacro:asus_camera_model>
     <xacro:hokuyo_utm30lx name="laser1" parent="laser1_link" ros_topic="laser1/scan" update_rate="40" ray_count="1081" min_angle="135" max_angle="-135">
       <origin xyz="${laser1_center_x_offset} 0 ${laser1_plane_height}" rpy="0 0 0"/>

File: hector_sensors_description/urdf/asus_camera.urdf.xacro (robot description, xacro)
@@ -32,10 +32,10 @@
         </collision>
         -->
-        <collision>
+<!--        <collision>
           <origin xyz="0 0 0" rpy="0 0 0" />
           <geometry>
             <mesh filename="package://hector_sensors_description/meshes/asus_camera/asus_camera_simple.dae"/>
           </geometry>
-        </collision>
+        </collision>-->
       </link>
       <joint name="${name}_depth_joint" type="fixed">

File: hector_sensors_description/urdf/hokuyo_utm30lx.urdf.xacro (robot description, xacro)
@@ -20,11 +20,11 @@
         </geometry>
         </visual>
-        <collision>
+<!--        <collision>
           <origin xyz="0 0 -0.0115" rpy="0 0 0" />
           <geometry>
-          <box size="0.058 0.058 0.087" />
+          <box size="0.058 0.058 0.087" />-->
           <!--<mesh filename="package://hector_sensors_description/meshes/hokuyo_utm30lx/hokuyo_utm_30lx.stl"/>-->
-        </geometry>
-        </collision>
+<!--        </geometry>
+        </collision>-->
       </link>
     </xacro:macro>

File: hector_sensors_description/urdf/thermaleye_camera.urdf.xacro (robot description, xacro)
@@ -16,10 +16,10 @@
           </geometry>
         </visual>
-        <collision>
+<!--        <collision>
           <origin xyz="0 0 0" rpy="0 0 0" />
           <geometry>
             <mesh filename="package://hector_sensors_description/meshes/thermaleye_camera/thermaleye_camera_hector_v2.stl"/>
           </geometry>
-        </collision>
+        </collision>-->
       </link>
       <xacro:add_optical_frame name="${name}" />

Commit message: update multisensor head files for usage with thor mang v3

File: hector_components_description/urdf/hector_multisensor_head.urdf.xacro (robot description, xacro)
@@ -25,5 +25,6 @@
       </link>
       <joint name="${name}_lidar_spinning_joint" type="continuous">
-         <origin xyz="0.061 0.0 0.134" rpy="0 0 0" />
+<!--         <origin xyz="0.061 0.0 0.134" rpy="0 0 0" />-->
+	 <origin xyz="0.061 0.0 0.083" rpy="0 0 0" />
          <parent link="${name}_link" />
          <child link="${name}_lidar_mount_link" />
@@ -37,5 +38,5 @@
          </xacro:inertial_sphere_with_pose_macro>
       </link>
-      <xacro:hokuyo_utm30lx name="${name}_link_hokuyo_laser" parent="${name}_lidar_mount_link" ros_topic="/head_lidar/scan" update_rate="40" ray_count="1040" min_angle="130" max_angle="-130">
+      <xacro:hokuyo_utm30lx name="${name}_link_hokuyo_laser" parent="${name}_lidar_mount_link" ros_topic="head_lidar/scan" update_rate="40" ray_count="1040" min_angle="130" max_angle="-130">
          <xacro:insert_block name="calibration" />
       </xacro:hokuyo_utm30lx>
@@ -54,5 +55,5 @@
       </gazebo>
       <xacro:asus_camera name="${name}_cam" parent="${name}_link">
-         <origin xyz="0.065 0.0 0.23" rpy="0 0 0" />
+         <origin xyz="0.065 0.0 0.179" rpy="0 0 0" />
       </xacro:asus_camera>
       <!-- <gazebo reference="${name}_spinning_lidar_root_link"><material>Gazebo/Grey</material></gazebo><gazebo reference="${name}_spinning_lidar_spin_link"><material>Gazebo/Grey</material></gazebo> -->

Commit message: center realsense camera

File: hector_components_description/urdf/hector_multisensor_head.urdf.xacro (robot description, xacro)
@@ -55,5 +55,5 @@
       </gazebo>
       <xacro:realsense_camera name="${name}_cam" parent="${name}_link">
-         <origin xyz="0.065 0.0 0.179" rpy="0 0 0" />
+         <origin xyz="0.035 -0.05 0.181" rpy="0 0 0" />
       </xacro:realsense_camera>
       <!-- <gazebo reference="${name}_spinning_lidar_root_link"><material>Gazebo/Grey</material></gazebo><gazebo reference="${name}_spinning_lidar_spin_link"><material>Gazebo/Grey</material></gazebo> -->

Commit message: add color to visual model

File: hector_components_description/urdf/hector_multisensor_head.urdf.xacro (robot description, xacro)
@@ -22,4 +22,5 @@
                <mesh filename="package://hector_components_description/meshes/hector_multisensor_head/multisensor_head.stl" scale="${scaling} ${scaling} ${scaling}" />
             </geometry>
+	    <material name="grey"/>
          </visual>
       </link>

Commit message: add angle of camera

File: hector_components_description/urdf/hector_multisensor_head.urdf.xacro (robot description, xacro)
@@ -55,5 +55,5 @@
       </gazebo>
       <xacro:realsense_camera name="${name}_cam" parent="${name}_link">
-         <origin xyz="0.035 -0.05 0.181" rpy="0 0 0" />
+         <origin xyz="0.015 -0.05 0.181" rpy="0 0.261799 0" />
       </xacro:realsense_camera>
       <!-- <gazebo reference="${name}_spinning_lidar_root_link"><material>Gazebo/Grey</material></gazebo><gazebo reference="${name}_spinning_lidar_spin_link"><material>Gazebo/Grey</material></gazebo> -->

Commit message: changes to make evaluation easier

File: hector_components_description/urdf/hector_multisensor_head.urdf.xacro (robot description, xacro)
@@ -56,5 +56,8 @@
       </gazebo>
       <xacro:realsense_camera name="${name}_cam" parent="${name}_link">
-         <origin xyz="0.015 -0.05 0.181" rpy="0 0.261799 0" />
+<!--         <origin xyz="0.015 -0.05 0.181" rpy="0 0.261799 0" />-->
+        <origin xyz="0.015 -0.05 0.181" rpy="0 0 0" />
+<!--         <origin xyz="${0.015 + 0.00809157} ${-0.05 + 0.0277386} ${0.181 + 0.0236774}" rpy="0.0503855 0.0507573 0.0492087" /> -->
+<!--         <origin xyz="${0.015 + -0.00189352} ${-0.05 + 0.0178069} ${0.181 + 0.0135799}" rpy="0.0503855 0.0507573 0.0492087" />  -->
       </xacro:realsense_camera>
       <!-- <gazebo reference="${name}_spinning_lidar_root_link"><material>Gazebo/Grey</material></gazebo><gazebo reference="${name}_spinning_lidar_spin_link"><material>Gazebo/Grey</material></gazebo> -->

File: hector_sensors_description/urdf/hokuyo_utm30lx.urdf.xacro (robot description, xacro)
@@ -49,5 +49,5 @@
             </scan>
             <range>
-              <min>0.08</min>
+              <min>0.2</min>
               <max>30.0</max>
               <resolution>0.01</resolution>
@@ -90,5 +90,5 @@
             </scan>
             <range>
-              <min>0.08</min>
+              <min>0.05</min>
               <max>30.0</max>
               <resolution>0.01</resolution>

File: hector_sensors_description/urdf/realsense_camera.urdf.xacro (robot description, xacro)
@@ -106,4 +106,5 @@
           <camera>
             <horizontal_fov>${62.8 * M_PI/180.0}</horizontal_fov>
+            <vertical_fov>${62.8 * M_PI/180.0}</vertical_fov>
             <image>
               <format>R8G8B8</format>
@@ -112,5 +113,5 @@
             </image>
             <clip>
-              <near>0.5</near>
+              <near>0.05</near>
               <far>9</far>
             </clip>

Commit message: updated multisensor head

File: hector_components_description/urdf/hector_multisensor_head.urdf.xacro (robot description, xacro)
@@ -1,61 +1,62 @@
-<?xml version="1.0"?>
-<robot
-    xmlns:xacro="http://www.ros.org/wiki/xacro" name="hector_multisensor_head">
-    <xacro:include filename="$(find hector_xacro_tools)/urdf/inertia_tensors.urdf.xacro"/>
-    <xacro:include filename="$(find hector_sensors_description)/urdf/hokuyo_utm30lx.urdf.xacro" />
-    <xacro:include filename="$(find hector_sensors_description)/urdf/asus_camera.urdf.xacro" />
-    <xacro:property name="M_PI" value="3.14159265359"/>
-    <xacro:macro name="hector_multisensor_head_macro" params="parent name scaling *origin *calibration">
-        <link name="${name}_link">
-             <inertial>
-	      <mass value="0.8"/>
-	      <inertia ixx="0.0025" ixy="0.0" ixz="0.0001" iyy="0.0013" iyz="0.0" izz="0.0026"/>
-	    </inertial>
-            <collision name="collision">
-                 <xacro:insert_block name="origin"/>
-                <geometry>
-                    <mesh filename="package://hector_components_description/meshes/hector_multisensor_head/multisensor_head_collision.stl" scale="${scaling} ${scaling} ${scaling}"/>
-                </geometry>
-            </collision>
-            <visual>
-                <xacro:insert_block name="origin"/>
-                <geometry>
-                    <mesh filename="package://hector_components_description/meshes/hector_multisensor_head/multisensor_head.stl" scale="${scaling} ${scaling} ${scaling}"/>
-                </geometry>
-            </visual>
-        </link>
-        <joint name="${name}_lidar_spinning_joint" type="continuous">
-            <origin xyz="0.061 0.0 0.134" rpy="0 0 0"/>
-            <parent link="${name}_link" />
-            <child link="${name}_lidar_mount_link"/>
-            <axis xyz="1 0 0" rpy="0 0 0"/>
-            <limit effort="1000" velocity="100"/>
-            <joint_properties damping="500.0" friction="200.0"/>
-        </joint>
-        <link name="${name}_lidar_mount_link">
-            <xacro:inertial_sphere_with_pose_macro mass="0.1" diameter="0.03">
-                <origin xyz="0.0 0.0 0.0" rpy="0 0 0"/>
-            </xacro:inertial_sphere_with_pose_macro>
-        </link>
-        <xacro:hokuyo_utm30lx name="${name}_link_hokuyo_laser" parent="${name}_lidar_mount_link" ros_topic="/head_lidar/scan" update_rate="40" ray_count="1040" min_angle="130" max_angle="-130">
-            <xacro:insert_block name="calibration" />
-        </xacro:hokuyo_utm30lx>
-        <transmission name="${name}_lidar_spinning_joint_transmission">
-            <type>transmission_interface/SimpleTransmission</type>
-            <joint name="${name}_lidar_spinning_joint">
-                <hardwareInterface>EffortJointInterface</hardwareInterface>
-            </joint>
-            <actuator name="${name}_lidar_spinning_joint_motor">
-                <hardwareInterface>EffortJointInterface</hardwareInterface>
-                <mechanicalReduction>1</mechanicalReduction>
-            </actuator>
-        </transmission>
-        <gazebo reference="${name}_lidar_spinning_joint">
-            <implicitSpringDamper>1</implicitSpringDamper>
-        </gazebo>
-	<xacro:asus_camera name="${name}_cam" parent="${name}_link">
-	                <origin xyz="0.065 0.0 0.23" rpy="0 0 0"/>
-	</xacro:asus_camera>
-        <!-- <gazebo reference="${name}_spinning_lidar_root_link"><material>Gazebo/Grey</material></gazebo><gazebo reference="${name}_spinning_lidar_spin_link"><material>Gazebo/Grey</material></gazebo> -->
-    </xacro:macro>
+<?xml version="1.0" encoding="UTF-8"?>
+<robot xmlns:xacro="http://ros.org/wiki/xacro" name="hector_multisensor_head">
+   <xacro:include filename="$(find hector_xacro_tools)/urdf/inertia_tensors.urdf.xacro" />
+   <xacro:include filename="$(find hector_sensors_description)/urdf/hokuyo_utm30lx.urdf.xacro" />
+   <xacro:include filename="$(find hector_sensors_description)/urdf/realsense_camera.urdf.xacro" />
+   <xacro:property name="M_PI" value="3.14159265359" />
+   <xacro:macro name="hector_multisensor_head_macro" params="parent name scaling *origin *calibration">
+      <link name="${name}_link">
+         <inertial>
+            <mass value="0.8" />
+            <inertia ixx="0.0025" ixy="0.0" ixz="0.0001" iyy="0.0013" iyz="0.0" izz="0.0026" />
+         </inertial>
+         <collision name="collision">
+            <xacro:insert_block name="origin" />
+            <geometry>
+               <mesh filename="package://hector_components_description/meshes/hector_multisensor_head/multisensor_head_collision.stl" scale="${scaling} ${scaling} ${scaling}" />
+            </geometry>
+         </collision>
+         <visual>
+            <xacro:insert_block name="origin" />
+            <geometry>
+               <mesh filename="package://hector_components_description/meshes/hector_multisensor_head/multisensor_head.stl" scale="${scaling} ${scaling} ${scaling}" />
+            </geometry>
+            <material name="grey"/>
+         </visual>
+      </link>
+      <joint name="${name}_lidar_spinning_joint" type="continuous">
+<!--         <origin xyz="0.061 0.0 0.134" rpy="0 0 0" />-->
+         <origin xyz="0.061 0.0 0.083" rpy="0 0 0" />
+         <parent link="${name}_link" />
+         <child link="${name}_lidar_mount_link" />
+         <axis xyz="1 0 0" rpy="0 0 0" />
+         <limit effort="1000" velocity="100" />
+         <joint_properties damping="500.0" friction="200.0" />
+      </joint>
+      <link name="${name}_lidar_mount_link">
+         <xacro:inertial_sphere_with_pose_macro mass="0.1" diameter="0.03">
+            <origin xyz="0.0 0.0 0.0" rpy="0 0 0" />
+         </xacro:inertial_sphere_with_pose_macro>
+      </link>
+      <xacro:hokuyo_utm30lx name="${name}_link_hokuyo_laser" parent="${name}_lidar_mount_link" ros_topic="head_lidar/scan" update_rate="40" ray_count="1040" min_angle="130" max_angle="-130">
+         <xacro:insert_block name="calibration" />
+      </xacro:hokuyo_utm30lx>
+      <transmission name="${name}_lidar_spinning_joint_transmission">
+         <type>transmission_interface/SimpleTransmission</type>
+         <joint name="${name}_lidar_spinning_joint">
+            <hardwareInterface>EffortJointInterface</hardwareInterface>
+         </joint>
+         <actuator name="${name}_lidar_spinning_joint_motor">
+            <hardwareInterface>EffortJointInterface</hardwareInterface>
+            <mechanicalReduction>1</mechanicalReduction>
+         </actuator>
+      </transmission>
+      <gazebo reference="${name}_lidar_spinning_joint">
+         <implicitSpringDamper>1</implicitSpringDamper>
+      </gazebo>
+      <xacro:realsense_camera_no_geom name="${name}_cam" parent="${name}_link">
+         <origin xyz="0.015 -0.05 0.181" rpy="0 0.261799 0" />
+      </xacro:realsense_camera_no_geom>
+      <!-- <gazebo reference="${name}_spinning_lidar_root_link"><material>Gazebo/Grey</material></gazebo><gazebo reference="${name}_spinning_lidar_spin_link"><material>Gazebo/Grey</material></gazebo> -->
+   </xacro:macro>
 </robot>
