Commit message: Update to transmissions, prepending "hardware_interface/"

File: hector_components_description/urdf/hector_multisensor_head.urdf.xacro (robot description, xacro)
@@ -3,4 +3,5 @@
     xmlns:xacro="http://www.ros.org/wiki/xacro" name="hector_multisensor_head">
     <xacro:include filename="$(find hector_xacro_tools)/urdf/inertia_tensors.urdf.xacro"/>
+    <xacro:include filename="$(find hector_xacro_tools)/urdf/joint_macros.urdf.xacro"/>
     <xacro:include filename="$(find hector_sensors_description)/urdf/hokuyo_utm30lx.urdf.xacro" />
     <xacro:include filename="$(find hector_sensors_description)/urdf/asus_camera.urdf.xacro" />
@@ -41,14 +42,5 @@
             <xacro:insert_block name="calibration" />
         </xacro:hokuyo_utm30lx>
-        <transmission name="${name}_lidar_spinning_joint_transmission">
-            <type>transmission_interface/SimpleTransmission</type>
-            <joint name="${name}_lidar_spinning_joint">
-                <hardwareInterface>EffortJointInterface</hardwareInterface>
-            </joint>
-            <actuator name="${name}_lidar_spinning_joint_motor">
-                <hardwareInterface>EffortJointInterface</hardwareInterface>
-                <mechanicalReduction>1</mechanicalReduction>
-            </actuator>
-        </transmission>
+        <xacro:joint_standard_transmission name="${name}_lidar_spinning_joint"/>
         <gazebo reference="${name}_lidar_spinning_joint">
             <implicitSpringDamper>1</implicitSpringDamper>

File: hector_xacro_tools/urdf/joint_macros.urdf.xacro (robot description, xacro)
@@ -5,8 +5,8 @@
       <type>transmission_interface/SimpleTransmission</type>
       <joint name="${name}">
-        <hardwareInterface>EffortJointInterface</hardwareInterface>
+        <hardwareInterface>hardware_interface/EffortJointInterface</hardwareInterface>
       </joint>
       <actuator name="${name}_joint_motor">
-        <hardwareInterface>EffortJointInterface</hardwareInterface>
+        <hardwareInterface>hardware_interface/EffortJointInterface</hardwareInterface>
         <mechanicalReduction>1</mechanicalReduction>
       </actuator>
