Commit message: Update headlight to remove visuals via plugins available in subt

File: hector_components_description/urdf/headlight.urdf.xacro (robot description, xacro)
@@ -47,5 +47,5 @@
             <direction>0 0 -1</direction>
           </light>
-<!--          <visual name="light_source_visual">
+          <visual name="light_source_visual">
             <geometry>
               <box>
@@ -59,5 +59,11 @@
               <emissive>0 0 0 1</emissive>
             </material>
-          </visual>-->
+            <plugin name='light_source_visualize' filename='libLightVisualPlugin.so'>
+              <light>
+                <id>light_source</id>
+                <visualize>false</visualize>
+              </light>
+            </plugin>
+          </visual>
 <!--          <inertial>
             <origin xyz="0 0 0" rpy="0 0 0"/>
@@ -70,5 +76,5 @@
           </inertial>-->
         </link>
-<!--        <plugin name='light_control' filename='libRosFlashLightPlugin.so'>
+        <plugin name='light_control' filename='libRosFlashLightPlugin.so'>
           <service_name>enable</service_name>
           <light>
@@ -79,5 +85,5 @@
             <color>1 1 1</color>
           </light>
-        </plugin>-->
+        </plugin>
       </model>
     </gazebo>

Commit message: Fix wrong box geom tag

File: hector_components_description/urdf/headlight.urdf.xacro (robot description, xacro)
@@ -2,26 +2,4 @@
 <robot xmlns:xacro="http://ros.org/wiki/xacro" name="headlight">
   <xacro:macro name="headlight" params="parent headlight_prefix xyz rpy">
-<!--    <link name="${headlight_prefix}_headlight_link">
-    <visual>
-        <origin xyz="0 0 0" rpy="0 0 0" />
-        <geometry>
-          <box size="0.01 0.01 0.01"/>
-        </geometry>
-      </visual>
-      <inertial>
-        <origin xyz="0 0 0" rpy="0 0 0"/>
-        <mass value="0.000001" />
-        <inertia
-          ixx="0.001"
-          ixy="0.0" iyy="0.001"
-          ixz="0.0" iyz="0.0" izz="0.001"
-        />
-      </inertial>
-    </link>
-    <joint name="${headlight_prefix}_headlight" type="fixed">
-      <parent link="base_link"/>
-      <child link="${headlight_prefix}_headlight_link"/>
-      <origin xyz="${xyz}" rpy="${rpy}"/>
-    </joint>-->
     <gazebo>
       <model name="${headlight_prefix}_headlight">
@@ -33,14 +11,14 @@
             <pose>0.0 0 0.0 0 -1.573 0</pose>
             <attenuation>
-              <range>50</range>
+              <range>25</range>
               <linear>0.0</linear>
               <constant>0.1</constant>
-              <quadratic>0.0</quadratic>
+              <quadratic>0.01</quadratic>
             </attenuation>
-            <diffuse>0.8 0.8 0.8 1</diffuse>
-            <specular>0.8 0.8 0.8 1</specular>
+            <diffuse>0.4 0.4 0.4 1</diffuse>
+            <specular>0.01 0.01 0.01 1</specular>
             <spot>
-              <inner_angle>1</inner_angle>
-              <outer_angle>1.1</outer_angle>
+              <inner_angle>0.8</inner_angle>
+              <outer_angle>1.9</outer_angle>
               <falloff>1</falloff>
             </spot>
@@ -49,6 +27,5 @@
           <visual name="light_source_visual">
             <geometry>
-              <box>
-              </box>
+              <box size="0.001 0.001 0.001"/>
             </geometry>
             <transparency>1</transparency>
@@ -66,13 +43,4 @@
             </plugin>
           </visual>
-<!--          <inertial>
-            <origin xyz="0 0 0" rpy="0 0 0"/>
-            <mass>0.000001</mass>
-            <inertia>
-              <ixx>0.001</ixx>
-              <ixy>0.0</ixy><iyy>0.001</iyy>
-              <ixz>0.0</ixz><iyz>0.0</iyz><izz>0.001</izz>
-            </inertia>
-          </inertial>-->
         </link>
         <plugin name='light_control' filename='libRosFlashLightPlugin.so'>

Commit message: Fix headlight geom properly. Uses SDF, not URDF syntax

File: hector_components_description/urdf/headlight.urdf.xacro (robot description, xacro)
@@ -27,5 +27,8 @@
           <visual name="light_source_visual">
             <geometry>
-              <box size="0.001 0.001 0.001"/>
+              <!--<box size="10.001 0.001 0.001"/>-->
+              <sphere>
+                <radius>0.01</radius>
+              </sphere>
             </geometry>
             <transparency>1</transparency>

Commit message: Reduce mass of headlight elements

File: hector_components_description/urdf/headlight.urdf.xacro (robot description, xacro)
@@ -25,4 +25,7 @@
             <direction>0 0 -1</direction>
           </light>
+          <inertial>
+            <mass>0.00001</mass>
+          </inertial>
           <visual name="light_source_visual">
             <geometry>

Commit message: Tune mass properties of light links

File: hector_components_description/urdf/headlight.urdf.xacro (robot description, xacro)
@@ -27,4 +27,9 @@
           <inertial>
             <mass>0.00001</mass>
+            <inertia>
+              <ixx>0.00000001</ixx>
+              <iyy>0.00000001</iyy>
+              <izz>0.00000001</izz>
+            </inertia>
           </inertial>
           <visual name="light_source_visual">
