Commit message: used textured table

File: hector_components_description/urdf/autonomy_box_on_table.urdf.xacro (robot description, xacro)
@@ -5,7 +5,7 @@
   <link name="base_link">
     <visual>
-      <origin xyz="0.0 0.0 0.0" rpy="${pi} 0 0"/>
+      <origin xyz="0.0 0.4 0.0" rpy="${0.5*pi} 0 0"/>
       <geometry>
-        <mesh filename="package://hector_components_description/meshes/table/table.stl" scale="0.001 0.001 0.001"/>
+        <mesh filename="package://hector_components_description/meshes/table/table.dae"/>
       </geometry>
     </visual>

Commit message: updated position on tbale & collision size

File: hector_components_description/urdf/autonomy_box_on_table.urdf.xacro (robot description, xacro)
@@ -1,4 +1,4 @@
 <?xml version="1.0"?>
-<robot xmlns:xacro="http://www.ros.org/wiki/xacro" name="autonomy_box_standalone">
+<robot xmlns:xacro="http://www.ros.org/wiki/xacro" name="autonomy_box_on_table">
   <xacro:include filename="$(find hector_components_description)/urdf/autonomy_box.urdf.xacro"/>
   <xacro:include filename="$(find hector_tracked_vehicles_description)/calibrations/spin_lidar_calibration.urdf.xacro"/>
@@ -29,6 +29,6 @@
     </collision>
   </link>
-  <xacro:autonomy_box_macro parent="base_link" alu_profile_collision_size_factor="1.0" name="autonomy_box" add_chilitags="false">
-    <origin xyz="0.255 0.0 0.005" rpy="0 0 0"/>
+  <xacro:autonomy_box_macro parent="base_link" alu_profile_collision_size_factor="1.25" name="autonomy_box" add_chilitags="false">
+    <origin xyz="0.205 0.0 0.005" rpy="0 0 0"/>
   </xacro:autonomy_box_macro>
 </robot>

Commit message: introduced table_link

File: hector_components_description/urdf/autonomy_box_on_table.urdf.xacro (robot description, xacro)
@@ -3,5 +3,11 @@
   <xacro:include filename="$(find hector_components_description)/urdf/autonomy_box.urdf.xacro"/>
   <xacro:include filename="$(find hector_tracked_vehicles_description)/calibrations/spin_lidar_calibration.urdf.xacro"/>
-  <link name="base_link">
+  <link name="base_link" />
+  <joint name="base_joint" type="fixed">
+    <parent link="base_link"/>
+    <child link="table_link"/>
+    <origin xyz="0.0 0.0 0.0" rpy="0 0 0"/>
+  </joint>
+  <link name="table_link">
     <visual>
       <origin xyz="0.0 0.4 0.0" rpy="${0.5*pi} 0 0"/>
@@ -29,6 +35,6 @@
     </collision>
   </link>
-  <xacro:autonomy_box_macro parent="base_link" alu_profile_collision_size_factor="1.25" name="autonomy_box" add_chilitags="false">
-    <origin xyz="0.205 0.0 0.005" rpy="0 0 0"/>
+  <xacro:autonomy_box_macro parent="table_link" alu_profile_collision_size_factor="1.25" name="autonomy_box" add_chilitags="false">
+    <origin xyz="0.255 0.0 0.005" rpy="0 0 0"/>
   </xacro:autonomy_box_macro>
 </robot>

Commit message: added collisoin geometry for table pushing person

File: hector_components_description/urdf/autonomy_box_on_table.urdf.xacro (robot description, xacro)
@@ -34,4 +34,10 @@
       </geometry>
     </collision>
+    <collision>
+      <origin xyz="-0.9 0.0 0.2" rpy="0 0 0"/>
+      <geometry>
+        <box size="1.0 1.0 2.0"/>
+      </geometry>
+    </collision>
   </link>
   <xacro:autonomy_box_macro parent="table_link" alu_profile_collision_size_factor="1.25" name="autonomy_box" add_chilitags="false">
