Commit message: rotated lidar

File: hector_components_description/urdf/autonomy_box.urdf.xacro (robot description, xacro)
@@ -236,5 +236,5 @@
     <!-- Spinning VLP16 -->
     <xacro:spinning_sensor_mount_macro parent="${name}_link"  name="spin_lidar" scaling="0.001">
-      <origin xyz="0 0 ${0.27 + 0.0944673}" rpy="0.0 0.0 ${M_PI}"/>
+      <origin xyz="0 0 ${0.27 + 0.0944673}" rpy="0.0 0.0 0.0"/>
     </xacro:spinning_sensor_mount_macro>
     <!-- 360 camera -->

Commit message: added collision model to camera360 macro added collision model to camera360 mount on autonomy box

File: hector_components_description/urdf/autonomy_box.urdf.xacro (robot description, xacro)
@@ -17,4 +17,7 @@
   <xacro:property name="handle_height" value="0.016"/>
   <xacro:property name="handle_y" value="0.138"/>
+  <xacro:property name="insta360_mounting_height" value="0.58"/>
+  <xacro:property name="insta360_radius" value="0.011"/>
+  <xacro:property name="insta360_collision_radius" value="0.015"/>
   <xacro:macro name="autonomy_box_macro" params="parent *origin alu_profile_collision_size_factor name:='autonomy_box'">
     <xacro:arg name="add_containment_self_filter_geom" default="false"/>
@@ -111,4 +114,14 @@
         </material>
       </visual>
+      <!-- 360 cam mount -->
+      <visual>
+        <origin xyz="0 0 ${0.5 * (top_protection_bottom + alu_profile_side_length + insta360_mounting_height - insta360_radius)}" rpy="0 0 0"/>
+        <geometry>
+          <box size="${alu_profile_side_length} ${alu_profile_side_length} ${insta360_mounting_height - top_protection_bottom - alu_profile_side_length - insta360_radius}"/>
+        </geometry>
+        <material name="Grey">
+          <color rgba="0.5 0.5 0.5 1"/>
+        </material>
+      </visual>
       <!-- Computer box-->
       <xacro:unless value="$(arg add_containment_self_filter_geom)">
@@ -199,4 +212,15 @@
           <!--<box size="${alu_profile_side_length} ${computer_box_width}  ${alu_profile_side_length}"/>-->
           <cylinder length="${computer_box_width}" radius="${alu_profile_side_length*0.5*alu_profile_collision_size_factor}"/>
+        </geometry>
+        <material name="Grey">
+          <color rgba="0.5 0.5 0.5 1"/>
+        </material>
+      </collision>
+      <!-- 360 cam mount -->
+      <collision>
+        <origin xyz="0 0 ${0.5 * (top_protection_bottom + alu_profile_side_length + insta360_mounting_height - insta360_radius)}" rpy="0 0 0"/>
+        <geometry>
+          <!--<box size="${computer_box_length} ${alu_profile_side_length} ${alu_profile_side_length}"/>-->
+          <cylinder length="${insta360_mounting_height - top_protection_bottom - alu_profile_side_length - insta360_radius}" radius="${alu_profile_side_length*0.5*alu_profile_collision_size_factor}"/>
         </geometry>
         <material name="Grey">
@@ -239,6 +263,6 @@
     </xacro:spinning_sensor_mount_macro>
     <!-- 360 camera -->
-    <xacro:camera360 name="camera360" right_cam_name="right" left_cam_name="left" parent="${name}_link" dist_between_cameras="-0.03850784" ros_topic="image_raw" update_rate="10" res_x="1504" res_y="1504" image_format="R8G8B8" fov="${M_PI}">
-      <origin xyz="0 0 0.58" rpy="0.0 0 0"/> <!-- base_link to camera mount transform -->
+    <xacro:camera360 name="camera360" right_cam_name="right" left_cam_name="left" parent="${name}_link" collision_radius="${insta360_collision_radius}" dist_between_cameras="-0.03850784" ros_topic="image_raw" update_rate="10" res_x="1504" res_y="1504" image_format="R8G8B8" fov="${M_PI}">
+      <origin xyz="0 0 ${insta360_mounting_height}" rpy="0.0 0 0"/> <!-- base_link to camera mount transform -->
       <origin xyz="0.00009742  0.00061696 -0.03850784" rpy="3.1373499 -0.0021358 -3.1279404"/> <!-- cam to cam transform (calibration by kalibr) -->
     </xacro:camera360>

File: hector_sensors_description/urdf/camera360.urdf.xacro (robot description, xacro)
@@ -2,5 +2,6 @@
 <robot xmlns:xacro="http://ros.org/wiki/xacro">
   <xacro:property name="M_PI" value="3.1415926535897931" />
-  <xacro:macro name="camera360" params="name right_cam_name left_cam_name parent *origin *calibration dist_between_cameras ros_topic update_rate res_x res_y image_format fov">
+  <xacro:property name="default_collision_radius" value="0.25" />
+  <xacro:macro name="camera360" params="name right_cam_name left_cam_name parent collision_radius:=${default_collision_radius} *origin *calibration dist_between_cameras ros_topic update_rate res_x res_y image_format fov">
     <joint name="${name}_center_joint" type="fixed">
       <xacro:insert_block name="origin" />
@@ -8,5 +9,24 @@
       <child link="${name}_center_link"/>
     </joint>
-    <link name="${name}_center_link" />
+    <link name="${name}_center_link">
+      <visual>
+        <origin xyz="0 0 0" rpy="0 0 0"/>
+        <geometry>
+          <sphere radius="0.011"/>
+        </geometry>
+        <material name="Grey">
+          <color rgba="0.5 0.5 0.5 1"/>
+        </material>
+      </visual>
+      <collision>
+        <origin xyz="0 0 0" rpy="0 0 0"/>
+        <geometry>
+          <sphere radius="${collision_radius}"/>
+        </geometry>
+        <material name="Grey">
+          <color rgba="0.5 0.5 0.5 1"/>
+        </material>
+      </collision>
+    </link>
     <joint name="${name}_${right_cam_name}_joint" type="fixed">
       <origin xyz="0 ${dist_between_cameras/2} 0" rpy="${M_PI*0.5} 0 ${-M_PI*0.5}"/>

Commit message: adjusted autonomy box sizes

File: hector_components_description/urdf/autonomy_box.urdf.xacro (robot description, xacro)
@@ -9,8 +9,8 @@
   <xacro:property name="M_PI" value="3.14159265359"/>
   <xacro:property name="alu_profile_side_length" value="0.02"/>
-  <xacro:property name="computer_box_height" value="0.15"/>
-  <xacro:property name="computer_box_width" value="0.191"/>
-  <xacro:property name="computer_box_length" value="0.191"/>
-  <xacro:property name="top_protection_bottom" value="0.47"/>
+  <xacro:property name="computer_box_height" value="0.121"/>
+  <xacro:property name="computer_box_width" value="0.19"/>
+  <xacro:property name="computer_box_length" value="0.19"/>
+  <xacro:property name="top_protection_bottom" value="0.4425"/>
   <xacro:property name="handle_width" value="0.07"/>
   <xacro:property name="handle_length" value="0.135"/>

Commit message: added chilitag to autonomy box

File: hector_components_description/urdf/autonomy_box.urdf.xacro (robot description, xacro)
@@ -20,4 +20,8 @@
   <xacro:property name="insta360_radius" value="0.011"/>
   <xacro:property name="insta360_collision_radius" value="0.015"/>
+  <xacro:property name="chilitag_white_border" value="0.005"/>
+  <xacro:property name="chilitag_28_x" value="${computer_box_width/2 - chilitag_white_border - chilitag_size/2}"/>
+  <xacro:property name="chilitag_28_y" value="${computer_box_width/2 - chilitag_white_border - chilitag_size/2}"/>
+  <xacro:property name="chilitag_28_z" value="${top_protection_bottom + alu_profile_side_length + 0.001}"/>
   <xacro:macro name="autonomy_box_macro" params="parent *origin alu_profile_collision_size_factor name:='autonomy_box'">
     <xacro:arg name="add_containment_self_filter_geom" default="false"/>
@@ -124,4 +128,8 @@
         </material>
       </visual>
+      <!-- Chilitags visual -->
+      <xacro:chilitag_visual_sized name="chilitag28" size="${chilitag_size}">
+        <origin xyz="${chilitag_28_x} ${chilitag_28_y} ${chilitag_28_z}" rpy="0 ${-M_PI/2} 0"/>
+      </xacro:chilitag_visual_sized>
       <!-- Computer box-->
       <xacro:unless value="$(arg add_containment_self_filter_geom)">
@@ -250,4 +258,8 @@
       </xacro:if>
     </link>
+        <!-- Chilitags -->
+    <xacro:chilitag_no_geom name="chilitag28" size="${chilitag_size}" parent="${name}_link">
+      <origin xyz="${chilitag_28_x} ${chilitag_28_y} ${chilitag_28_z}" rpy="${0} 0 ${0}" />
+    </xacro:chilitag_no_geom>
     <!-- IMU -->
     <joint name="imu_link_joint" type="fixed">

Commit message: fixed chilitag rotation

File: hector_components_description/urdf/autonomy_box.urdf.xacro (robot description, xacro)
@@ -130,5 +130,6 @@
       <!-- Chilitags visual -->
       <xacro:chilitag_visual_sized name="chilitag28" size="${chilitag_size}">
-        <origin xyz="${chilitag_28_x} ${chilitag_28_y} ${chilitag_28_z}" rpy="0 ${-M_PI/2} 0"/>
+<!--        <origin xyz="${chilitag_28_x} ${chilitag_28_y} ${chilitag_28_z}" rpy="0 ${-M_PI/2} 0"/>-->
+        <origin xyz="${chilitag_28_x} ${chilitag_28_y} ${chilitag_28_z}" rpy="${M_PI} ${0} ${M_PI/2}"/>
       </xacro:chilitag_visual_sized>
       <!-- Computer box-->
@@ -260,5 +261,5 @@
         <!-- Chilitags -->
     <xacro:chilitag_no_geom name="chilitag28" size="${chilitag_size}" parent="${name}_link">
-      <origin xyz="${chilitag_28_x} ${chilitag_28_y} ${chilitag_28_z}" rpy="${0} 0 ${0}" />
+        <origin xyz="${chilitag_28_x} ${chilitag_28_y} ${chilitag_28_z}" rpy="${M_PI} ${0} ${M_PI/2}"/>
     </xacro:chilitag_no_geom>
     <!-- IMU -->

Commit message: added collision for insta360 cable

File: hector_components_description/urdf/autonomy_box.urdf.xacro (robot description, xacro)
@@ -19,5 +19,5 @@
   <xacro:property name="insta360_mounting_height" value="0.58"/>
   <xacro:property name="insta360_radius" value="0.011"/>
-  <xacro:property name="insta360_collision_radius" value="0.015"/>
+  <xacro:property name="insta360_collision_radius" value="0.02"/>
   <xacro:property name="chilitag_white_border" value="0.005"/>
   <xacro:property name="chilitag_28_x" value="${computer_box_width/2 - chilitag_white_border - chilitag_size/2}"/>

File: hector_sensors_description/urdf/camera360.urdf.xacro (robot description, xacro)
@@ -3,4 +3,6 @@
   <xacro:property name="M_PI" value="3.1415926535897931" />
   <xacro:property name="default_collision_radius" value="0.25" />
+  <xacro:property name="visual_radius" value="0.011" />
+  <xacro:property name="cable_collision_length" value="0.05" />
   <xacro:macro name="camera360" params="name right_cam_name left_cam_name parent collision_radius:=${default_collision_radius} *origin *calibration dist_between_cameras ros_topic update_rate res_x res_y image_format fov">
     <joint name="${name}_center_joint" type="fixed">
@@ -10,8 +12,9 @@
     </joint>
     <link name="${name}_center_link">
+      <!-- Sphere body -->
       <visual>
         <origin xyz="0 0 0" rpy="0 0 0"/>
         <geometry>
-          <sphere radius="0.011"/>
+          <sphere radius="${visual_radius}"/>
         </geometry>
         <material name="Grey">
@@ -23,4 +26,23 @@
         <geometry>
           <sphere radius="${collision_radius}"/>
+        </geometry>
+        <material name="Grey">
+          <color rgba="0.5 0.5 0.5 1"/>
+        </material>
+      </collision>
+      <!-- Cable -->
+<!--      <visual>
+        <origin xyz="${visual_radius + cable_collision_length/2} 0 0" rpy="0 0 0"/>
+        <geometry>
+          <box size="${cable_collision_length} 0.03 0.03"/>
+        </geometry>
+        <material name="Grey">
+          <color rgba="0.5 0.5 0.5 1"/>
+        </material>
+      </visual>-->
+      <collision>
+        <origin xyz="${0.011 + cable_collision_length/2} 0 0" rpy="0 0 0"/>
+        <geometry>
+          <box size="${cable_collision_length} 0.03 0.03"/>
         </geometry>
         <material name="Grey">

Commit message: significatly increased collision model size of insta360

File: hector_components_description/urdf/autonomy_box.urdf.xacro (robot description, xacro)
@@ -19,5 +19,5 @@
   <xacro:property name="insta360_mounting_height" value="0.58"/>
   <xacro:property name="insta360_radius" value="0.011"/>
-  <xacro:property name="insta360_collision_radius" value="0.02"/>
+  <xacro:property name="insta360_collision_radius" value="0.04"/>
   <xacro:property name="chilitag_white_border" value="0.005"/>
   <xacro:property name="chilitag_28_x" value="${computer_box_width/2 - chilitag_white_border - chilitag_size/2}"/>

Commit message: added thickness of tags

File: hector_components_description/urdf/autonomy_box.urdf.xacro (robot description, xacro)
@@ -21,7 +21,8 @@
   <xacro:property name="insta360_collision_radius" value="0.04"/>
   <xacro:property name="chilitag_white_border" value="0.005"/>
+  <xacro:property name="chilitag_thickness" value="0.003"/>
   <xacro:property name="chilitag_28_x" value="${computer_box_width/2 - chilitag_white_border - chilitag_size/2}"/>
   <xacro:property name="chilitag_28_y" value="${computer_box_width/2 - chilitag_white_border - chilitag_size/2}"/>
-  <xacro:property name="chilitag_28_z" value="${top_protection_bottom + alu_profile_side_length + 0.001}"/>
+  <xacro:property name="chilitag_28_z" value="${top_protection_bottom + alu_profile_side_length + chilitag_thickness}"/>
   <xacro:macro name="autonomy_box_macro" params="parent *origin alu_profile_collision_size_factor name:='autonomy_box'">
     <xacro:arg name="add_containment_self_filter_geom" default="false"/>

Commit message: moved chilitag

File: hector_components_description/urdf/autonomy_box.urdf.xacro (robot description, xacro)
@@ -22,5 +22,5 @@
   <xacro:property name="chilitag_white_border" value="0.005"/>
   <xacro:property name="chilitag_thickness" value="0.003"/>
-  <xacro:property name="chilitag_28_x" value="${computer_box_width/2 - chilitag_white_border - chilitag_size/2}"/>
+  <xacro:property name="chilitag_28_x" value="${-computer_box_width/2 + 0.01 + chilitag_size/2}"/> <!-- border is bigger on this side -->
   <xacro:property name="chilitag_28_y" value="${computer_box_width/2 - chilitag_white_border - chilitag_size/2}"/>
   <xacro:property name="chilitag_28_z" value="${top_protection_bottom + alu_profile_side_length + chilitag_thickness}"/>

File: hector_sensors_description/urdf/realsense_d435_camera.urdf.xacro (robot description, xacro)
@@ -75,10 +75,10 @@
           <plugin name="${name}_camera_controller" filename="libgazebo_ros_openni_kinect.so">
             <cameraName>${name}</cameraName>
-            <imageTopicName>rgb/${image_topic}</imageTopicName>
-            <cameraInfoTopicName>rgb/camera_info</cameraInfoTopicName>
+            <imageTopicName>color/${image_topic}</imageTopicName>
+            <cameraInfoTopicName>color/camera_info</cameraInfoTopicName>
             <depthImageTopicName>depth/image_raw</depthImageTopicName>
             <depthImageCameraInfoTopicName>depth/camera_info</depthImageCameraInfoTopicName>
             <pointCloudTopicName>${depth_points_topic}</pointCloudTopicName>
-            <frameName>${name}_depth_optical_frame</frameName>
+            <frameName>${name}_color_optical_frame</frameName>
           </plugin>
         </sensor>

Commit message: updated chilitag

File: hector_components_description/urdf/autonomy_box.urdf.xacro (robot description, xacro)
@@ -22,7 +22,7 @@
   <xacro:property name="chilitag_white_border" value="0.005"/>
   <xacro:property name="chilitag_thickness" value="0.003"/>
-  <xacro:property name="chilitag_28_x" value="${-computer_box_width/2 + 0.01 + chilitag_size/2}"/> <!-- border is bigger on this side -->
-  <xacro:property name="chilitag_28_y" value="${computer_box_width/2 - chilitag_white_border - chilitag_size/2}"/>
-  <xacro:property name="chilitag_28_z" value="${top_protection_bottom + alu_profile_side_length + chilitag_thickness}"/>
+  <xacro:property name="chilitag_29_x" value="${-computer_box_width/2 + 0.01 + chilitag_size/2}"/> <!-- border is bigger on this side -->
+  <xacro:property name="chilitag_29_y" value="${-computer_box_width/2 + 2*chilitag_white_border + chilitag_size/2}"/>
+  <xacro:property name="chilitag_29_z" value="${top_protection_bottom + alu_profile_side_length + chilitag_thickness}"/>
   <xacro:macro name="autonomy_box_macro" params="parent *origin alu_profile_collision_size_factor name:='autonomy_box'">
     <xacro:arg name="add_containment_self_filter_geom" default="false"/>
@@ -130,7 +130,7 @@
       </visual>
       <!-- Chilitags visual -->
-      <xacro:chilitag_visual_sized name="chilitag28" size="${chilitag_size}">
+      <xacro:chilitag_visual_sized name="chilitag29" size="${chilitag_size}">
 <!--        <origin xyz="${chilitag_28_x} ${chilitag_28_y} ${chilitag_28_z}" rpy="0 ${-M_PI/2} 0"/>-->
-        <origin xyz="${chilitag_28_x} ${chilitag_28_y} ${chilitag_28_z}" rpy="${M_PI} ${0} ${M_PI/2}"/>
+        <origin xyz="${chilitag_29_x} ${chilitag_29_y} ${chilitag_29_z}" rpy="${M_PI} ${0} ${-M_PI/2}"/>
       </xacro:chilitag_visual_sized>
       <!-- Computer box-->
@@ -260,7 +260,7 @@
       </xacro:if>
     </link>
-        <!-- Chilitags -->
-    <xacro:chilitag_no_geom name="chilitag28" size="${chilitag_size}" parent="${name}_link">
-        <origin xyz="${chilitag_28_x} ${chilitag_28_y} ${chilitag_28_z}" rpy="${M_PI} ${0} ${M_PI/2}"/>
+    <!-- Chilitags -->
+    <xacro:chilitag_no_geom name="chilitag29" size="${chilitag_size}" parent="${name}_link">
+      <origin xyz="${chilitag_29_x} ${chilitag_29_y} ${chilitag_29_z}" rpy="${M_PI} ${0} ${-M_PI/2}"/>
     </xacro:chilitag_no_geom>
     <!-- IMU -->

Commit message: rotate the spinning lidar 180° to be compatible to the legacy dynamixel driver

File: hector_components_description/urdf/autonomy_box.urdf.xacro (robot description, xacro)
@@ -274,5 +274,5 @@
     <!-- Spinning VLP16 -->
     <xacro:spinning_sensor_mount_macro parent="${name}_link"  name="spin_lidar" scaling="0.001">
-      <origin xyz="0 0 ${0.27 + 0.0944673}" rpy="0.0 0.0 0.0"/>
+      <origin xyz="0 0 ${0.27 + 0.0944673}" rpy="0.0 0.0 ${M_PI}"/>
     </xacro:spinning_sensor_mount_macro>
     <!-- 360 camera -->

Commit message: fixed chilitag position

File: hector_components_description/urdf/autonomy_box.urdf.xacro (robot description, xacro)
@@ -22,5 +22,5 @@
   <xacro:property name="chilitag_white_border" value="0.005"/>
   <xacro:property name="chilitag_thickness" value="0.003"/>
-  <xacro:property name="chilitag_29_x" value="${-computer_box_width/2 + 0.01 + chilitag_size/2}"/> <!-- border is bigger on this side -->
+  <xacro:property name="chilitag_29_x" value="${-computer_box_width/2 + chilitag_white_border + chilitag_size/2}"/> <!-- border is bigger on this side -->
   <xacro:property name="chilitag_29_y" value="${-computer_box_width/2 + 2*chilitag_white_border + chilitag_size/2}"/>
   <xacro:property name="chilitag_29_z" value="${top_protection_bottom + alu_profile_side_length + chilitag_thickness}"/>

Commit message: insta 3 exstrinsic calibration

File: hector_components_description/urdf/autonomy_box.urdf.xacro (robot description, xacro)
@@ -279,5 +279,7 @@
     <xacro:camera360 name="camera360" right_cam_name="right" left_cam_name="left" parent="${name}_link" collision_radius="${insta360_collision_radius}" dist_between_cameras="-0.03850784" ros_topic="image_raw" update_rate="10" res_x="1504" res_y="1504" image_format="R8G8B8" fov="${M_PI}">
       <origin xyz="0 0 ${insta360_mounting_height}" rpy="0.0 0 0"/> <!-- base_link to camera mount transform -->
-      <origin xyz="0.00009742  0.00061696 -0.03850784" rpy="3.1373499 -0.0021358 -3.1279404"/> <!-- cam to cam transform (calibration by kalibr) -->
+      <!-- cam to cam transform (calibration by kalibr) -->
+      <!--<origin xyz="0.00009742  0.00061696 -0.03850784" rpy="3.1373499 -0.0021358 -3.1279404"/>--> <!-- insta #1 -->
+      <origin xyz="0.002862424041614364  -0.00013127655875068252 -0.03724378451297336" rpy="-3.1402707 0.0036289 -3.1175768"/> <!-- insta #3 -->
     </xacro:camera360>
     <gazebo reference="structure_addons_link">

Commit message: Add missing chilitag include (should be removed completely in the future) Add imu_link as a param with default

File: hector_components_description/urdf/autonomy_box.urdf.xacro (robot description, xacro)
@@ -5,4 +5,5 @@
   <xacro:include filename="$(find hector_components_description)/urdf/vlp16_mount.urdf.xacro.xml"/>
   <xacro:include filename="$(find hector_sensors_description)/urdf/camera360.urdf.xacro"/>
+  <xacro:include filename="$(find hector_chilitag_description)/urdf/chilitag.urdf.xacro"/>
 <!--  <xacro:arg name="add_self_filter_geom" default="0"/>-->
   <!--<xacro:property name="add_self_filter_geom" value="${arg add_self_filter_geom}"/>-->
@@ -25,5 +26,5 @@
   <xacro:property name="chilitag_29_y" value="${-computer_box_width/2 + 2*chilitag_white_border + chilitag_size/2}"/>
   <xacro:property name="chilitag_29_z" value="${top_protection_bottom + alu_profile_side_length + chilitag_thickness}"/>
-  <xacro:macro name="autonomy_box_macro" params="parent *origin alu_profile_collision_size_factor name:='autonomy_box'">
+  <xacro:macro name="autonomy_box_macro" params="parent *origin alu_profile_collision_size_factor name:='autonomy_box' imu_link='imu_link'">
     <xacro:arg name="add_containment_self_filter_geom" default="false"/>
     <joint name="${name}_joint" type="fixed">
@@ -268,7 +269,7 @@
       <origin xyz="0 0 0" rpy="0 0 0"/>
       <parent link="${name}_link" />
-      <child link="imu_link"/>
+      <child link="${imu_link}"/>
     </joint>
-    <link name="imu_link">
+    <link name="${imu_link}">
     </link>
     <!-- Spinning VLP16 -->

Commit message: Fix autonomy box material color

File: hector_components_description/urdf/autonomy_box.urdf.xacro (robot description, xacro)
@@ -284,6 +284,13 @@
       <origin xyz="0.002862424041614364  -0.00013127655875068252 -0.03724378451297336" rpy="-3.1402707 0.0036289 -3.1175768"/> <!-- insta #3 -->
     </xacro:camera360>
-    <gazebo reference="structure_addons_link">
-      <material>Gazebo/Grey</material>
+    <gazebo reference="${name}_link">
+      <visual>
+      <material>
+        <ambient>0.1 0.1 0.1 1</ambient>
+        <diffuse>0.48 0.48 0.48 1</diffuse>
+        <emissive>0.237 0.237 0.237 1</emissive>
+        <specular>0.8 0.8 0.8 1</specular>
+      </material>
+    </visual>
     </gazebo>
   </xacro:macro>

Commit message: switched back to new dynamixel controller (which reports positions with an offset of pi)

File: hector_components_description/urdf/autonomy_box.urdf.xacro (robot description, xacro)
@@ -275,5 +275,5 @@
     <!-- Spinning VLP16 -->
     <xacro:spinning_sensor_mount_macro parent="${name}_link"  name="spin_lidar" scaling="0.001">
-      <origin xyz="0 0 ${0.27 + 0.0944673}" rpy="0.0 0.0 ${M_PI}"/>
+      <origin xyz="0 0 ${0.27 + 0.0944673}" rpy="0.0 0.0 0.0"/>
     </xacro:spinning_sensor_mount_macro>
     <!-- 360 camera -->

Commit message: Revert "switched back to new dynamixel controller (which reports positions with an offset of pi)"
This reverts commit a9de57af00b22a533b5f1e452efc315a02ba4ca0.

File: hector_components_description/urdf/autonomy_box.urdf.xacro (robot description, xacro)
@@ -275,5 +275,5 @@
     <!-- Spinning VLP16 -->
     <xacro:spinning_sensor_mount_macro parent="${name}_link"  name="spin_lidar" scaling="0.001">
-      <origin xyz="0 0 ${0.27 + 0.0944673}" rpy="0.0 0.0 0.0"/>
+      <origin xyz="0 0 ${0.27 + 0.0944673}" rpy="0.0 0.0 ${M_PI}"/>
     </xacro:spinning_sensor_mount_macro>
     <!-- 360 camera -->
