Commit message: added realsense t265 tracking camera to autonomy box

File: hector_components_description/urdf/autonomy_box.urdf.xacro (robot description, xacro)
@@ -6,4 +6,5 @@
   <xacro:include filename="$(find hector_sensors_description)/urdf/camera360.urdf.xacro"/>
   <xacro:include filename="$(find hector_chilitag_description)/urdf/chilitag.urdf.xacro"/>
+  <xacro:include filename="$(find hector_sensors_description)/urdf/realsense_t265.urdf.xacro"/>
 <!--  <xacro:arg name="add_self_filter_geom" default="0"/>-->
   <!--<xacro:property name="add_self_filter_geom" value="${arg add_self_filter_geom}"/>-->
@@ -284,4 +285,8 @@
       <origin xyz="0.002862424041614364  -0.00013127655875068252 -0.03724378451297336" rpy="-3.1402707 0.0036289 -3.1175768"/> <!-- insta #3 -->
     </xacro:camera360>
+    <!-- Realsense T265 Tracking camera -->
+    <xacro:realsense_t265_tracking_camera_housing name="tracking_camera" parent="${name}_link">
+      <origin xyz="${computer_box_width/2.0 - alu_profile_side_length + realsense_t265_depth/2.0} ${computer_box_width/2.0 - alu_profile_side_length - realsense_t265_width/2.0} ${top_protection_bottom - realsense_t265_height/2.0}" rpy="0 0 0"/>
+    </xacro:realsense_t265_tracking_camera_housing>
     <gazebo reference="${name}_link">
       <visual>

Commit message: added parameter to add chilitags in autonomy box macro

File: hector_components_description/urdf/autonomy_box.urdf.xacro (robot description, xacro)
@@ -5,26 +5,28 @@
   <xacro:include filename="$(find hector_components_description)/urdf/vlp16_mount.urdf.xacro.xml"/>
   <xacro:include filename="$(find hector_sensors_description)/urdf/camera360.urdf.xacro"/>
-  <xacro:include filename="$(find hector_chilitag_description)/urdf/chilitag.urdf.xacro"/>
 <!--  <xacro:arg name="add_self_filter_geom" default="0"/>-->
   <!--<xacro:property name="add_self_filter_geom" value="${arg add_self_filter_geom}"/>-->
   <xacro:property name="M_PI" value="3.14159265359"/>
-  <xacro:property name="alu_profile_side_length" value="0.02"/>
-  <xacro:property name="computer_box_height" value="0.121"/>
-  <xacro:property name="computer_box_width" value="0.19"/>
-  <xacro:property name="computer_box_length" value="0.19"/>
-  <xacro:property name="top_protection_bottom" value="0.4425"/>
-  <xacro:property name="handle_width" value="0.07"/>
-  <xacro:property name="handle_length" value="0.135"/>
-  <xacro:property name="handle_height" value="0.016"/>
-  <xacro:property name="handle_y" value="0.138"/>
-  <xacro:property name="insta360_mounting_height" value="0.58"/>
-  <xacro:property name="insta360_radius" value="0.011"/>
-  <xacro:property name="insta360_collision_radius" value="0.04"/>
-  <xacro:property name="chilitag_white_border" value="0.005"/>
-  <xacro:property name="chilitag_thickness" value="0.003"/>
-  <xacro:property name="chilitag_29_x" value="${-computer_box_width/2 + chilitag_white_border + chilitag_size/2}"/> <!-- border is bigger on this side -->
-  <xacro:property name="chilitag_29_y" value="${-computer_box_width/2 + 2*chilitag_white_border + chilitag_size/2}"/>
-  <xacro:property name="chilitag_29_z" value="${top_protection_bottom + alu_profile_side_length + chilitag_thickness}"/>
-  <xacro:macro name="autonomy_box_macro" params="parent *origin alu_profile_collision_size_factor name:='autonomy_box' imu_link='imu_link'">
+  <xacro:macro name="autonomy_box_macro" params="parent *origin alu_profile_collision_size_factor name:='autonomy_box' imu_link='imu_link' add_chilitags:='true'">
+    <xacro:if value="${add_chilitags}">
+      <xacro:include filename="$(find hector_chilitag_description)/urdf/chilitag.urdf.xacro"/>
+      <xacro:property name="chilitag_white_border" value="0.005"/>
+      <xacro:property name="chilitag_thickness" value="0.003"/>
+      <xacro:property name="chilitag_29_x" value="${-computer_box_width/2 + chilitag_white_border + chilitag_size/2}"/> <!-- border is bigger on this side -->
+      <xacro:property name="chilitag_29_y" value="${-computer_box_width/2 + 2*chilitag_white_border + chilitag_size/2}"/>
+      <xacro:property name="chilitag_29_z" value="${top_protection_bottom + alu_profile_side_length + chilitag_thickness}"/>
+    </xacro:if>
+    <xacro:property name="alu_profile_side_length" value="0.02"/>
+    <xacro:property name="computer_box_height" value="0.121"/>
+    <xacro:property name="computer_box_width" value="0.19"/>
+    <xacro:property name="computer_box_length" value="0.19"/>
+    <xacro:property name="top_protection_bottom" value="0.4425"/>
+    <xacro:property name="handle_width" value="0.07"/>
+    <xacro:property name="handle_length" value="0.135"/>
+    <xacro:property name="handle_height" value="0.016"/>
+    <xacro:property name="handle_y" value="0.138"/>
+    <xacro:property name="insta360_mounting_height" value="0.58"/>
+    <xacro:property name="insta360_radius" value="0.011"/>
+    <xacro:property name="insta360_collision_radius" value="0.04"/>
     <xacro:arg name="add_containment_self_filter_geom" default="false"/>
     <joint name="${name}_joint" type="fixed">
@@ -131,8 +133,10 @@
       </visual>
       <!-- Chilitags visual -->
-      <xacro:chilitag_visual_sized name="chilitag29" size="${chilitag_size}">
-<!--        <origin xyz="${chilitag_28_x} ${chilitag_28_y} ${chilitag_28_z}" rpy="0 ${-M_PI/2} 0"/>-->
-        <origin xyz="${chilitag_29_x} ${chilitag_29_y} ${chilitag_29_z}" rpy="${M_PI} ${0} ${-M_PI/2}"/>
-      </xacro:chilitag_visual_sized>
+      <xacro:if value="${add_chilitags}">
+        <xacro:chilitag_visual_sized name="chilitag29" size="${chilitag_size}">
+  <!--        <origin xyz="${chilitag_28_x} ${chilitag_28_y} ${chilitag_28_z}" rpy="0 ${-M_PI/2} 0"/>-->
+          <origin xyz="${chilitag_29_x} ${chilitag_29_y} ${chilitag_29_z}" rpy="${M_PI} ${0} ${-M_PI/2}"/>
+        </xacro:chilitag_visual_sized>
+      </xacro:if>
       <!-- Computer box-->
       <xacro:unless value="$(arg add_containment_self_filter_geom)">
@@ -262,7 +266,9 @@
     </link>
     <!-- Chilitags -->
-    <xacro:chilitag_no_geom name="chilitag29" size="${chilitag_size}" parent="${name}_link">
-      <origin xyz="${chilitag_29_x} ${chilitag_29_y} ${chilitag_29_z}" rpy="${M_PI} ${0} ${-M_PI/2}"/>
-    </xacro:chilitag_no_geom>
+    <xacro:if value="${add_chilitags}">
+      <xacro:chilitag_no_geom name="chilitag29" size="${chilitag_size}" parent="${name}_link">
+        <origin xyz="${chilitag_29_x} ${chilitag_29_y} ${chilitag_29_z}" rpy="${M_PI} ${0} ${-M_PI/2}"/>
+      </xacro:chilitag_no_geom>
+    </xacro:if>
     <!-- IMU -->
     <joint name="imu_link_joint" type="fixed">

Commit message: moved autonomy box properties outside of macro scope again

File: hector_components_description/urdf/autonomy_box.urdf.xacro (robot description, xacro)
@@ -7,4 +7,12 @@
 <!--  <xacro:arg name="add_self_filter_geom" default="0"/>-->
   <!--<xacro:property name="add_self_filter_geom" value="${arg add_self_filter_geom}"/>-->
+  <xacro:property name="alu_profile_side_length" value="0.02"/>
+  <xacro:property name="computer_box_height" value="0.121"/>
+  <xacro:property name="computer_box_width" value="0.19"/>
+  <xacro:property name="computer_box_length" value="0.19"/>
+  <xacro:property name="top_protection_bottom" value="0.4425"/>
+  <xacro:property name="insta360_mounting_height" value="0.58"/>
+  <xacro:property name="insta360_radius" value="0.011"/>
+  <xacro:property name="insta360_collision_radius" value="0.04"/>
   <xacro:property name="M_PI" value="3.14159265359"/>
   <xacro:macro name="autonomy_box_macro" params="parent *origin alu_profile_collision_size_factor name:='autonomy_box' imu_link='imu_link' add_chilitags:='true'">
@@ -17,16 +25,4 @@
       <xacro:property name="chilitag_29_z" value="${top_protection_bottom + alu_profile_side_length + chilitag_thickness}"/>
     </xacro:if>
-    <xacro:property name="alu_profile_side_length" value="0.02"/>
-    <xacro:property name="computer_box_height" value="0.121"/>
-    <xacro:property name="computer_box_width" value="0.19"/>
-    <xacro:property name="computer_box_length" value="0.19"/>
-    <xacro:property name="top_protection_bottom" value="0.4425"/>
-    <xacro:property name="handle_width" value="0.07"/>
-    <xacro:property name="handle_length" value="0.135"/>
-    <xacro:property name="handle_height" value="0.016"/>
-    <xacro:property name="handle_y" value="0.138"/>
-    <xacro:property name="insta360_mounting_height" value="0.58"/>
-    <xacro:property name="insta360_radius" value="0.011"/>
-    <xacro:property name="insta360_collision_radius" value="0.04"/>
     <xacro:arg name="add_containment_self_filter_geom" default="false"/>
     <joint name="${name}_joint" type="fixed">

Commit message: fixed insta360 and lidar mounting height

File: hector_components_description/urdf/autonomy_box.urdf.xacro (robot description, xacro)
@@ -12,5 +12,5 @@
   <xacro:property name="computer_box_length" value="0.19"/>
   <xacro:property name="top_protection_bottom" value="0.4425"/>
-  <xacro:property name="insta360_mounting_height" value="0.58"/>
+  <xacro:property name="insta360_mounting_height" value="${top_protection_bottom + alu_profile_side_length + 0.12}"/>
   <xacro:property name="insta360_radius" value="0.011"/>
   <xacro:property name="insta360_collision_radius" value="0.04"/>
@@ -277,5 +277,5 @@
     <!-- Spinning VLP16 -->
     <xacro:spinning_sensor_mount_macro parent="${name}_link"  name="spin_lidar" scaling="0.001">
-      <origin xyz="0 0 ${0.27 + 0.0944673}" rpy="0.0 0.0 0.0"/>
+      <origin xyz="0 0 ${0.27 + 0.0944673 - 0.029}" rpy="0.0 0.0 0.0"/>
     </xacro:spinning_sensor_mount_macro>
     <!-- 360 camera -->

Commit message: removed containment filter box for jasmine arm from autonomy box macro

File: hector_components_description/urdf/autonomy_box.urdf.xacro (robot description, xacro)
@@ -250,5 +250,5 @@
         </material>
       </collision>
-      <collision>
+<!--      <collision>
         <origin xyz="-0.18 0 ${computer_box_height/2+0.07}" rpy="0 0 0"/>
         <geometry>
@@ -258,5 +258,5 @@
           <color rgba="0.5 0.5 0.5 1"/>
         </material>
-      </collision>
+      </collision>-->
       </xacro:if>
     </link>

Commit message: added front/back realsenses to autonomy box

File: hector_components_description/urdf/autonomy_box.urdf.xacro (robot description, xacro)
@@ -286,4 +286,17 @@
       <origin xyz="0.002862424041614364  -0.00013127655875068252 -0.03724378451297336" rpy="-3.1402707 0.0036289 -3.1175768"/> <!-- insta #3 -->
     </xacro:camera360>
+    <!-- +++++ Cage Realsenses +++++ -->
+    <xacro:property name="autonomy_box_realsense_x_offset" value="0.1"/>
+    <xacro:property name="autonomy_box_realsense_y_offset" value="0.0"/>
+    <xacro:property name="autonomy_box_realsense_z_offset" value="0.01"/>
+    <xacro:property name="autonomy_box_realsense_pitch" value="${25*M_PI/180.0}"/>
+    <!-- Realsense D435 front -->
+    <xacro:realsense_d435_camera_comprehensive_params name="front_rgbd_cam" parent="${name}_link" image_topic="image_rect_color" depth_points_topic="depth/points" min_range="0.3" max_range="9.0" update_rate="20">
+      <origin xyz="${autonomy_box_realsense_x_offset} ${autonomy_box_realsense_y_offset} ${top_protection_bottom + alu_profile_side_length + autonomy_box_realsense_z_offset}" rpy="0.0 ${autonomy_box_realsense_pitch} 0"/>
+    </xacro:realsense_d435_camera_comprehensive_params>
+    <!-- Realsense D435 back -->
+    <xacro:realsense_d435_camera_comprehensive_params name="back_rgbd_cam" parent="${name}_link" image_topic="image_rect_color" depth_points_topic="depth/points" min_range="0.3" max_range="9.0" update_rate="20">
+      <origin xyz="${-1 * autonomy_box_realsense_x_offset} ${autonomy_box_realsense_y_offset} ${top_protection_bottom + alu_profile_side_length + autonomy_box_realsense_z_offset}" rpy="0.0 ${autonomy_box_realsense_pitch} ${M_PI}"/>
+    </xacro:realsense_d435_camera_comprehensive_params>
     <gazebo reference="${name}_link">
       <visual>

Commit message: corrected sizes of autonomy box

File: hector_components_description/urdf/autonomy_box.urdf.xacro (robot description, xacro)
@@ -8,8 +8,8 @@
   <!--<xacro:property name="add_self_filter_geom" value="${arg add_self_filter_geom}"/>-->
   <xacro:property name="alu_profile_side_length" value="0.02"/>
-  <xacro:property name="computer_box_height" value="0.121"/>
+  <xacro:property name="computer_box_height" value="0.119"/>
   <xacro:property name="computer_box_width" value="0.19"/>
   <xacro:property name="computer_box_length" value="0.19"/>
-  <xacro:property name="top_protection_bottom" value="0.4425"/>
+  <xacro:property name="top_protection_bottom" value="${computer_box_height + 0.32}"/>
   <xacro:property name="insta360_mounting_height" value="${top_protection_bottom + alu_profile_side_length + 0.12}"/>
   <xacro:property name="insta360_radius" value="0.011"/>
@@ -277,5 +277,5 @@
     <!-- Spinning VLP16 -->
     <xacro:spinning_sensor_mount_macro parent="${name}_link"  name="spin_lidar" scaling="0.001">
-      <origin xyz="0 0 ${0.27 + 0.0944673 - 0.029}" rpy="0.0 0.0 0.0"/>
+      <origin xyz="0 0 ${0.27 + 0.0944673 - 0.025}" rpy="0.0 0.0 0.0"/>
     </xacro:spinning_sensor_mount_macro>
     <!-- 360 camera -->
@@ -287,11 +287,12 @@
     </xacro:camera360>
     <!-- +++++ Cage Realsenses +++++ -->
-    <xacro:property name="autonomy_box_realsense_x_offset" value="0.1"/>
-    <xacro:property name="autonomy_box_realsense_y_offset" value="0.0"/>
-    <xacro:property name="autonomy_box_realsense_z_offset" value="0.01"/>
+    <xacro:property name="autonomy_box_realsense_x_offset" value="0.08743"/>
+    <xacro:property name="autonomy_box_realsense_y_offset" value="0.015"/>
+    <xacro:property name="autonomy_box_realsense_z_offset" value="0.00995"/>
+<!--     <xacro:property name="autonomy_box_realsense_z_offset" value="0.46895"/> -->
     <xacro:property name="autonomy_box_realsense_pitch" value="${25*M_PI/180.0}"/>
     <!-- Realsense D435 front -->
     <xacro:realsense_d435_camera_comprehensive_params name="front_rgbd_cam" parent="${name}_link" image_topic="image_rect_color" depth_points_topic="depth/points" min_range="0.3" max_range="9.0" update_rate="20">
-      <origin xyz="${autonomy_box_realsense_x_offset} ${autonomy_box_realsense_y_offset} ${top_protection_bottom + alu_profile_side_length + autonomy_box_realsense_z_offset}" rpy="0.0 ${autonomy_box_realsense_pitch} 0"/>
+      <origin xyz="${autonomy_box_realsense_x_offset} ${-1 * autonomy_box_realsense_y_offset} ${top_protection_bottom + alu_profile_side_length + autonomy_box_realsense_z_offset}" rpy="0.0 ${autonomy_box_realsense_pitch} 0"/>
     </xacro:realsense_d435_camera_comprehensive_params>
     <!-- Realsense D435 back -->

Commit message: fixed lidar position realsense origin is now in mounting hole

File: hector_components_description/urdf/autonomy_box.urdf.xacro (robot description, xacro)
@@ -277,5 +277,5 @@
     <!-- Spinning VLP16 -->
     <xacro:spinning_sensor_mount_macro parent="${name}_link"  name="spin_lidar" scaling="0.001">
-      <origin xyz="0 0 ${0.27 + 0.0944673 - 0.025}" rpy="0.0 0.0 0.0"/>
+      <origin xyz="0 0 0.34708" rpy="0.0 0.0 0.0"/>
     </xacro:spinning_sensor_mount_macro>
     <!-- 360 camera -->
@@ -287,17 +287,17 @@
     </xacro:camera360>
     <!-- +++++ Cage Realsenses +++++ -->
-    <xacro:property name="autonomy_box_realsense_x_offset" value="0.08743"/>
-    <xacro:property name="autonomy_box_realsense_y_offset" value="0.015"/>
-    <xacro:property name="autonomy_box_realsense_z_offset" value="0.00995"/>
+    <xacro:property name="autonomy_box_realsense_x_offset" value="0.07187"/>
+    <xacro:property name="autonomy_box_realsense_y_offset" value="0.03"/>
+    <xacro:property name="autonomy_box_realsense_z_offset" value="0.00395"/>
 <!--     <xacro:property name="autonomy_box_realsense_z_offset" value="0.46895"/> -->
     <xacro:property name="autonomy_box_realsense_pitch" value="${25*M_PI/180.0}"/>
     <!-- Realsense D435 front -->
-    <xacro:realsense_d435_camera_comprehensive_params name="front_rgbd_cam" parent="${name}_link" image_topic="image_rect_color" depth_points_topic="depth/points" min_range="0.3" max_range="9.0" update_rate="20">
+    <xacro:realsense_d435_camera_with_mount_comprehensive_params name="front_rgbd_cam" parent="${name}_link" image_topic="image_rect_color" depth_points_topic="depth/color/points" min_range="0.3" max_range="9.0" update_rate="20">
       <origin xyz="${autonomy_box_realsense_x_offset} ${-1 * autonomy_box_realsense_y_offset} ${top_protection_bottom + alu_profile_side_length + autonomy_box_realsense_z_offset}" rpy="0.0 ${autonomy_box_realsense_pitch} 0"/>
-    </xacro:realsense_d435_camera_comprehensive_params>
+    </xacro:realsense_d435_camera_with_mount_comprehensive_params>
     <!-- Realsense D435 back -->
-    <xacro:realsense_d435_camera_comprehensive_params name="back_rgbd_cam" parent="${name}_link" image_topic="image_rect_color" depth_points_topic="depth/points" min_range="0.3" max_range="9.0" update_rate="20">
+    <xacro:realsense_d435_camera_with_mount_comprehensive_params name="back_rgbd_cam" parent="${name}_link" image_topic="image_rect_color" depth_points_topic="depth/color/points" min_range="0.3" max_range="9.0" update_rate="20">
       <origin xyz="${-1 * autonomy_box_realsense_x_offset} ${autonomy_box_realsense_y_offset} ${top_protection_bottom + alu_profile_side_length + autonomy_box_realsense_z_offset}" rpy="0.0 ${autonomy_box_realsense_pitch} ${M_PI}"/>
-    </xacro:realsense_d435_camera_comprehensive_params>
+    </xacro:realsense_d435_camera_with_mount_comprehensive_params>
     <gazebo reference="${name}_link">
       <visual>

Commit message: added collision geom to lidar for manipulation

File: hector_components_description/urdf/autonomy_box.urdf.xacro (robot description, xacro)
@@ -17,4 +17,6 @@
   <xacro:property name="M_PI" value="3.14159265359"/>
   <xacro:macro name="autonomy_box_macro" params="parent *origin alu_profile_collision_size_factor name:='autonomy_box' imu_link='imu_link' add_chilitags:='true'">
+    <xacro:arg name="add_containment_self_filter_geom" default="false"/>
+    <xacro:arg name="add_manipulation_geom" default="false"/>
     <xacro:if value="${add_chilitags}">
       <xacro:include filename="$(find hector_chilitag_description)/urdf/chilitag.urdf.xacro"/>
@@ -25,5 +27,4 @@
       <xacro:property name="chilitag_29_z" value="${top_protection_bottom + alu_profile_side_length + chilitag_thickness}"/>
     </xacro:if>
-    <xacro:arg name="add_containment_self_filter_geom" default="false"/>
     <joint name="${name}_joint" type="fixed">
       <xacro:insert_block name="origin"/>
@@ -239,4 +240,16 @@
         </material>
       </collision>
+      <xacro:if value="$(arg add_manipulation_geom)">
+        <!-- Lidar protection geom -->
+        <collision>
+          <origin xyz="0 0 ${computer_box_height + 0.5*(top_protection_bottom - computer_box_height)}" rpy="0 0 0"/>
+          <geometry>
+            <cylinder length="${top_protection_bottom - computer_box_height}" radius="${computer_box_width / 2.0}"/>
+          </geometry>
+          <material name="Grey">
+            <color rgba="0.5 0.5 0.5 1"/>
+          </material>
+        </collision>
+      </xacro:if>
       </xacro:unless>
       <xacro:if value="$(arg add_containment_self_filter_geom)">

Commit message: moved t265

File: hector_components_description/urdf/autonomy_box.urdf.xacro (robot description, xacro)
@@ -302,5 +302,5 @@
     <!-- Realsense T265 Tracking camera -->
     <xacro:realsense_t265_tracking_camera name="tracking_camera" parent="${name}_link">
-      <origin xyz="${computer_box_width/2.0 - alu_profile_side_length + realsense_t265_depth/2.0} ${computer_box_width/2.0 - alu_profile_side_length - realsense_t265_width/2.0} ${top_protection_bottom - realsense_t265_height/2.0}" rpy="0 0 0"/>
+      <origin xyz="${computer_box_width/2.0 - realsense_t265_depth/2.0} ${computer_box_width/2.0 - alu_profile_side_length - realsense_t265_width/2.0} ${top_protection_bottom - realsense_t265_height/2.0}" rpy="0 0 0"/>
     </xacro:realsense_t265_tracking_camera>
     <!-- +++++ Cage Realsenses +++++ -->
