Commit message: Fixed misaligned depth cloud

File: hector_components_description/urdf/autonomy_box.urdf.xacro (robot description, xacro)
@@ -229,9 +229,9 @@
     <xacro:property name="autonomy_box_realsense_pitch" value="${25*M_PI/180.0}"/>
     <!-- Realsense D435 front -->
-    <xacro:realsense_d435_camera_with_mount_comprehensive_params name="front_rgbd_cam" parent="${name}_link" image_topic="image_rect_color" depth_topic="image_rect_raw" depth_points_topic="depth/color/points" min_range="0.3" max_range="9.0" update_rate="15">
+    <xacro:realsense_d435_camera_with_mount_comprehensive_params name="front_rgbd_cam" parent="${name}_link" image_topic="image_rect_color" depth_topic="image_rect_raw" depth_points_topic="depth/color/points" frame_name="depth" min_range="0.3" max_range="9.0" update_rate="15">
       <origin xyz="${autonomy_box_realsense_x_offset} ${-1 * autonomy_box_realsense_y_offset} ${top_protection_bottom + alu_profile_side_length + autonomy_box_realsense_z_offset}" rpy="0.0 ${autonomy_box_realsense_pitch} 0"/>
     </xacro:realsense_d435_camera_with_mount_comprehensive_params>
     <!-- Realsense D435 back -->
-    <xacro:realsense_d435_camera_with_mount_comprehensive_params name="back_rgbd_cam" parent="${name}_link" image_topic="image_rect_color" depth_topic="image_rect_raw" depth_points_topic="depth/color/points" min_range="0.3" max_range="9.0" update_rate="15">
+    <xacro:realsense_d435_camera_with_mount_comprehensive_params name="back_rgbd_cam" parent="${name}_link" image_topic="image_rect_color" depth_topic="image_rect_raw" depth_points_topic="depth/color/points" frame_name="depth" min_range="0.3" max_range="9.0" update_rate="15">
       <origin xyz="${-1 * autonomy_box_realsense_x_offset} ${autonomy_box_realsense_y_offset} ${top_protection_bottom + alu_profile_side_length + autonomy_box_realsense_z_offset}" rpy="0.0 ${autonomy_box_realsense_pitch} ${M_PI}"/>
     </xacro:realsense_d435_camera_with_mount_comprehensive_params>

File: hector_sensors_description/urdf/realsense_d435_camera.urdf.xacro (robot description, xacro)
@@ -82,5 +82,5 @@
       </link>
     </xacro:macro>
-    <xacro:macro name="realsense_d435_camera_gazebo_plugin_macro" params="name parent image_topic depth_topic:=image_raw depth_points_topic min_range max_range update_rate">
+    <xacro:macro name="realsense_d435_camera_gazebo_plugin_macro" params="name parent image_topic depth_topic:=image_raw depth_points_topic frame_name:=color min_range max_range update_rate">
       <gazebo reference="${name}_link">
         <sensor type="depth" name="${name}">
@@ -105,5 +105,9 @@
             <depthImageCameraInfoTopicName>depth/camera_info</depthImageCameraInfoTopicName>
             <pointCloudTopicName>${depth_points_topic}</pointCloudTopicName>
-            <frameName>${name}_color_optical_frame</frameName>
+            <frameName>${name}_${frame_name}_optical_frame</frameName>
+            <!-- Important information about frames: Currently, this plugin only supports simulation of color image and depth image/cloud from a single frame.
+            This frame is given in the <gazebo reference=""> tag above and is set to the ${name}_link which coincides with the depth camera frame. The camera axis is the X-axis. ROS requires an optical frame
+            with the Z-axis as camera axis. It is advised to use the depth_optical_frame for this purpose (frame_name="depth"), even though camera images will have the same frame.
+            The color_optical_frame does not coincide with the depth_optical_frame, so depth image/cloud will be misaligned! -->
           </plugin>
         </sensor>
@@ -139,21 +143,21 @@
       <xacro:realsense_camera_gazebo_plugin_macro name="${name}" parent="${parent}" image_topic="image_raw" depth_points_topic="depth/points" min_range="0.3" max_range="9.0" update_rate="20"/>
     </xacro:macro>
-    <xacro:macro name="realsense_d435_camera_no_geom_comprehensive_params" params="name parent *origin image_topic depth_topic:=image_raw depth_points_topic min_range max_range update_rate">
+    <xacro:macro name="realsense_d435_camera_no_geom_comprehensive_params" params="name parent *origin image_topic depth_topic:=image_raw depth_points_topic frame_name:=color min_range max_range update_rate">
       <xacro:realsense_d435_camera_model_no_geom name="${name}" parent="${parent}">
         <xacro:insert_block name="origin" />
       </xacro:realsense_d435_camera_model_no_geom>
-      <xacro:realsense_camera_gazebo_plugin_macro name="${name}" parent="${parent}" image_topic="${image_topic}" depth_topic="${depth_topic}" depth_points_topic="${depth_points_topic}" min_range="${min_range}" max_range="${max_range}" update_rate="${update_rate}"/>
+      <xacro:realsense_camera_gazebo_plugin_macro name="${name}" parent="${parent}" image_topic="${image_topic}" depth_topic="${depth_topic}" depth_points_topic="${depth_points_topic}" frame_name="${frame_name}" min_range="${min_range}" max_range="${max_range}" update_rate="${update_rate}"/>
     </xacro:macro>
-    <xacro:macro name="realsense_d435_camera_comprehensive_params" params="name parent *origin image_topic depth_topic:=image_raw depth_points_topic min_range max_range update_rate">
+    <xacro:macro name="realsense_d435_camera_comprehensive_params" params="name parent *origin image_topic depth_topic:=image_raw depth_points_topic frame_name:=color min_range max_range update_rate">
       <xacro:realsense_d435_camera_model name="${name}" parent="${parent}">
         <xacro:insert_block name="origin" />
       </xacro:realsense_d435_camera_model>
-      <xacro:realsense_d435_camera_gazebo_plugin_macro name="${name}" parent="${parent}" image_topic="${image_topic}" depth_topic="${depth_topic}" depth_points_topic="${depth_points_topic}" min_range="${min_range}" max_range="${max_range}" update_rate="${update_rate}"/>
+      <xacro:realsense_d435_camera_gazebo_plugin_macro name="${name}" parent="${parent}" image_topic="${image_topic}" depth_topic="${depth_topic}" depth_points_topic="${depth_points_topic}" frame_name="${frame_name}" min_range="${min_range}" max_range="${max_range}" update_rate="${update_rate}"/>
     </xacro:macro>
-    <xacro:macro name="realsense_d435_camera_with_mount_comprehensive_params" params="name parent *origin image_topic depth_topic:=image_raw depth_points_topic min_range max_range update_rate">
+    <xacro:macro name="realsense_d435_camera_with_mount_comprehensive_params" params="name parent *origin image_topic depth_topic:=image_raw depth_points_topic frame_name:=color min_range max_range update_rate">
       <xacro:realsense_d435_camera_model_with_mount name="${name}" parent="${parent}">
         <xacro:insert_block name="origin" />
       </xacro:realsense_d435_camera_model_with_mount>
-      <xacro:realsense_d435_camera_gazebo_plugin_macro name="${name}" parent="${parent}" image_topic="${image_topic}" depth_topic="${depth_topic}" depth_points_topic="${depth_points_topic}" min_range="${min_range}" max_range="${max_range}" update_rate="${update_rate}"/>
+      <xacro:realsense_d435_camera_gazebo_plugin_macro name="${name}" parent="${parent}" image_topic="${image_topic}" depth_topic="${depth_topic}" depth_points_topic="${depth_points_topic}" frame_name="${frame_name}" min_range="${min_range}" max_range="${max_range}" update_rate="${update_rate}"/>
     </xacro:macro>
   </robot>

Commit message: replaced the cage D435s by D455s

File: hector_components_description/urdf/autonomy_box.urdf.xacro (robot description, xacro)
@@ -223,16 +223,11 @@
       <origin xyz="0.002862424041614364  -0.00013127655875068252 -0.03724378451297336" rpy="-3.1402707 0.0036289 -3.1175768"/> <!-- insta #3 -->
     </xacro:camera360>
-    <!-- +++++ Cage Realsenses +++++ -->
-    <xacro:property name="autonomy_box_realsense_x_offset" value="0.07187"/>
-    <xacro:property name="autonomy_box_realsense_y_offset" value="0.03"/>
-    <xacro:property name="autonomy_box_realsense_z_offset" value="0.00395"/>
-    <xacro:property name="autonomy_box_realsense_pitch" value="${25*M_PI/180.0}"/>
-    <!-- Realsense D435 front -->
+    <!-- Realsense D455 front -->
     <xacro:realsense_d435_camera_with_mount_comprehensive_params name="front_rgbd_cam" parent="${name}_link" image_topic="image_rect_color" depth_topic="image_rect_raw" depth_points_topic="depth/color/points" frame_name="depth" min_range="0.3" max_range="9.0" update_rate="15">
-      <origin xyz="${autonomy_box_realsense_x_offset} ${-1 * autonomy_box_realsense_y_offset} ${top_protection_bottom + alu_profile_side_length + autonomy_box_realsense_z_offset}" rpy="0.0 ${autonomy_box_realsense_pitch} 0"/>
+      <origin xyz="0.12 0.0 ${top_protection_bottom + alu_profile_side_length + 0.02}" rpy="${M_PI} ${radians(50)} 0"/>
     </xacro:realsense_d435_camera_with_mount_comprehensive_params>
-    <!-- Realsense D435 back -->
+    <!-- Realsense D455 back -->
     <xacro:realsense_d435_camera_with_mount_comprehensive_params name="back_rgbd_cam" parent="${name}_link" image_topic="image_rect_color" depth_topic="image_rect_raw" depth_points_topic="depth/color/points" frame_name="depth" min_range="0.3" max_range="9.0" update_rate="15">
-      <origin xyz="${-1 * autonomy_box_realsense_x_offset} ${autonomy_box_realsense_y_offset} ${top_protection_bottom + alu_profile_side_length + autonomy_box_realsense_z_offset}" rpy="0.0 ${autonomy_box_realsense_pitch} ${M_PI}"/>
+      <origin xyz="-0.105 0.0 ${top_protection_bottom + alu_profile_side_length + 0.025}" rpy="${M_PI} ${radians(30)} ${M_PI}"/>
     </xacro:realsense_d435_camera_with_mount_comprehensive_params>
     <!-- Vive Tracker -->

Commit message: added imu to autonomy box

File: hector_components_description/urdf/autonomy_box.urdf.xacro (robot description, xacro)
@@ -203,4 +203,10 @@
     </joint>
     <link name="${imu_link}">
+      <inertial>
+        <origin xyz='0.0 0.0 0.0' rpy='0.0 0.0 0.0'/>
+        <mass value='0.1'/>
+        <inertia ixx='1.0' ixy='0.0' ixz='0.0'
+                 iyy='1.0' iyz='0.0' izz='1.0'/>
+      </inertial>
     </link>
     <!-- Mocap -->
@@ -248,4 +254,22 @@
     </visual>
     </gazebo>
+    <gazebo reference="imu_link_joint">
+      <preserveFixedJoint>true</preserveFixedJoint>
+    </gazebo>
+    <gazebo>
+      <!-- IMU plugin -->
+      <plugin name="imu_controller" filename="libhector_gazebo_ros_imu.so">
+        <alwaysOn>true</alwaysOn>
+        <updateRate>50.0</updateRate>
+        <bodyName>${imu_link}</bodyName>
+        <topicName>imu/data</topicName>
+        <accelDrift>0.0 0.0 0.0</accelDrift>
+        <accelGaussianNoise>0.1 0.1 0.1</accelGaussianNoise>
+        <rateDrift>0.0 0.0 0.0</rateDrift>
+        <rateGaussianNoise>0.05 0.05 0.05</rateGaussianNoise>
+        <headingDrift>0.0</headingDrift>
+        <headingGaussianNoise>0.05</headingGaussianNoise>
+      </plugin>
+    </gazebo>
   </xacro:macro>
 </robot>

Commit message: adjusted imu weight to match real imu

File: hector_components_description/urdf/autonomy_box.urdf.xacro (robot description, xacro)
@@ -205,5 +205,5 @@
       <inertial>
         <origin xyz='0.0 0.0 0.0' rpy='0.0 0.0 0.0'/>
-        <mass value='0.1'/>
+        <mass value='0.0165'/>
         <inertia ixx='1.0' ixy='0.0' ixz='0.0'
                  iyy='1.0' iyz='0.0' izz='1.0'/>
@@ -257,18 +257,64 @@
       <preserveFixedJoint>true</preserveFixedJoint>
     </gazebo>
-    <gazebo>
-      <!-- IMU plugin -->
-      <plugin name="imu_controller" filename="libhector_gazebo_ros_imu.so">
+    <gazebo reference="${imu_link}">
+      <sensor name="imu" type="imu">
+        <pose>0 0 0 0 0 0</pose>
         <alwaysOn>true</alwaysOn>
         <updateRate>50.0</updateRate>
-        <bodyName>${imu_link}</bodyName>
-        <topicName>imu/data</topicName>
-        <accelDrift>0.0 0.0 0.0</accelDrift>
-        <accelGaussianNoise>0.1 0.1 0.1</accelGaussianNoise>
-        <rateDrift>0.0 0.0 0.0</rateDrift>
-        <rateGaussianNoise>0.05 0.05 0.05</rateGaussianNoise>
-        <headingDrift>0.0</headingDrift>
-        <headingGaussianNoise>0.05</headingGaussianNoise>
-      </plugin>
+        <topic>imu/data</topic>
+        <angular_velocity>
+          <x>
+            <noise type="gaussian">
+              <mean>0.0</mean>
+              <stddev>0.05</stddev>
+              <bias_mean>0.0</bias_mean>
+              <bias_stdev>0.0</bias_stdev>
+            </noise>
+          </x>
+          <y>
+            <noise type="gaussian">
+              <mean>0.0</mean>
+              <stddev>0.05</stddev>
+              <bias_mean>0.0</bias_mean>
+              <bias_stdev>0.0</bias_stdev>
+            </noise>
+          </y>
+          <z>
+            <noise type="gaussian">
+              <mean>0.0</mean>
+              <stddev>0.05</stddev>
+              <bias_mean>0.0</bias_mean>
+              <bias_stdev>0.0</bias_stdev>
+            </noise>
+          </z>
+        </angular_velocity>
+        <linear_acceleration>
+         <x>
+            <noise type="gaussian">
+              <mean>0.0</mean>
+              <stddev>0.05</stddev>
+              <bias_mean>0.0</bias_mean>
+              <bias_stdev>0.0</bias_stdev>
+            </noise>
+          </x>
+          <y>
+            <noise type="gaussian">
+              <mean>0.0</mean>
+              <stddev>0.05</stddev>
+              <bias_mean>0.0</bias_mean>
+              <bias_stdev>0.0</bias_stdev>
+            </noise>
+          </y>
+          <z>
+            <noise type="gaussian">
+              <mean>0.0</mean>
+              <stddev>0.05</stddev>
+              <bias_mean>0.0</bias_mean>
+              <bias_stdev>0.0</bias_stdev>
+            </noise>
+          </z>
+        </linear_acceleration>
+        <enable_orientation>true</enable_orientation>
+      </sensor>
     </gazebo>
   </xacro:macro>

Commit message: Revert "adjusted imu weight to match real imu"
This reverts commit 639e31cb68182274d2899c9572e8ef23d5a624e4.

File: hector_components_description/urdf/autonomy_box.urdf.xacro (robot description, xacro)
@@ -205,5 +205,5 @@
       <inertial>
         <origin xyz='0.0 0.0 0.0' rpy='0.0 0.0 0.0'/>
-        <mass value='0.0165'/>
+        <mass value='0.1'/>
         <inertia ixx='1.0' ixy='0.0' ixz='0.0'
                  iyy='1.0' iyz='0.0' izz='1.0'/>
@@ -257,64 +257,18 @@
       <preserveFixedJoint>true</preserveFixedJoint>
     </gazebo>
-    <gazebo reference="${imu_link}">
-      <sensor name="imu" type="imu">
-        <pose>0 0 0 0 0 0</pose>
+    <gazebo>
+      <!-- IMU plugin -->
+      <plugin name="imu_controller" filename="libhector_gazebo_ros_imu.so">
         <alwaysOn>true</alwaysOn>
         <updateRate>50.0</updateRate>
-        <topic>imu/data</topic>
-        <angular_velocity>
-          <x>
-            <noise type="gaussian">
-              <mean>0.0</mean>
-              <stddev>0.05</stddev>
-              <bias_mean>0.0</bias_mean>
-              <bias_stdev>0.0</bias_stdev>
-            </noise>
-          </x>
-          <y>
-            <noise type="gaussian">
-              <mean>0.0</mean>
-              <stddev>0.05</stddev>
-              <bias_mean>0.0</bias_mean>
-              <bias_stdev>0.0</bias_stdev>
-            </noise>
-          </y>
-          <z>
-            <noise type="gaussian">
-              <mean>0.0</mean>
-              <stddev>0.05</stddev>
-              <bias_mean>0.0</bias_mean>
-              <bias_stdev>0.0</bias_stdev>
-            </noise>
-          </z>
-        </angular_velocity>
-        <linear_acceleration>
-         <x>
-            <noise type="gaussian">
-              <mean>0.0</mean>
-              <stddev>0.05</stddev>
-              <bias_mean>0.0</bias_mean>
-              <bias_stdev>0.0</bias_stdev>
-            </noise>
-          </x>
-          <y>
-            <noise type="gaussian">
-              <mean>0.0</mean>
-              <stddev>0.05</stddev>
-              <bias_mean>0.0</bias_mean>
-              <bias_stdev>0.0</bias_stdev>
-            </noise>
-          </y>
-          <z>
-            <noise type="gaussian">
-              <mean>0.0</mean>
-              <stddev>0.05</stddev>
-              <bias_mean>0.0</bias_mean>
-              <bias_stdev>0.0</bias_stdev>
-            </noise>
-          </z>
-        </linear_acceleration>
-        <enable_orientation>true</enable_orientation>
-      </sensor>
+        <bodyName>${imu_link}</bodyName>
+        <topicName>imu/data</topicName>
+        <accelDrift>0.0 0.0 0.0</accelDrift>
+        <accelGaussianNoise>0.1 0.1 0.1</accelGaussianNoise>
+        <rateDrift>0.0 0.0 0.0</rateDrift>
+        <rateGaussianNoise>0.05 0.05 0.05</rateGaussianNoise>
+        <headingDrift>0.0</headingDrift>
+        <headingGaussianNoise>0.05</headingGaussianNoise>
+      </plugin>
     </gazebo>
   </xacro:macro>

Commit message: fixed imu weight

File: hector_components_description/urdf/autonomy_box.urdf.xacro (robot description, xacro)
@@ -205,5 +205,5 @@
       <inertial>
         <origin xyz='0.0 0.0 0.0' rpy='0.0 0.0 0.0'/>
-        <mass value='0.1'/>
+        <mass value='0.0165'/>
         <inertia ixx='1.0' ixy='0.0' ixz='0.0'
                  iyy='1.0' iyz='0.0' izz='1.0'/>

Commit message: reverted lense placement and tuned D455 locations. Added static transform publisher for D455

File: hector_components_description/urdf/autonomy_box.urdf.xacro (robot description, xacro)
@@ -6,5 +6,4 @@
   <xacro:include filename="$(find hector_sensors_description)/urdf/camera360.urdf.xacro"/>
   <xacro:include filename="$(find hector_sensors_description)/urdf/realsense_d455_camera.urdf.xacro"/>
-  <!--<xacro:include filename="$(find realsense2_description)/urdf/_d455.urdf.xacro"/>  -->
 <!--  <xacro:arg name="add_self_filter_geom" default="0"/>-->
   <!--<xacro:property name="add_self_filter_geom" value="${arg add_self_filter_geom}"/>-->
@@ -226,9 +225,9 @@
     <!-- Realsense D455 front -->
     <xacro:realsense_d455_camera_with_mount_comprehensive_params name="front_rgbd_cam" parent="${name}_link" image_topic="image_rect_color" depth_topic="image_rect_raw" depth_points_topic="depth/color/points" frame_name="depth" min_range="0.3" max_range="9.0" update_rate="15">
-      <origin xyz="0.12 0.0 ${top_protection_bottom + alu_profile_side_length + 0.02}" rpy="${M_PI} ${radians(50)} 0"/>
+      <origin xyz="0.12 -0.034 ${top_protection_bottom + alu_profile_side_length + 0.02}" rpy="${M_PI + radians(2)} ${radians(50)} 0"/>
     </xacro:realsense_d455_camera_with_mount_comprehensive_params>
     <!-- Realsense D455 back -->
     <xacro:realsense_d455_camera_with_mount_comprehensive_params name="back_rgbd_cam" parent="${name}_link" image_topic="image_rect_color" depth_topic="image_rect_raw" depth_points_topic="depth/color/points" frame_name="depth" min_range="0.3" max_range="9.0" update_rate="15">
-      <origin xyz="-0.105 0.0 ${top_protection_bottom + alu_profile_side_length + 0.025}" rpy="${M_PI} ${radians(30)} ${M_PI}"/>
+      <origin xyz="-0.105 0.014 ${top_protection_bottom + alu_profile_side_length + 0.025}" rpy="${M_PI} ${radians(27)} ${M_PI - radians(1)}"/>
     </xacro:realsense_d455_camera_with_mount_comprehensive_params>
     <!-- Vive Tracker -->

File: hector_sensors_description/urdf/realsense_d455_camera.urdf.xacro (robot description, xacro)
@@ -44,10 +44,10 @@
       <parent link="${name}_mount_link"/>
       <child link="${name}_link"/>
-      <origin xyz="${d455_mount_hole_to_front - d455_front_to_depth} ${d455_mount_hole_to_color_cam} ${d455_cam_height/2}" rpy="0 0 0"/>
+      <origin xyz="${d455_mount_hole_to_front - d455_front_to_depth} ${d455_cam_depth_py} ${d455_cam_height/2}" rpy="0 0 0"/>
     </joint>
     <link name="${name}_link">
       <visual>
         <!-- the mesh origin is at front plate in between the two infrared camera axes -->
-        <origin xyz="${d455_front_to_depth} ${-d455_mount_hole_to_color_cam} 0" rpy="0 0 ${M_PI/2}"/>
+        <origin xyz="${d455_front_to_depth} ${-d455_cam_depth_py} 0" rpy="0 0 ${M_PI/2}"/>
         <geometry>
           <!-- <box size="${d455_cam_depth} ${d455_cam_width} ${d455_cam_height}"/> -->
@@ -57,5 +57,5 @@
       </visual>
       <collision>
-        <origin xyz="${-d455_cam_depth/2 + d455_front_to_depth} ${-d455_mount_hole_to_color_cam} 0" rpy="0 0 0"/>
+        <origin xyz="${-d455_cam_depth/2 + d455_front_to_depth} ${-d455_cam_depth_py} 0" rpy="0 0 0"/>
         <geometry>
           <box size="${d455_cam_depth} ${d455_cam_width} ${d455_cam_height}"/>

Commit message: tuned pitch of damaged D455

File: hector_components_description/urdf/autonomy_box.urdf.xacro (robot description, xacro)
@@ -235,5 +235,5 @@
     <!-- Realsense D455 back -->
     <xacro:realsense_d455_camera_with_mount_comprehensive_params name="back_rgbd_cam" parent="${name}_link" image_topic="image_rect_color" depth_topic="image_rect_raw" depth_points_topic="depth/color/points" frame_name="depth" min_range="0.3" max_range="9.0" update_rate="15">
-      <origin xyz="-0.105 0.014 ${top_protection_bottom + alu_profile_side_length + 0.025}" rpy="${M_PI} ${radians(27)} ${M_PI - radians(1)}"/>
+      <origin xyz="-0.105 0.014 ${top_protection_bottom + alu_profile_side_length + 0.025}" rpy="${M_PI} ${radians(30)} ${M_PI - radians(1)}"/>
     </xacro:realsense_d455_camera_with_mount_comprehensive_params>
     <!-- Vive Tracker -->
