Commit message: Filter everything at the top of the vision box for simplicity.
We don't need the points straight up and there are cables, mounts and other elements that change and clutter the pointcloud.

File: hector_components_description/urdf/autonomy_box.urdf.xacro (robot description, xacro)
@@ -106,38 +106,7 @@
       <!--Top geom-->
       <collision>
-        <origin xyz="0 ${ (computer_box_width/2-alu_profile_side_length/2)} ${top_protection_bottom + alu_profile_side_length/2}" rpy="0 ${M_PI*0.5} 0"/>
-        <geometry>
-          <!--<box size="${computer_box_length} ${alu_profile_side_length} ${alu_profile_side_length}"/>-->
-          <cylinder length="${computer_box_length}" radius="${alu_profile_side_length*0.5*alu_profile_collision_size_factor}"/>
-        </geometry>
-        <material name="Grey">
-          <color rgba="0.5 0.5 0.5 1"/>
-        </material>
-      </collision>
-      <collision>
-        <origin xyz="0 ${-(computer_box_width/2-alu_profile_side_length/2)} ${top_protection_bottom + alu_profile_side_length/2}" rpy="0 ${M_PI*0.5} 0"/>
-        <geometry>
-          <!--<box size="${computer_box_length} ${alu_profile_side_length} ${alu_profile_side_length}"/>-->
-          <cylinder length="${computer_box_length}" radius="${alu_profile_side_length*0.5*alu_profile_collision_size_factor}"/>
-        </geometry>
-        <material name="Grey">
-          <color rgba="0.5 0.5 0.5 1"/>
-        </material>
-      </collision>
-      <collision>
-        <origin xyz="${ (computer_box_length/2-alu_profile_side_length/2)} 0 ${top_protection_bottom + alu_profile_side_length/2}" rpy="${M_PI*0.5} ${M_PI*0.5} 0"/>
-        <geometry>
-          <!--<box size="${alu_profile_side_length} ${computer_box_width}  ${alu_profile_side_length}"/>-->
-          <cylinder length="${computer_box_width}" radius="${alu_profile_side_length*0.5*alu_profile_collision_size_factor}"/>
-        </geometry>
-        <material name="Grey">
-          <color rgba="0.5 0.5 0.5 1"/>
-        </material>
-      </collision>
-      <collision>
-        <origin xyz="${-(computer_box_length/2-alu_profile_side_length/2)} 0 ${top_protection_bottom + alu_profile_side_length/2}" rpy="${M_PI*0.5} ${M_PI*0.5} 0"/>
-        <geometry>
-          <!--<box size="${alu_profile_side_length} ${computer_box_width}  ${alu_profile_side_length}"/>-->
-          <cylinder length="${computer_box_width}" radius="${alu_profile_side_length*0.5*alu_profile_collision_size_factor}"/>
+        <origin xyz="0 0 ${top_protection_bottom + alu_profile_side_length/2}" />
+        <geometry>
+          <box size="${computer_box_length} ${computer_box_length} ${alu_profile_side_length}"/>
         </geometry>
         <material name="Grey">

Commit message: Added weight to autonomy box to make it more realistic.

File: hector_components_description/urdf/autonomy_box.urdf.xacro (robot description, xacro)
@@ -35,5 +35,7 @@
     <!-- Computer box and cage -->
     <link name="${name}_link">
-      <xacro:inertial_sphere mass="0.1" diameter="0.07"/>
+      <xacro:inertial_sphere_with_pose mass="5.6" diameter="0.07">
+        <origin xyz="0.0 0.0 0.30" rpy="0 0 0" />
+      </xacro:inertial_sphere_with_pose>
       <visual>
         <origin rpy="0 0 0" xyz="-0.095 -0.095 0"/>

Commit message: added new rgbd pos to urdf

File: hector_components_description/urdf/autonomy_box.urdf.xacro (robot description, xacro)
@@ -202,9 +202,9 @@
     <!-- Realsense D455 front -->
     <xacro:realsense_d455_camera_with_mount_comprehensive_params name="front_rgbd_cam" parent="${name}_link" image_topic="image_rect_color" depth_topic="image_rect_raw" depth_points_topic="depth/color/points" frame_name="depth" min_range="0.3" max_range="9.0" update_rate="15">
-      <origin xyz="0.12 -0.034 ${top_protection_bottom + alu_profile_side_length + 0.02}" rpy="${M_PI + radians(2)} ${radians(50)} 0"/>
+      <origin xyz="0.0775 0.0115 ${top_protection_bottom + alu_profile_side_length + 0.01}" rpy="${radians(0)} ${radians(48)} 0"/>
     </xacro:realsense_d455_camera_with_mount_comprehensive_params>
     <!-- Realsense D455 back -->
     <xacro:realsense_d455_camera_with_mount_comprehensive_params name="back_rgbd_cam" parent="${name}_link" image_topic="image_rect_color" depth_topic="image_rect_raw" depth_points_topic="depth/color/points" frame_name="depth" min_range="0.3" max_range="9.0" update_rate="15">
-      <origin xyz="-0.105 0.014 ${top_protection_bottom + alu_profile_side_length + 0.025}" rpy="${M_PI} ${radians(30)} ${M_PI - radians(1)}"/>
+      <origin xyz="-0.0765 -0.0115 ${top_protection_bottom + alu_profile_side_length + 0.005}" rpy="${radians(0)} ${radians(25)} ${M_PI - radians(0)}"/>
     </xacro:realsense_d455_camera_with_mount_comprehensive_params>
     <!-- Vive Tracker -->

Commit message: updated vision_box stl

File: hector_components_description/urdf/autonomy_box.urdf.xacro (robot description, xacro)
@@ -39,5 +39,5 @@
       </xacro:inertial_sphere_with_pose>
       <visual>
-        <origin rpy="0 0 0" xyz="-0.095 -0.095 0"/>
+	<origin rpy="0 0 ${M_PI}" xyz="-0.095 -0.095 0"/>
         <geometry>
           <mesh filename="package://hector_components_description/meshes/autonomy_box/visionbox_no_lidar.stl" scale="0.001 0.001 0.001" />

Commit message: Updated Asterix RGBD Positions and stl (#14)
* added new rgbd pos to urdf

* replaced autonomybox stl with newer version

* updated vision_box stl

* added new vision_box.stl

---------

Co-authored-by: lenng853 <116359042+lenng853@users.noreply.github.com>

File: hector_components_description/urdf/autonomy_box.urdf.xacro (robot description, xacro)
@@ -39,5 +39,5 @@
       </xacro:inertial_sphere_with_pose>
       <visual>
-        <origin rpy="0 0 0" xyz="-0.095 -0.095 0"/>
+	<origin rpy="0 0 ${M_PI}" xyz="-0.095 -0.095 0"/>
         <geometry>
           <mesh filename="package://hector_components_description/meshes/autonomy_box/visionbox_no_lidar.stl" scale="0.001 0.001 0.001" />
@@ -202,9 +202,9 @@
     <!-- Realsense D455 front -->
     <xacro:realsense_d455_camera_with_mount_comprehensive_params name="front_rgbd_cam" parent="${name}_link" image_topic="image_rect_color" depth_topic="image_rect_raw" depth_points_topic="depth/color/points" frame_name="depth" min_range="0.3" max_range="9.0" update_rate="15">
-      <origin xyz="0.12 -0.034 ${top_protection_bottom + alu_profile_side_length + 0.02}" rpy="${M_PI + radians(2)} ${radians(50)} 0"/>
+      <origin xyz="0.0775 0.0115 ${top_protection_bottom + alu_profile_side_length + 0.01}" rpy="${radians(0)} ${radians(48)} 0"/>
     </xacro:realsense_d455_camera_with_mount_comprehensive_params>
     <!-- Realsense D455 back -->
     <xacro:realsense_d455_camera_with_mount_comprehensive_params name="back_rgbd_cam" parent="${name}_link" image_topic="image_rect_color" depth_topic="image_rect_raw" depth_points_topic="depth/color/points" frame_name="depth" min_range="0.3" max_range="9.0" update_rate="15">
-      <origin xyz="-0.105 0.014 ${top_protection_bottom + alu_profile_side_length + 0.025}" rpy="${M_PI} ${radians(30)} ${M_PI - radians(1)}"/>
+      <origin xyz="-0.0765 -0.0115 ${top_protection_bottom + alu_profile_side_length + 0.005}" rpy="${radians(0)} ${radians(25)} ${M_PI - radians(0)}"/>
     </xacro:realsense_d455_camera_with_mount_comprehensive_params>
     <!-- Vive Tracker -->

Commit message: back rgbd calibration

File: hector_components_description/urdf/autonomy_box.urdf.xacro (robot description, xacro)
@@ -206,5 +206,5 @@
     <!-- Realsense D455 back -->
     <xacro:realsense_d455_camera_with_mount_comprehensive_params name="back_rgbd_cam" parent="${name}_link" image_topic="image_rect_color" depth_topic="image_rect_raw" depth_points_topic="depth/color/points" frame_name="depth" min_range="0.3" max_range="9.0" update_rate="15">
-      <origin xyz="-0.0765 -0.0115 ${top_protection_bottom + alu_profile_side_length + 0.005}" rpy="${radians(0)} ${radians(25)} ${M_PI - radians(0)}"/>
+      <origin xyz="-0.0765 -0.0115 ${top_protection_bottom + alu_profile_side_length + 0.005}" rpy="${radians(0)} ${radians(22.5)} ${M_PI - radians(0)}"/>
     </xacro:realsense_d455_camera_with_mount_comprehensive_params>
     <!-- Vive Tracker -->
