Commit message: Add additional macros

File: hector_xacro_tools/urdf/inertia_tensors.urdf.xacro (robot description, xacro)
@@ -3,4 +3,14 @@
   <xacro:macro name="inertial_cuboid" params="mass x_length y_length z_length">
     <inertial>
+      <mass value="${mass}" />
+      <origin xyz="0 0 0" />
+      <inertia ixx="${(1/12) * mass* (y_length*y_length+ z_length*z_length)}" ixy="0.0" ixz="0.0"
+               iyy="${(1/12) * mass* (x_length*x_length+ z_length*z_length)}" iyz="0.0"
+               izz="${(1/12) * mass* (x_length*x_length+ y_length*y_length)}" />
+    </inertial>
+  </xacro:macro>
+  <xacro:macro name="inertial_cuboid_with_pose" params="mass x_length y_length z_length *origin">
+    <inertial>
+      <insert_block name="origin"/>
       <mass value="${mass}" />
       <origin xyz="0 0 0" />
@@ -19,3 +29,12 @@
     </inertial>
   </xacro:macro>
+  <xacro:macro name="inertial_sphere_with_pose" params="mass diameter *origin">
+    <inertial>
+      <insert_block name="origin"/>
+      <mass value="${mass}" />
+      <inertia ixx="${(2/5) * mass* ( (diameter*0.5)) * (diameter*0.5))}" ixy="0.0" ixz="0.0"
+               iyy="${(2/5) * mass* ( (diameter*0.5)) * (diameter*0.5))}" iyz="0.0"
+               izz="${(2/5) * mass* ( (diameter*0.5)) * (diameter*0.5))}" />
+    </inertial>
+  </xacro:macro>
 </robot>

Commit message: Remove origin tag as already set via insert block

File: hector_xacro_tools/urdf/inertia_tensors.urdf.xacro (robot description, xacro)
@@ -14,5 +14,4 @@
       <insert_block name="origin"/>
       <mass value="${mass}" />
-      <origin xyz="0 0 0" />
       <inertia ixx="${(1/12) * mass* (y_length*y_length+ z_length*z_length)}" ixy="0.0" ixz="0.0"
                iyy="${(1/12) * mass* (x_length*x_length+ z_length*z_length)}" iyz="0.0"

Commit message: hector_xacro_tools: fixed invalid brackets in inertial_sphere* xacro macros

File: hector_xacro_tools/urdf/inertia_tensors.urdf.xacro (robot description, xacro)
@@ -5,7 +5,7 @@
       <mass value="${mass}" />
       <origin xyz="0 0 0" />
-      <inertia ixx="${(1/12) * mass* (y_length*y_length+ z_length*z_length)}" ixy="0.0" ixz="0.0"
-               iyy="${(1/12) * mass* (x_length*x_length+ z_length*z_length)}" iyz="0.0"
-               izz="${(1/12) * mass* (x_length*x_length+ y_length*y_length)}" />
+      <inertia ixx="${(1/12) * mass * (y_length*y_length + z_length*z_length)}" ixy="0.0" ixz="0.0"
+               iyy="${(1/12) * mass * (x_length*x_length + z_length*z_length)}" iyz="0.0"
+               izz="${(1/12) * mass * (x_length*x_length + y_length*y_length)}" />
     </inertial>
   </xacro:macro>
@@ -14,7 +14,7 @@
       <xacro:insert_block name="origin"/>
       <mass value="${mass}" />
-      <inertia ixx="${(1/12) * mass* (y_length*y_length+ z_length*z_length)}" ixy="0.0" ixz="0.0"
-               iyy="${(1/12) * mass* (x_length*x_length+ z_length*z_length)}" iyz="0.0"
-               izz="${(1/12) * mass* (x_length*x_length+ y_length*y_length)}" />
+      <inertia ixx="${(1/12) * mass * (y_length*y_length + z_length*z_length)}" ixy="0.0" ixz="0.0"
+               iyy="${(1/12) * mass * (x_length*x_length + z_length*z_length)}" iyz="0.0"
+               izz="${(1/12) * mass * (x_length*x_length + y_length*y_length)}" />
     </inertial>
   </xacro:macro>
@@ -23,7 +23,7 @@
       <mass value="${mass}" />
       <origin xyz="0 0 0" />
-      <inertia ixx="${(2/5) * mass* ( (diameter*0.5)) * (diameter*0.5))}" ixy="0.0" ixz="0.0"
-               iyy="${(2/5) * mass* ( (diameter*0.5)) * (diameter*0.5))}" iyz="0.0"
-               izz="${(2/5) * mass* ( (diameter*0.5)) * (diameter*0.5))}" />
+      <inertia ixx="${(2/5) * mass * ( (diameter*0.5) * (diameter*0.5) )}" ixy="0.0" ixz="0.0"
+               iyy="${(2/5) * mass * ( (diameter*0.5) * (diameter*0.5) )}" iyz="0.0"
+               izz="${(2/5) * mass * ( (diameter*0.5) * (diameter*0.5) )}" />
     </inertial>
   </xacro:macro>
@@ -32,7 +32,7 @@
       <xacro:insert_block name="origin"/>
       <mass value="${mass}" />
-      <inertia ixx="${(2/5) * mass* ( (diameter*0.5)) * (diameter*0.5))}" ixy="0.0" ixz="0.0"
-               iyy="${(2/5) * mass* ( (diameter*0.5)) * (diameter*0.5))}" iyz="0.0"
-               izz="${(2/5) * mass* ( (diameter*0.5)) * (diameter*0.5))}" />
+      <inertia ixx="${(2/5) * mass * ( (diameter*0.5) * (diameter*0.5) )}" ixy="0.0" ixz="0.0"
+               iyy="${(2/5) * mass * ( (diameter*0.5) * (diameter*0.5) )}" iyz="0.0"
+               izz="${(2/5) * mass * ( (diameter*0.5) * (diameter*0.5) )}" />
     </inertial>
   </xacro:macro>
