Commit message: position interface macro

File: hector_xacro_tools/urdf/joint_macros.urdf.xacro (robot description, xacro)
@@ -16,3 +16,18 @@
     </gazebo>
   </xacro:macro>
+  <xacro:macro name="joint_position_transmission" params="name">
+    <transmission name="${name}_joint_transmission">
+      <type>transmission_interface/SimpleTransmission</type>
+      <joint name="${name}">
+        <hardwareInterface>hardware_interface/PositionJointInterface</hardwareInterface>
+      </joint>
+      <actuator name="${name}_joint_motor">
+        <hardwareInterface>hardware_interface/PositionJointInterface</hardwareInterface>
+        <mechanicalReduction>1</mechanicalReduction>
+      </actuator>
+    </transmission>
+    <gazebo reference="${name}">
+      <implicitSpringDamper>1</implicitSpringDamper>
+    </gazebo>
+  </xacro:macro>
 </robot>

Commit message: Added velociy transmission

File: hector_xacro_tools/urdf/joint_macros.urdf.xacro (robot description, xacro)
@@ -31,3 +31,18 @@
     </gazebo>
   </xacro:macro>
+  <xacro:macro name="joint_velocity_transmission" params="name">
+    <transmission name="${name}_joint_transmission">
+      <type>transmission_interface/SimpleTransmission</type>
+      <joint name="${name}">
+        <hardwareInterface>hardware_interface/VelocityJointInterface</hardwareInterface>
+      </joint>
+      <actuator name="${name}_joint_motor">
+        <hardwareInterface>hardware_interface/VelocityJointInterface</hardwareInterface>
+        <mechanicalReduction>1</mechanicalReduction>
+      </actuator>
+    </transmission>
+    <gazebo reference="${name}">
+      <implicitSpringDamper>1</implicitSpringDamper>
+    </gazebo>
+  </xacro:macro>
 </robot>
