Commit message: add insta360air

File: gazebo/insta360_air.gazebo.xacro (robot description, xacro)
@@ -1,5 +1,63 @@
 <?xml version="1.0"?>
 <robot xmlns:xacro="http://ros.org/wiki/xacro">
+    <xacro:property name="M_PI" value="3.14159"/>
     <xacro:macro name="insta360_air_gazebo" params="name:=default">
+        <gazebo reference="insta360_air_${name}_left_optical_frame">
+            <sensor type="wideanglecamera" name="insta360_air_${name}_left">
+                <always_on>true</always_on>
+                <visualize>true</visualize>
+                <update_rate>15</update_rate>
+                <topic>/$(arg robot_name)/insta360_air_${name}_left/rgb/image_raw</topic>
+                <gz_frame_id>insta360_air_${name}_left_optical_frame</gz_frame_id>
+                <camera>
+                    <camera_info_topic>/$(arg robot_name)/insta360_air_${name}_left/rgb/camera_info</camera_info_topic>
+                    <horizontal_fov>${M_PI}</horizontal_fov>
+                    <image>
+                        <format>R8G8B8</format>
+                        <width>720</width>
+                        <height>480</height>
+                    </image>
+                    <clip>
+                        <near>0.05</near>
+                        <far>10</far>
+                    </clip>
+                    <lens>
+                        <type>stereographic</type>
+                        <scale_to_hfov>true</scale_to_hfov>
+                        <cutoff_angle>1.5707</cutoff_angle>
+                        <env_texture_size>512</env_texture_size>
+                    </lens>
+                </camera>
+            </sensor>
+        </gazebo>
+        <gazebo reference="insta360_air_${name}_right_optical_frame">
+            <sensor type="wideanglecamera" name="insta360_air_${name}_right">
+                <always_on>true</always_on>
+                <visualize>true</visualize>
+                <update_rate>15</update_rate>
+                <topic>/$(arg robot_name)/insta360_air_${name}_right/rgb/image_raw</topic>
+                <gz_frame_id>insta360_air_${name}_right_optical_frame</gz_frame_id>
+                <camera>
+                    <camera_info_topic>/$(arg robot_name)/insta360_air_${name}_right/rgb/camera_info</camera_info_topic>
+                    <optical_frame_id>insta360_air_${name}_right_optical_frame</optical_frame_id>
+                    <horizontal_fov>${M_PI}</horizontal_fov>
+                    <image>
+                        <format>R8G8B8</format>
+                        <width>720</width>
+                        <height>480</height>
+                    </image>
+                    <clip>
+                        <near>0.05</near>
+                        <far>10</far>
+                    </clip>
+                    <lens>
+                        <type>stereographic</type>
+                        <scale_to_hfov>true</scale_to_hfov>
+                        <cutoff_angle>1.5707</cutoff_angle>
+                        <env_texture_size>512</env_texture_size>
+                    </lens>
+                </camera>
+            </sensor>
+        </gazebo>
     </xacro:macro>
 </robot>

File: gazebo/seek_thermal_xr.gazebo.xacro (robot description, xacro)
@@ -1,4 +1,5 @@
 <?xml version="1.0"?>
 <robot xmlns:xacro="http://ros.org/wiki/xacro">
+	<xacro:property name="M_PI" value="3.14159"/>
     <xacro:macro name="seek_thermal_xr_gazebo" params="name:=default">
     </xacro:macro>

File: urdf/astra_stereo_s_u3.xacro (robot description, xacro)
@@ -1,5 +1,11 @@
 <?xml version="1.0"?>
 <robot xmlns:xacro="http://ros.org/wiki/xacro">
-    <xacro:macro name="orbbec_astra_stereo_s_u3" params="name:=default">
+    <xacro:property name="M_PI" value="3.14159"/>
+    <xacro:macro name="orbbec_astra_stereo_s_u3" params="name:=default *origin *parent">
+        <joint name="astra_stereo_s_${name}_base_joint" type="fixed">
+            <child link="astra_stereo_s_${name}_base_link"/>
+            <xacro:insert_block name="origin"/>
+            <xacro:insert_block name="parent"/>
+        </joint>
         <!-- Camera base -->
         <link name="astra_stereo_s_${name}_base_link">

File: urdf/insta360_air.xacro (robot description, xacro)
@@ -1,5 +1,11 @@
 <?xml version="1.0"?>
 <robot xmlns:xacro="http://ros.org/wiki/xacro">
-    <xacro:macro name="insta360_air" params="name:=default">
+    <xacro:property name="M_PI" value="3.14159"/>
+    <xacro:macro name="insta360_air" params="name:=default *origin *parent">
+        <joint name="insta360_air_${name}_base_joint" type="fixed">
+            <child link="insta360_air_${name}_base_link"/>
+            <xacro:insert_block name="origin"/>
+            <xacro:insert_block name="parent"/>
+        </joint>
         <!-- Camera base -->
         <link name="insta360_air_${name}_base_link">
@@ -18,15 +24,15 @@
         </link>
         <!-- Camera RGB sensor -->
-        <link name="insta360_air_${name}_left_optical_link"/>
+        <link name="insta360_air_${name}_left_optical_frame"/>
         <joint name="insta360_air_${name}_left_optical_joint" type="fixed">
             <origin xyz="0 0 0" rpy="0 0 0" />
             <parent link="insta360_air_${name}_base_link" />
-            <child link="insta360_air_${name}_left_optical_link" />
+            <child link="insta360_air_${name}_left_optical_frame" />
         </joint>
-        <link name="insta360_air_${name}_right_optical_link"/>
+        <link name="insta360_air_${name}_right_optical_frame"/>
         <joint name="insta360_air_${name}_right_optical_joint" type="fixed">
             <origin xyz="0 0 0" rpy="0 0 ${M_PI}" />
             <parent link="insta360_air_${name}_base_link" />
-            <child link="insta360_air_${name}_right_optical_link" />
+            <child link="insta360_air_${name}_right_optical_frame" />
         </joint>
     </xacro:macro>

File: urdf/livox_mid360.xacro (robot description, xacro)
@@ -2,5 +2,10 @@
 <robot xmlns:xacro="http://ros.org/wiki/xacro">
 	<xacro:property name="M_PI" value="3.14159"/>
-	<xacro:macro name="livox_mid360" params="name:=default">
+	<xacro:macro name="livox_mid360" params="name:=default *origin *parent">
+		<joint name="livox_mid360_${name}_joint" type="fixed">
+			<child link="livox_mid360_${name}_link"/>
+			<xacro:insert_block name="origin"/>
+			<xacro:insert_block name="parent"/>
+		</joint>
 		<link name="livox_mid360_${name}_link">
 			<visual>

File: urdf/orbbec_astra2.xacro (robot description, xacro)
@@ -2,5 +2,10 @@
 <robot xmlns:xacro="http://ros.org/wiki/xacro">
     <xacro:property name="M_PI" value="3.14159"/>
-    <xacro:macro name="orbbec_astra2" params="name:=default">
+    <xacro:macro name="orbbec_astra2" params="name:=default *origin *parent">
+		<joint name="astra2_${name}_base_joint" type="fixed">
+			<child link="astra2_${name}_base_link"/>
+			<xacro:insert_block name="origin"/>
+			<xacro:insert_block name="parent"/>
+		</joint>
         <!-- Camera base -->
         <link name="astra2_${name}_base_link">

File: urdf/seek_thermal_xr.xacro (robot description, xacro)
@@ -1,7 +1,13 @@
 <?xml version="1.0"?>
 <robot xmlns:xacro="http://ros.org/wiki/xacro">
-    <xacro:macro name="seek_thermal_xr" params="name:=default">
+    <xacro:property name="M_PI" value="3.14159"/>
+    <xacro:macro name="seek_thermal_xr" params="name:=default *origin *parent">
+        <joint name="seek_thermal_xr_${name}_base_joint" type="fixed">
+            <child link="seek_thermal_xr_${name}_base_link"/>
+            <xacro:insert_block name="origin"/>
+            <xacro:insert_block name="parent"/>
+        </joint>
         <!-- Camera base -->
-        <link name="seek_thermal_${name}_base_link">
+        <link name="seek_thermal_xr_${name}_base_link">
             <visual>
                 <origin xyz="0 0 0" rpy="0 0 0" />
@@ -18,9 +24,9 @@
         </link>
         <!-- Camera sensor -->
-        <link name="seek_thermal_${name}_link"/>
-        <joint name="seek_thermal_${name}_sensor_joint" type="fixed">
+        <link name="seek_thermal_xr_${name}_link"/>
+        <joint name="seek_thermal_xr_${name}_sensor_joint" type="fixed">
             <origin xyz="0.025 0 0" rpy="0 0 0" />
-            <parent link="seek_thermal_${name}_base_link" />
-            <child link="seek_thermal_${name}_link" />
+            <parent link="seek_thermal_xr_${name}_base_link" />
+            <child link="seek_thermal_xr_${name}_link" />
         </joint>
     </xacro:macro>

File: urdf/sensor_macros.urdf.xacro (robot description, xacro)
@@ -1,11 +1,12 @@
 <?xml version="1.0"?>
 <robot xmlns:xacro="http://www.ros.org/wiki/xacro">
-  <xacro:macro name="add_optical_frame" params="name">
-    <joint name="${name}_optical_joint" type="fixed">
-      <origin xyz="0 0 0" rpy="${-M_PI/2} 0.0 ${-M_PI/2}" />
-      <parent link="${name}_frame" />
-      <child link="${name}_optical_frame"/>
-    </joint>
-    <link name="${name}_optical_frame" />
-  </xacro:macro>
+	<xacro:property name="M_PI" value="3.14159"/>
+	<xacro:macro name="add_optical_frame" params="name">
+		<joint name="${name}_optical_joint" type="fixed">
+			<origin xyz="0 0 0" rpy="${-M_PI/2} 0.0 ${-M_PI/2}" />
+			<parent link="${name}_frame" />
+			<child link="${name}_optical_frame"/>
+		</joint>
+		<link name="${name}_optical_frame" />
+	</xacro:macro>
 </robot>
